Commit message: 20250303 增加末端工具

File: catkin_ws/src/fr5v6_single_moveit_config/config/gazebo_fr5v6_single_arm.urdf (robot description, URDF)
Before this commit: robot fr5v6_single_arm, 10 links, 9 joints
Links:
- added link fr5v6_tool_Link, mass 0; collision mesh filename=package://frcobot_description/meshes/fr5v6/collision/toolA-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 scale=0.001 0.001 0.001; visual mesh filename=package://frcobot_description/meshes/fr5v6/visual/toolA-250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 scale=0.001 0.001 0.001
- added link fr5v6_tool_tcp_link, mass 0.001; visual sphere radius=0.005
- link fr5v6_base_link: geometry collision mesh filename=package://frcobot_description/meshes/fr5v6/collision/base_l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 scale=1 1 1; visual mesh filename=package://frcobot_description/meshes/fr5v6/visual/base_link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 scale=1 1 1
- link fr5v6_extra_base_link: geometry collision mesh filename=package://frcobot_description/meshes/fr5v6/collision/extra_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 scale=1 1 1; visual mesh filename=package://frcobot_description/meshes/fr5v6/visual/extra_bas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 scale=1 1 1
- link fr5v6_j1_Link: geometry collision mesh filename=package://frcobot_description/meshes/fr5v6/collision/j1_Lin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 scale=1 1 1; visual mesh filename=package://frcobot_description/meshes/fr5v6/visual/j1_Link.D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 scale=1 1 1
- link fr5v6_j2_Link: geometry collision mesh filename=package://frcobot_description/meshes/fr5v6/collision/j2_Lin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 scale=1 1 1; visual mesh filename=package://frcobot_description/meshes/fr5v6/visual/j2_Link.D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 scale=1 1 1
- link fr5v6_j3_Link: geometry collision mesh filename=package://frcobot_description/meshes/fr5v6/collision/j3_Lin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 scale=1 1 1; visual mesh filename=package://frcobot_description/meshes/fr5v6/visual/j3_Link.D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 scale=1 1 1
- link fr5v6_j4_Link: geometry collision mesh filename=package://frcobot_description/meshes/fr5v6/collision/j4_Lin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 scale=1 1 1; visual mesh filename=package://frcobot_description/meshes/fr5v6/visual/j4_Link.D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 scale=1 1 1
- link fr5v6_j5_Link: geometry collision mesh filename=package://frcobot_description/meshes/fr5v6/collision/j5_Lin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 scale=1 1 1; visual mesh filename=package://frcobot_description/meshes/fr5v6/visual/j5_Link.D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 scale=1 1 1
- link fr5v6_j6_Link: geometry collision mesh filename=package://frcobot_description/meshes/fr5v6/collision/j6_Lin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 scale=1 1 1; visual mesh filename=package://frcobot_description/meshes/fr5v6/visual/j6_Link.D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 scale=1 1 1
- link fr5v6_plant_link: geometry collision mesh filename=package://frcobot_description/meshes/fr5v6/collision/plant_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 scale=1 1 1; visual mesh filename=package://frcobot_description/meshes/fr5v6/visual/plant_lin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 scale=1 1 1
Joints:
- added joint fr5v6_tool: type fixed, parent fr5v6_j6_Link, child fr5v6_tool_Link, origin xyz=0 0 0.1 rpy=0 0 0, axis 0 0 1, limit lower=0 upper=0 effort=0 velocity=0
- added joint fr5v6_tool_tcp_joint: type fixed, parent fr5v6_tool_Link, child fr5v6_tool_tcp_link, origin xyz=0 0 0.25 rpy=0 0 0

File: catkin_ws/src/frcobot_description/urdf/fr5v6_library.xacro (robot description, xacro)
@@ -14,5 +14,5 @@
         <xacro:property name="material_name" value="" />
         <xacro:macro name="link_with_inertial"
-            params="name xyz rpy mass ixx ixy ixz iyy iyz izz visual_mesh collision_mesh">
+            params="name xyz rpy mass ixx ixy ixz iyy iyz izz visual_mesh collision_mesh scale:='1 1 1'">
             <link name="${name}">
                 <inertial>
@@ -25,5 +25,5 @@
                     <origin xyz="0 0 0" rpy="0 0 0" />
                     <geometry>
-                        <mesh filename="${visual_mesh}" />
+                        <mesh filename="${visual_mesh}" scale="${scale}"/>
                     </geometry>
                     <material name="${material_name}">
@@ -34,5 +34,5 @@
                     <origin xyz="0 0 0" rpy="0 0 0" />
                     <geometry>
-                        <mesh filename="${collision_mesh}" />
+                        <mesh filename="${collision_mesh}" scale="${scale}"/>
                     </geometry>
                 </collision>
@@ -59,10 +59,10 @@
             rpy="0 0 0"
             mass="0.40503"
-        ixx="0.0008273"
-        ixy="-2.5374E-19"
-        ixz="1.6905E-22"
-        iyy="0.0008273"
-        iyz="-2.1817E-22"
-        izz="0.0016373"
+            ixx="0.0008273"
+            ixy="-2.5374E-19"
+            ixz="1.6905E-22"
+            iyy="0.0008273"
+            iyz="-2.1817E-22"
+            izz="0.0016373"
             visual_mesh="package://frcobot_description/meshes/fr5v6/visual/plant_link.DAE"
             collision_mesh="package://frcobot_description/meshes/fr5v6/collision/plant_link.STL" />
@@ -187,22 +187,53 @@
                 k_velocity="10" />
         </joint>
+        <!-- Uncomment and modify the following section if you have a tool link -->
+        <xacro:link_with_inertial name="${arm_id}_tool_Link" xyz="0.24412 0.079181 -0.126"
+            rpy="0 0 0"
+            mass="0"
+            ixx="0.10666" ixy="-0.046059" ixz="0.046354" iyy="0.87967" iyz="0.0095222" izz="0.85231"
+            visual_mesh="package://frcobot_description/meshes/fr5v6/visual/toolA-250mm.DAE"
+            collision_mesh="package://frcobot_description/meshes/fr5v6/collision/toolA-250mm.STL"
+            scale="0.001 0.001 0.001" />
+        <joint name="${arm_id}_tool" type="fixed">
+            <origin xyz="0 0 0.1" rpy="0 0 0" />
+            <parent link="${arm_id}_j6_Link" />
+            <child link="${arm_id}_tool_Link" />
+            <axis xyz="0 0 1" />
+            <limit lower="0" upper="0" effort="0" velocity="0" />
+            <calibration rising="0" falling="0" />
+            <dynamics damping="0" friction="0" />
+            <safety_controller soft_lower_limit="0" soft_upper_limit="0" k_position="0"
+                k_velocity="0" />
+        </joint>
+        <!-- 添加工具末端TCP坐标系（使用基本几何体） -->
+        <link name="${arm_id}_tool_tcp_link">
+            <inertial>
+                <origin xyz="0 0 0" rpy="0 0 0" />
+                <mass value="0.001" />
+                <inertia ixx="0.0000001" ixy="0" ixz="0" iyy="0.0000001" iyz="0" izz="0.0000001" />
+            </inertial>
+            <visual>
+                <origin xyz="0 0 0" rpy="0 0 0" />
+                <geometry>
+                    <sphere radius="0.005"/>
+                </geometry>
+                <material name="">
+                    <color rgba="1 0 0 1" />
+                </material>
+            </visual>
+            <!-- 添加碰撞几何体 -->
+            <collision>
+                <origin xyz="0 0 0" rpy="0 0 0" />
+                <geometry>
+                    <sphere radius="0.005"/>
+                </geometry>
+            </collision>
+        </link>
+        <joint name="${arm_id}_tool_tcp_joint" type="fixed">
+            <origin xyz="0 0 0.25" rpy="0 0 0" />
+            <parent link="${arm_id}_tool_Link" />
+            <child link="${arm_id}_tool_tcp_link" />
+        </joint>
     </xacro:macro>
-    <!-- Uncomment and modify the following section if you have a tool link -->
-    <!--
-  <xacro:link_with_inertial name="tool_Link" xyz="0.24412 0.079181 -0.126" rpy="0 0 0" mass="0"
-                            ixx="0.10666" ixy="-0.046059" ixz="0.046354" iyy="0.87967" iyz="0.0095222" izz="0.85231"
-                            visual_mesh="package://frcobot_description/meshes/fr5v6/visual/tool_Link.STL"
-                            collision_mesh="package://frcobot_description/meshes/fr5v6/collision/tool_Link.STL"/>
-  <joint name="tool" type="fixed">
-    <origin xyz="0 0 0.1" rpy="0 0 0"/>
-    <parent link="j6_Link"/>
-    <child link="tool_Link"/>
-    <axis xyz="0 0 1"/>
-    <limit lower="0" upper="0" effort="0" velocity="0"/>
-    <calibration rising="0" falling="0"/>
-    <dynamics damping="0" friction="0"/>
-    <safety_controller soft_lower_limit="0" soft_upper_limit="0" k_position="0" k_velocity="0"/>
-  </joint>
-  -->
     <xacro:macro name="gazebo-joint" params="joint ">
         <transmission name="trans_${joint}">

Commit message: 20250303 修改Link为link

File: catkin_ws/src/fr5v6_single_moveit_config/config/gazebo_fr5v6_single_arm.urdf (robot description, URDF)
Before this commit: robot fr5v6_single_arm, 12 links, 11 joints
Links:
- removed link fr5v6_j1_Link
- removed link fr5v6_j2_Link
- removed link fr5v6_j3_Link
- removed link fr5v6_j4_Link
- removed link fr5v6_j5_Link
- removed link fr5v6_j6_Link
- removed link fr5v6_tool_Link
- added link fr5v6_j1_link, mass 4.3771; collision mesh filename=package://frcobot_description/meshes/fr5v6/collision/j1_lin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 scale=1 1 1; visual mesh filename=package://frcobot_description/meshes/fr5v6/visual/j1_link.D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 scale=1 1 1
- added link fr5v6_j2_link, mass 14.458; collision mesh filename=package://frcobot_description/meshes/fr5v6/collision/j2_lin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 scale=1 1 1; visual mesh filename=package://frcobot_description/meshes/fr5v6/visual/j2_link.D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 scale=1 1 1
- added link fr5v6_j3_link, mass 7.6737; collision mesh filename=package://frcobot_description/meshes/fr5v6/collision/j3_lin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 scale=1 1 1; visual mesh filename=package://frcobot_description/meshes/fr5v6/visual/j3_link.D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 scale=1 1 1
- added link fr5v6_j4_link, mass 1.6266; collision mesh filename=package://frcobot_description/meshes/fr5v6/collision/j4_lin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 scale=1 1 1; visual mesh filename=package://frcobot_description/meshes/fr5v6/visual/j4_link.D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 scale=1 1 1
- added link fr5v6_j5_link, mass 1.5812; collision mesh filename=package://frcobot_description/meshes/fr5v6/collision/j5_lin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 scale=1 1 1; visual mesh filename=package://frcobot_description/meshes/fr5v6/visual/j5_link.D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 scale=1 1 1
- added link fr5v6_j6_link, mass 0.52542; collision mesh filename=package://frcobot_description/meshes/fr5v6/collision/j6_lin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 scale=1 1 1; visual mesh filename=package://frcobot_description/meshes/fr5v6/visual/j6_link.D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 scale=1 1 1
- added link fr5v6_tool_link, mass 0; collision mesh filename=package://frcobot_description/meshes/fr5v6/collision/toolA-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 scale=0.001 0.001 0.001; visual mesh filename=package://frcobot_description/meshes/fr5v6/visual/toolA-250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 scale=0.001 0.001 0.001
- link fr5v6_tool_tcp_link: geometry collision sphere radius=0.005; visual sphere radius=0.005
Joints:
- joint fr5v6_j1: child fr5v6_j1_Link -> fr5v6_j1_link
- joint fr5v6_j2: child fr5v6_j2_Link -> fr5v6_j2_link; parent fr5v6_j1_Link -> fr5v6_j1_link
- joint fr5v6_j3: child fr5v6_j3_Link -> fr5v6_j3_link; parent fr5v6_j2_Link -> fr5v6_j2_link
- joint fr5v6_j4: child fr5v6_j4_Link -> fr5v6_j4_link; parent fr5v6_j3_Link -> fr5v6_j3_link
- joint fr5v6_j5: child fr5v6_j5_Link -> fr5v6_j5_link; parent fr5v6_j4_Link -> fr5v6_j4_link
- joint fr5v6_j6: child fr5v6_j6_Link -> fr5v6_j6_link; parent fr5v6_j5_Link -> fr5v6_j5_link
- joint fr5v6_tool: child fr5v6_tool_Link -> fr5v6_tool_link; parent fr5v6_j6_Link -> fr5v6_j6_link
- joint fr5v6_tool_tcp_joint: parent fr5v6_tool_Link -> fr5v6_tool_link

File: catkin_ws/src/frcobot_description/urdf/fr5v6_gazebo.urdf (robot description, URDF)
Before this commit: robot fr5v6, 8 links, 7 joints
Links:
- removed link j1_Link
- removed link j2_Link
- removed link j3_Link
- removed link j4_Link
- removed link j5_Link
- removed link j6_Link
- added link j1_link, mass 4.3771; collision mesh filename=package://frcobot_description/meshes/fr5v6/collision/j1_lin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; visual mesh filename=package://frcobot_description/meshes/fr5v6/visual/j1_link.D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
- added link j2_link, mass 14.458; collision mesh filename=package://frcobot_description/meshes/fr5v6/collision/j2_lin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; visual mesh filename=package://frcobot_description/meshes/fr5v6/visual/j2_link.D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
- added link j3_link, mass 7.6737; collision mesh filename=package://frcobot_description/meshes/fr5v6/collision/j3_lin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; visual mesh filename=package://frcobot_description/meshes/fr5v6/visual/j3_link.D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
- added link j4_link, mass 1.6266; collision mesh filename=package://frcobot_description/meshes/fr5v6/collision/j4_lin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; visual mesh filename=package://frcobot_description/meshes/fr5v6/visual/j4_link.D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
- added link j5_link, mass 1.5812; collision mesh filename=package://frcobot_description/meshes/fr5v6/collision/j5_lin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; visual mesh filename=package://frcobot_description/meshes/fr5v6/visual/j5_link.D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
- added link j6_link, mass 0.52542; collision mesh filename=package://frcobot_description/meshes/fr5v6/collision/j6_lin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; visual mesh filename=package://frcobot_description/meshes/fr5v6/visual/j6_link.D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
Joints:
- joint j1: child j1_Link -> j1_link
- joint j2: child j2_Link -> j2_link; parent j1_Link -> j1_link
- joint j3: child j3_Link -> j3_link; parent j2_Link -> j2_link
- joint j4: child j4_Link -> j4_link; parent j3_Link -> j3_link
- joint j5: child j5_Link -> j5_link; parent j4_Link -> j4_link
- joint j6: child j6_Link -> j6_link; parent j5_Link -> j5_link

File: catkin_ws/src/frcobot_description/urdf/fr5v6_library.xacro (robot description, xacro)
@@ -79,15 +79,15 @@
             visual_mesh="package://frcobot_description/meshes/fr5v6/visual/base_link.DAE"
             collision_mesh="package://frcobot_description/meshes/fr5v6/collision/base_link.STL" />
-        <xacro:link_with_inertial name="${arm_id}_j1_Link" xyz="5.0029E-07 -0.0040922 0.14629"
+        <xacro:link_with_inertial name="${arm_id}_j1_link" xyz="5.0029E-07 -0.0040922 0.14629"
             rpy="0 0 0"
             mass="4.3771"
             ixx="0.010731" ixy="-8.0587E-09" ixz="-3.6773E-08" iyy="0.010408" iyz="0.00012853"
             izz="0.0081793"
-            visual_mesh="package://frcobot_description/meshes/fr5v6/visual/j1_Link.DAE"
-            collision_mesh="package://frcobot_description/meshes/fr5v6/collision/j1_Link.STL" />
+            visual_mesh="package://frcobot_description/meshes/fr5v6/visual/j1_link.DAE"
+            collision_mesh="package://frcobot_description/meshes/fr5v6/collision/j1_link.STL" />
         <joint name="${arm_id}_j1" type="revolute">
             <origin xyz="0 0 0" rpy="0 0 0" />
             <parent link="${arm_id}_base_link" />
-            <child link="${arm_id}_j1_Link" />
+            <child link="${arm_id}_j1_link" />
             <axis xyz="0 0 1" />
             <limit lower="-3.0543" upper="3.0543" effort="150" velocity="3.15" />
@@ -97,15 +97,15 @@
                 k_velocity="10" />
         </joint>
-        <xacro:link_with_inertial name="${arm_id}_j2_Link" xyz="-0.2125 -5.7643E-09 0.1346"
+        <xacro:link_with_inertial name="${arm_id}_j2_link" xyz="-0.2125 -5.7643E-09 0.1346"
             rpy="0 0 0"
             mass="14.458"
             ixx="0.028392" ixy="-1.337E-07" ixz="-3.9895E-09" iyy="0.4559" iyz="4.214E-08"
             izz="0.44974"
-            visual_mesh="package://frcobot_description/meshes/fr5v6/visual/j2_Link.DAE"
-            collision_mesh="package://frcobot_description/meshes/fr5v6/collision/j2_Link.STL" />
+            visual_mesh="package://frcobot_description/meshes/fr5v6/visual/j2_link.DAE"
+            collision_mesh="package://frcobot_description/meshes/fr5v6/collision/j2_link.STL" />
         <joint name="${arm_id}_j2" type="revolute">
             <origin xyz="0 0 0.152" rpy="1.5708 0 0" />
-            <parent link="${arm_id}_j1_Link" />
-            <child link="${arm_id}_j2_Link" />
+            <parent link="${arm_id}_j1_link" />
+            <child link="${arm_id}_j2_link" />
             <axis xyz="0 0 1" />
             <limit lower="-4.6251" upper="1.4835" effort="150" velocity="3.15" />
@@ -115,15 +115,15 @@
                 k_velocity="10" />
         </joint>
-        <xacro:link_with_inertial name="${arm_id}_j3_Link" xyz="-0.18793 -8.4503E-07 0.0066357"
+        <xacro:link_with_inertial name="${arm_id}_j3_link" xyz="-0.18793 -8.4503E-07 0.0066357"
             rpy="0 0 0"
             mass="7.6737"
             ixx="0.0085096" ixy="2.1613E-06" ixz="-0.0068678" iyy="0.16971" iyz="3.7086E-08"
             izz="0.16854"
-            visual_mesh="package://frcobot_description/meshes/fr5v6/visual/j3_Link.DAE"
-            collision_mesh="package://frcobot_description/meshes/fr5v6/collision/j3_Link.STL" />
+            visual_mesh="package://frcobot_description/meshes/fr5v6/visual/j3_link.DAE"
+            collision_mesh="package://frcobot_description/meshes/fr5v6/collision/j3_link.STL" />
         <joint name="${arm_id}_j3" type="revolute">
             <origin xyz="-0.425 0 0" rpy="0 0 0" />
-            <parent link="${arm_id}_j2_Link" />
-            <child link="${arm_id}_j3_Link" />
+            <parent link="${arm_id}_j2_link" />
+            <child link="${arm_id}_j3_link" />
             <axis xyz="0 0 1" />
             <limit lower="-2.8274" upper="2.8274" effort="150" velocity="3.15" />
@@ -133,15 +133,15 @@
                 k_velocity="10" />
         </joint>
-        <xacro:link_with_inertial name="${arm_id}_j4_Link" xyz="4.98E-07 -0.003754 0.097155"
+        <xacro:link_with_inertial name="${arm_id}_j4_link" xyz="4.98E-07 -0.003754 0.097155"
             rpy="0 0 0"
             mass="1.6266"
             ixx="0.00216" ixy="4.888E-09" ixz="3.1528E-08" iyy="0.0015455" iyz="3.7678E-05"
             izz="0.0019902"
-            visual_mesh="package://frcobot_description/meshes/fr5v6/visual/j4_Link.DAE"
-            collision_mesh="package://frcobot_description/meshes/fr5v6/collision/j4_Link.STL" />
+            visual_mesh="package://frcobot_description/meshes/fr5v6/visual/j4_link.DAE"
+            collision_mesh="package://frcobot_description/meshes/fr5v6/collision/j4_link.STL" />
         <joint name="${arm_id}_j4" type="revolute">
             <origin xyz="-0.39501 0 0" rpy="0 0 0" />
-            <parent link="${arm_id}_j3_Link" />
-            <child link="${arm_id}_j4_Link" />
+            <parent link="${arm_id}_j3_link" />
+            <child link="${arm_id}_j4_link" />
             <axis xyz="0 0 1" />
             <limit lower="-4.6251" upper="1.4835" effort="28" velocity="3.2" />
@@ -151,15 +151,15 @@
                 k_velocity="10" />
         </joint>
-        <xacro:link_with_inertial name="${arm_id}_j5_Link" xyz="-4.5588E-07 0.0038617 0.098257"
+        <xacro:link_with_inertial name="${arm_id}_j5_link" xyz="-4.5588E-07 0.0038617 0.098257"
             rpy="0 0 0"
             mass="1.5812"
             ixx="0.0020612" ixy="8.7064E-09" ixz="-3.4742E-08" iyy="0.0014477" iyz="-2.8534E-05"
             izz="0.0019573"
-            visual_mesh="package://frcobot_description/meshes/fr5v6/visual/j5_Link.DAE"
-            collision_mesh="package://frcobot_description/meshes/fr5v6/collision/j5_Link.STL" />
+            visual_mesh="package://frcobot_description/meshes/fr5v6/visual/j5_link.DAE"
+            collision_mesh="package://frcobot_description/meshes/fr5v6/collision/j5_link.STL" />
         <joint name="${arm_id}_j5" type="revolute">
             <origin xyz="0 0 0.1021" rpy="1.5708 0 0" />
-            <parent link="${arm_id}_j4_Link" />
-            <child link="${arm_id}_j5_Link" />
+            <parent link="${arm_id}_j4_link" />
+            <child link="${arm_id}_j5_link" />
             <axis xyz="0 0 1" />
             <limit lower="-3.0543" upper="3.0543" effort="28" velocity="3.2" />
@@ -169,15 +169,15 @@
                 k_velocity="10" />
         </joint>
-        <xacro:link_with_inertial name="${arm_id}_j6_Link" xyz="7.7496E-05 1.7751E-05 0.076122"
+        <xacro:link_with_inertial name="${arm_id}_j6_link" xyz="7.7496E-05 1.7751E-05 0.076122"
             rpy="0 0 0"
             mass="0.52542"
             ixx="0.00027721" ixy="-1.8677E-09" ixz="-1.188E-07" iyy="0.00027839" iyz="2.2607E-07"
             izz="0.00041605"
-            visual_mesh="package://frcobot_description/meshes/fr5v6/visual/j6_Link.DAE"
-            collision_mesh="package://frcobot_description/meshes/fr5v6/collision/j6_Link.STL" />
+            visual_mesh="package://frcobot_description/meshes/fr5v6/visual/j6_link.DAE"
+            collision_mesh="package://frcobot_description/meshes/fr5v6/collision/j6_link.STL" />
         <joint name="${arm_id}_j6" type="revolute">
             <origin xyz="0 0 0.102" rpy="-1.5708 0 0" />
-            <parent link="${arm_id}_j5_Link" />
-            <child link="${arm_id}_j6_Link" />
+            <parent link="${arm_id}_j5_link" />
+            <child link="${arm_id}_j6_link" />
             <axis xyz="0 0 1" />
             <limit lower="-3.0543" upper="3.0543" effort="28" velocity="3.2" />
@@ -188,5 +188,5 @@
         </joint>
         <!-- Uncomment and modify the following section if you have a tool link -->
-        <xacro:link_with_inertial name="${arm_id}_tool_Link" xyz="0.24412 0.079181 -0.126"
+        <xacro:link_with_inertial name="${arm_id}_tool_link" xyz="0.24412 0.079181 -0.126"
             rpy="0 0 0"
             mass="0"
@@ -197,6 +197,6 @@
         <joint name="${arm_id}_tool" type="fixed">
             <origin xyz="0 0 0.1" rpy="0 0 0" />
-            <parent link="${arm_id}_j6_Link" />
-            <child link="${arm_id}_tool_Link" />
+            <parent link="${arm_id}_j6_link" />
+            <child link="${arm_id}_tool_link" />
             <axis xyz="0 0 1" />
             <limit lower="0" upper="0" effort="0" velocity="0" />
@@ -232,5 +232,5 @@
         <joint name="${arm_id}_tool_tcp_joint" type="fixed">
             <origin xyz="0 0 0.25" rpy="0 0 0" />
-            <parent link="${arm_id}_tool_Link" />
+            <parent link="${arm_id}_tool_link" />
             <child link="${arm_id}_tool_tcp_link" />
         </joint>

Commit message: 20250319 修复gazebo仿真机械臂底座移动问题

File: catkin_ws/src/fr5v6_single_moveit_config/config/gazebo_fr5v6_single_arm.urdf (robot description, URDF)
Before this commit: robot fr5v6_single_arm, 12 links, 11 joints
Links:
- removed link robot_base
- added link world
- link frrobot_base0_link: mass 6.8715 -> 50.058
- link frrobot_base1_link: mass 0.40503 -> 3.1592
Joints:
- joint frrobot_base0_to_base1: origin xyz=-0.00031408 0.00046097 0.41799 rpy=0 0 0 -> xyz=0 0 0.487 rpy=0 0 0
- joint frrobot_joint_base: parent robot_base -> world

File: catkin_ws/src/frcobot_description/urdf/fr5v6_single_arm.xacro (robot description, xacro)
@@ -6,7 +6,7 @@
     <xacro:include filename="$(find frcobot_description)/urdf/fr5v6_library.xacro" />
     <!-- 添加虚拟根链接 -->
-    <link name="robot_base" />
+    <link name="world" />
     <!-- 实例化机械臂 -->
-    <xacro:fr5v6_arm arm_id="$(arg arm_id)" connected_to="robot_base" xyz="0 0 0" rpy="0 0 0" />
+    <xacro:fr5v6_arm arm_id="$(arg arm_id)" connected_to="world" xyz="0 0 0" rpy="0 0 0" />
     <xacro:gazebo-joint joint="$(arg arm_id)_j1" />
     <xacro:gazebo-joint joint="$(arg arm_id)_j2" />

Commit message: 20250402 修复moveit配置，删除tool

File: catkin_ws/src/fr5v6_single_moveit_config/config/gazebo_fr5v6_single_arm.urdf (robot description, URDF)
Before this commit: robot fr5v6_single_arm, 12 links, 11 joints
Links:
- removed link frrobot_tool_tcp_link
- link frrobot_tool_link: mass 0.05 -> 0.1; geometry 
Joints:
- removed joint frrobot_tcp_joint
- joint frrobot_tool_joint: axis 0 0 1 -> (none); limit lower=0 upper=0 effort=0 velocity=0 -> (none)
