Commit message: feat: 添加工具包管理系统
- 创建frcobot_tools包，支持模块化工具管理
- 支持simple和urdf_package两种工具类型
- 添加工具加载器(tool_loader.xacro)支持从工具包加载
- 修改fr5v6_library.xacro支持工具包系统
- 更新single_arm和dual_arms xacro文件支持工具参数
- 添加工具包模板和示例工具(tool_none, tool_250mm)
- 添加permanent_magnet工具包示例
- 保持向后兼容，仍支持旧的tools.yaml配置方式
- 添加工具管理脚本(list_tools.py等)

File: catkin_ws/src/frcobot_description/urdf/fr5v6_dual_arms.xacro (robot description, xacro)
@@ -10,7 +10,4 @@
     <xacro:property name="calibration_file" value="$(find frcobot_description)/config/dual_arm_calibration.yaml"/>
     <xacro:property name="calib" value="${xacro.load_yaml(calibration_file)}"/>
-    <!-- 加载工具配置文件 -->
-    <xacro:property name="tools_config" value="$(find frcobot_description)/config/tools.yaml"/>
-    <xacro:property name="tools" value="${xacro.load_yaml(tools_config)}"/>
     <!-- 获取标定参数 -->
     <xacro:property name="trans_x" value="${calib['left_to_right_transform']['translation']['x']}"/>
@@ -20,7 +17,36 @@
     <xacro:property name="pitch" value="${calib['left_to_right_transform']['rpy']['pitch']}"/>
     <xacro:property name="yaw" value="${calib['left_to_right_transform']['rpy']['yaw']}"/>
-    <!-- 获取工具配置 -->
-    <xacro:property name="robot1_tool_config" value="${tools['tools']['$(arg robot1_tool)']}"/>
-    <xacro:property name="robot2_tool_config" value="${tools['tools']['$(arg robot2_tool)']}"/>
+    <!-- 加载工具配置 -->
+    <!-- 优先从工具包加载，如果工具包不存在则从旧的tools.yaml加载 -->
+    <!-- 注意：如果工具包不存在，xacro会报错，此时需要确保旧的tools.yaml中有对应配置 -->
+    <!-- 获取robot1工具配置 -->
+    <!-- 首先尝试从工具包加载 -->
+    <xacro:property name="robot1_tool_package_path"
+                    value="$(find frcobot_tools)/tools/$(arg robot1_tool)/config/tool.yaml"/>
+    <xacro:property name="robot1_tool_config" value="${None}"/>
+    <!-- 尝试加载工具包配置 -->
+    <!-- 如果工具包存在，使用工具包配置；否则需要在下面取消注释使用旧配置 -->
+    <xacro:property name="robot1_tool_package_config"
+                    value="${xacro.load_yaml(robot1_tool_package_path)}"/>
+    <xacro:property name="robot1_tool_config" value="${robot1_tool_package_config}"/>
+    <!-- 如果工具包不存在，取消下面注释使用旧配置 -->
+    <!--
+    <xacro:property name="old_tools_config" value="$(find frcobot_description)/config/tools.yaml"/>
+    <xacro:property name="old_tools" value="${xacro.load_yaml(old_tools_config)}"/>
+    <xacro:property name="robot1_tool_config" value="${old_tools['tools']['$(arg robot1_tool)']}"/>
+    -->
+    <!-- 获取robot2工具配置 -->
+    <xacro:property name="robot2_tool_package_path"
+                    value="$(find frcobot_tools)/tools/$(arg robot2_tool)/config/tool.yaml"/>
+    <xacro:property name="robot2_tool_config" value="${None}"/>
+    <xacro:property name="robot2_tool_package_config"
+                    value="${xacro.load_yaml(robot2_tool_package_path)}"/>
+    <xacro:property name="robot2_tool_config" value="${robot2_tool_package_config}"/>
+    <!-- 如果工具包不存在，取消下面注释使用旧配置 -->
+    <!--
+    <xacro:property name="old_tools_config" value="$(find frcobot_description)/config/tools.yaml"/>
+    <xacro:property name="old_tools" value="${xacro.load_yaml(old_tools_config)}"/>
+    <xacro:property name="robot2_tool_config" value="${old_tools['tools']['$(arg robot2_tool)']}"/>
+    -->
     <!-- 添加虚拟根链接 -->
     <xacro:include filename="$(find frcobot_description)/urdf/fr5v6_library.xacro" />

File: catkin_ws/src/frcobot_description/urdf/fr5v6_library.xacro (robot description, xacro)
@@ -194,84 +194,95 @@
                 k_velocity="10" />
         </joint>
-        <!-- 添加工具链接 - 始终创建 -->
-        <link name="${arm_id}_tool_link">
+        <!-- 加载工具加载器 -->
+        <xacro:include filename="$(find frcobot_description)/urdf/tool_loader.xacro" />
+        <!-- 检查是否使用工具包系统 -->
+        <xacro:property name="use_tool_package" value="${'tool_type' in tool_config}"/>
+        <!-- 如果使用工具包系统，使用新的工具加载器 -->
+        <xacro:if value="${use_tool_package and tool_name != 'none'}">
+            <xacro:load_tool arm_id="${arm_id}" tool_name="${tool_name}" tool_config="${tool_config}"/>
+        </xacro:if>
+        <!-- 否则使用旧的工具配置方式（向后兼容） -->
+        <xacro:unless value="${use_tool_package}">
+            <!-- 添加工具链接 - 始终创建 -->
+            <link name="${arm_id}_tool_link">
+                <xacro:if value="${tool_name != 'none'}">
+                    <visual>
+                        <origin
+                            xyz="${tool_config['origin']['xyz'][0]}
+                                ${tool_config['origin']['xyz'][1]}
+                                ${tool_config['origin']['xyz'][2]}"
+                            rpy="${tool_config['origin']['rpy'][0]}
+                                ${tool_config['origin']['rpy'][1]}
+                                ${tool_config['origin']['rpy'][2]}" />
+                        <geometry>
+                            <mesh filename="${tool_config['mesh_path']}" scale="0.001 0.001 0.001" />
+                        </geometry>
+                    </visual>
+                    <collision>
+                        <origin
+                            xyz="${tool_config['origin']['xyz'][0]}
+                                ${tool_config['origin']['xyz'][1]}
+                                ${tool_config['origin']['xyz'][2]}"
+                            rpy="${tool_config['origin']['rpy'][0]}
+                                ${tool_config['origin']['rpy'][1]}
+                                ${tool_config['origin']['rpy'][2]}" />
+                        <geometry>
+                            <mesh filename="${tool_config['collision_mesh']}" scale="0.001 0.001 0.001" />
+                        </geometry>
+                    </collision>
+                </xacro:if>
+                <inertial>
+                    <origin xyz="0 0 0" rpy="0 0 0"/>
+                    <xacro:if value="${tool_name == 'none'}">
+                        <mass value="0.1" />
+                        <inertia
+                            ixx="0.1" ixy="0.0" ixz="0.0"
+                            iyy="0.1" iyz="0.0" izz="0.1" />
+                    </xacro:if>
+                    <xacro:unless value="${tool_name == 'none'}">
+                        <mass value="${tool_config['mass']}" />
+                        <inertia
+                            ixx="${tool_config['inertia']['ixx']}"
+                            ixy="${tool_config['inertia']['ixy']}"
+                            ixz="${tool_config['inertia']['ixz']}"
+                            iyy="${tool_config['inertia']['iyy']}"
+                            iyz="${tool_config['inertia']['iyz']}"
+                            izz="${tool_config['inertia']['izz']}" />
+                    </xacro:unless>
+                </inertial>
+            </link>
+            <!-- 总是创建工具关节 -->
+            <joint name="${arm_id}_tool_joint" type="fixed">
+                <parent link="${arm_id}_j6_link" />
+                <child link="${arm_id}_tool_link" />
+                <!-- 先应用固定的法兰偏移 -->
+                <origin xyz="0 0 0.1" rpy="0 0 0" />
+            </joint>
+            <!-- 只在有tool时创建TCP链接和关节 -->
             <xacro:if value="${tool_name != 'none'}">
-                <visual>
+                <link name="${arm_id}_tcp_link">
+                    <visual>
+                        <origin xyz="0 0 0" rpy="0 0 0" />
+                        <geometry>
+                            <sphere radius="0.005" />
+                        </geometry>
+                        <material name="">
+                            <color rgba="1 0 0 1" />
+                        </material>
+                    </visual>
+                </link>
+                <joint name="${arm_id}_tcp_joint" type="fixed">
+                    <parent link="${arm_id}_tool_link" />
+                    <child link="${arm_id}_tcp_link" />
                     <origin
-                        xyz="${tool_config['origin']['xyz'][0]}
-                            ${tool_config['origin']['xyz'][1]}
-                            ${tool_config['origin']['xyz'][2]}"
-                        rpy="${tool_config['origin']['rpy'][0]}
-                            ${tool_config['origin']['rpy'][1]}
-                            ${tool_config['origin']['rpy'][2]}" />
-                    <geometry>
-                        <mesh filename="${tool_config['mesh_path']}" scale="0.001 0.001 0.001" />
-                    </geometry>
-                </visual>
-                <collision>
-                    <origin
-                        xyz="${tool_config['origin']['xyz'][0]}
-                            ${tool_config['origin']['xyz'][1]}
-                            ${tool_config['origin']['xyz'][2]}"
-                        rpy="${tool_config['origin']['rpy'][0]}
-                            ${tool_config['origin']['rpy'][1]}
-                            ${tool_config['origin']['rpy'][2]}" />
-                    <geometry>
-                        <mesh filename="${tool_config['collision_mesh']}" scale="0.001 0.001 0.001" />
-                    </geometry>
-                </collision>
+                        xyz="${tool_config['tcp']['xyz'][0]}
+                            ${tool_config['tcp']['xyz'][1]}
+                            ${tool_config['tcp']['xyz'][2]}"
+                        rpy="${tool_config['tcp']['rpy'][0]}
+                            ${tool_config['tcp']['rpy'][1]}
+                            ${tool_config['tcp']['rpy'][2]}" />
+                </joint>
             </xacro:if>
-            <inertial>
-                <origin xyz="0 0 0" rpy="0 0 0"/>
-                <xacro:if value="${tool_name == 'none'}">
-                    <mass value="0.1" />
-                    <inertia
-                        ixx="0.1" ixy="0.0" ixz="0.0"
-                        iyy="0.1" iyz="0.0" izz="0.1" />
-                </xacro:if>
-                <xacro:unless value="${tool_name == 'none'}">
-                    <mass value="${tool_config['mass']}" />
-                    <inertia
-                        ixx="${tool_config['inertia']['ixx']}"
-                        ixy="${tool_config['inertia']['ixy']}"
-                        ixz="${tool_config['inertia']['ixz']}"
-                        iyy="${tool_config['inertia']['iyy']}"
-                        iyz="${tool_config['inertia']['iyz']}"
-                        izz="${tool_config['inertia']['izz']}" />
-                </xacro:unless>
-            </inertial>
-        </link>
-        <!-- 总是创建工具关节 -->
-        <joint name="${arm_id}_tool_joint" type="fixed">
-            <parent link="${arm_id}_j6_link" />
-            <child link="${arm_id}_tool_link" />
-            <!-- 先应用固定的法兰偏移 -->
-            <origin xyz="0 0 0.1" rpy="0 0 0" />
-        </joint>
-        <!-- 只在有tool时创建TCP链接和关节 -->
-        <xacro:if value="${tool_name != 'none'}">
-            <link name="${arm_id}_tcp_link">
-                <visual>
-                    <origin xyz="0 0 0" rpy="0 0 0" />
-                    <geometry>
-                        <sphere radius="0.005" />
-                    </geometry>
-                    <material name="">
-                        <color rgba="1 0 0 1" />
-                    </material>
-                </visual>
-            </link>
-            <joint name="${arm_id}_tcp_joint" type="fixed">
-                <parent link="${arm_id}_tool_link" />
-                <child link="${arm_id}_tcp_link" />
-                <origin
-                    xyz="${tool_config['tcp']['xyz'][0]}
-                        ${tool_config['tcp']['xyz'][1]}
-                        ${tool_config['tcp']['xyz'][2]}"
-                    rpy="${tool_config['tcp']['rpy'][0]}
-                        ${tool_config['tcp']['rpy'][1]}
-                        ${tool_config['tcp']['rpy'][2]}" />
-            </joint>
-        </xacro:if>
+        </xacro:unless>
     </xacro:macro>
     <xacro:macro name="gazebo-joint" params="joint ">

File: catkin_ws/src/frcobot_description/urdf/fr5v6_single_arm.xacro (robot description, xacro)
@@ -3,4 +3,22 @@
     <!-- 定义参数 -->
     <xacro:arg name="arm_id" default="frrobot" />
+    <!-- 定义工具参数 -->
+    <xacro:arg name="tool_name" default="none"/>
+    <!-- 加载工具配置 -->
+    <!-- 优先从工具包加载，如果工具包不存在则从旧的tools.yaml加载 -->
+    <xacro:property name="tool_package_path"
+                    value="$(find frcobot_tools)/tools/$(arg tool_name)/config/tool.yaml"/>
+    <xacro:property name="tool_config" value="${None}"/>
+    <!-- 尝试加载工具包配置 -->
+    <!-- 如果工具包存在，使用工具包配置；否则需要在下面取消注释使用旧配置 -->
+    <xacro:property name="tool_package_config"
+                    value="${xacro.load_yaml(tool_package_path)}"/>
+    <xacro:property name="tool_config" value="${tool_package_config}"/>
+    <!-- 如果工具包不存在，取消下面注释使用旧配置 -->
+    <!--
+    <xacro:property name="old_tools_config" value="$(find frcobot_description)/config/tools.yaml"/>
+    <xacro:property name="old_tools" value="${xacro.load_yaml(old_tools_config)}"/>
+    <xacro:property name="tool_config" value="${old_tools['tools']['$(arg tool_name)']}"/>
+    -->
     <!-- 添加虚拟根链接 -->
     <xacro:include filename="$(find frcobot_description)/urdf/fr5v6_library.xacro" />
@@ -8,5 +26,11 @@
     <link name="world" />
     <!-- 实例化机械臂 -->
-    <xacro:fr5v6_arm arm_id="$(arg arm_id)" connected_to="world" xyz="0 0 0" rpy="0 0 0" />
+    <xacro:fr5v6_arm
+        arm_id="$(arg arm_id)"
+        connected_to="world"
+        xyz="0 0 0"
+        rpy="0 0 0"
+        tool_name="$(arg tool_name)"
+        tool_config="${tool_config}" />
     <xacro:gazebo-joint joint="$(arg arm_id)_j1" />
     <xacro:gazebo-joint joint="$(arg arm_id)_j2" />
