Commit message: 20250222 完成单一机械臂xacro和urdf代码编写

File: catkin_ws/src/frcobot_description/urdf/fr5v6_library.xacro (robot description, xacro)
@@ -1,5 +1,6 @@
 <?xml version="1.0" encoding="utf-8"?>
 <robot name="fr5v6" xmlns:xacro="http://www.ros.org/wiki/xacro">
-    <xacro:macro name="fr5v6_arm" params="arm_id:='fr5v6' connected_to:='' xyz:='0 0 0' rpy:='0 0 0'">
+    <xacro:macro name="fr5v6_arm"
+        params="arm_id:='fr5v6' connected_to:='' xyz:='0 0 0' rpy:='0 0 0'">
         <xacro:unless value="${not connected_to}">
             <joint name="${arm_id}_joint_${connected_to}" type="fixed">
@@ -12,9 +13,4 @@
         <xacro:property name="color" value="0.89804 0.91765 0.92941 1" />
         <xacro:property name="material_name" value="" />
-        <!-- <link name="world" />
-        <joint name="world" type="fixed">
-            <parent link="world" />
-            <child link="base_link" />
-        </joint> -->
         <xacro:macro name="link_with_inertial"
             params="name xyz rpy mass ixx ixy ixz iyy iyz izz visual_mesh collision_mesh">

File: catkin_ws/src/frcobot_description/urdf/fr5v6_multiple_arms.xacro (robot description, xacro)
@@ -9,5 +9,5 @@
     <!-- <xacro:include filename="$(find franka_description)/robots/common/franka_arm.xacro" /> -->
     <!-- <xacro:include filename="$(find franka_description)/robots/common/franka_hand.xacro" /> -->
-    <xacro:include filename="$(find frcobot_description)/urdf/fr5v6.xacro" />
+    <xacro:include filename="$(find frcobot_description)/urdf/fr5v6_library.xacro" />
     <link name="world" />
     <!-- box shaped table as base for the 2 Pandas -->
@@ -53,6 +53,6 @@
     <!-- <xacro:franka_hand arm_id="$(arg arm_id_2)" rpy="0 0 ${-pi/4}"
         connected_to="$(arg arm_id_2)_link8" gazebo="true" safety_distance="0.03" /> -->
-        <xacro:fr5v6_arm arm_id="$(arg arm_id_1)" connected_to="base" xyz="0 -0.5 1" />
-        <xacro:fr5v6_arm arm_id="$(arg arm_id_2)" connected_to="base" xyz="0 0.5 1" />
+    <xacro:fr5v6_arm arm_id="$(arg arm_id_1)" connected_to="base" xyz="0 -0.5 1" />
+    <xacro:fr5v6_arm arm_id="$(arg arm_id_2)" connected_to="base" xyz="0 0.5 1" />
     <!-- right arm joints control interface -->
     <xacro:gazebo-joint joint="$(arg arm_id_1)_j1" />

Commit message: 20250222 配置moveit

File: catkin_ws/src/frcobot_description/urdf/fr5v6_library.xacro (robot description, xacro)
@@ -4,5 +4,5 @@
         params="arm_id:='fr5v6' connected_to:='' xyz:='0 0 0' rpy:='0 0 0'">
         <xacro:unless value="${not connected_to}">
-            <joint name="${arm_id}_joint_${connected_to}" type="fixed">
+            <joint name="${arm_id}_joint_base" type="fixed">
                 <parent link="${connected_to}" />
                 <child link="${arm_id}_base_link" />

File: catkin_ws/src/frcobot_description/urdf/fr5v6_single_arm.urdf (robot description, URDF)
Before this commit: robot fr5v6_single_arm, 8 links, 8 joints
Joints:
- removed joint fr5v6_joint_world
- removed joint world_joint
- added joint fr5v6_joint_base: type fixed, parent world, child fr5v6_base_link, origin xyz=0 0 0 rpy=0 0 0

File: catkin_ws/src/frcobot_description/urdf/fr5v6_single_arm.xacro (robot description, xacro)
@@ -7,10 +7,4 @@
     <!-- 添加虚拟根链接 -->
     <link name="world" />
-    <!-- 将实际的根链接连接到虚拟根链接 -->
-    <joint name="world_joint" type="fixed">
-        <parent link="world" />
-        <child link="${arm_id}_base_link" />
-        <origin xyz="0 0 0" rpy="0 0 0" />
-    </joint>
     <!-- 实例化机械臂 -->
     <xacro:fr5v6_arm arm_id="${arm_id}" connected_to="world" xyz="0 0 0" rpy="0 0 0" />

Commit message: 20250229 增加机械臂基座文件

File: catkin_ws/src/frcobot_description/urdf/fr5v6_library.xacro (robot description, xacro)
@@ -6,5 +6,5 @@
             <joint name="${arm_id}_joint_base" type="fixed">
                 <parent link="${connected_to}" />
-                <child link="${arm_id}_base_link" />
+                <child link="${arm_id}_extra_base_link" />
                 <origin rpy="${rpy}" xyz="${xyz}" />
             </joint>
@@ -39,4 +39,37 @@
             </link>
         </xacro:macro>
+        <xacro:link_with_inertial name="${arm_id}_extra_base_link"
+            xyz="-0.00035477 0.0011738 0.038422"
+            rpy="0 0 0"
+            mass="6.8715"
+            ixx="0.11261"
+            ixy="-2.8693E-05"
+            ixz="-0.0017586"
+            iyy="0.11265"
+            iyz="0.002588"
+            izz="0.19704"
+            visual_mesh="package://frcobot_description/meshes/fr5v6/visual/extra_base_link.DAE"
+            collision_mesh="package://frcobot_description/meshes/fr5v6/collision/extra_base_link.STL" />
+        <joint name="${arm_id}_extra_base_to_plant" type="fixed">
+            <parent link="${arm_id}_extra_base_link" />
+            <child link="${arm_id}_plant_link" />
+            <origin xyz="-0.00031408 0.00046097 0.41799" rpy="0 0 0" />
+        </joint>
+        <xacro:link_with_inertial name="${arm_id}_plant_link" xyz="2.7756E-16 0 -0.008"
+            rpy="0 0 0"
+            mass="0.40503"
+        ixx="0.0008273"
+        ixy="-2.5374E-19"
+        ixz="1.6905E-22"
+        iyy="0.0008273"
+        iyz="-2.1817E-22"
+        izz="0.0016373"
+            visual_mesh="package://frcobot_description/meshes/fr5v6/visual/plant_link.DAE"
+            collision_mesh="package://frcobot_description/meshes/fr5v6/collision/plant_link.STL" />
+        <joint name="${arm_id}_extra_plant_to_base" type="fixed">
+            <parent link="${arm_id}_plant_link" />
+            <child link="${arm_id}_base_link" />
+            <origin xyz="0 0 0.0001" rpy="0 0 0" />
+        </joint>
         <xacro:link_with_inertial name="${arm_id}_base_link" xyz="-0.00031896 -0.00029673 0.042463"
             rpy="0 0 0"

Commit message: 20250308 修复模型文件的一些BUG

File: catkin_ws/src/frcobot_description/urdf/fr5v6_library.xacro (robot description, xacro)
@@ -40,24 +40,25 @@
         </xacro:macro>
         <xacro:link_with_inertial name="${arm_id}_base0_link"
-            xyz="-0.00035477 0.0011738 0.038422"
-            rpy="0 0 0"
-            mass="60.8715"
-            ixx="0.11261"
-            ixy="-2.8693E-05"
-            ixz="-0.0017586"
-            iyy="0.11265"
-            iyz="0.002588"
-            izz="0.19704"
+            xyz="0.00022281 -3.2078E-06 0.11314"
+            rpy="0 0 0"
+            mass="50.058"
+            ixx="0.87603"
+            ixy="-2.9247E-05"
+            ixz="9.7148E-05"
+            iyy="0.87602"
+            iyz="-1.6883E-06"
+            izz="1.5353"
             visual_mesh="package://frcobot_description/meshes/fr5v6/visual/extra_base_link.DAE"
             collision_mesh="package://frcobot_description/meshes/fr5v6/collision/extra_base_link.STL" />
-        <xacro:link_with_inertial name="${arm_id}_base1_link" xyz="2.7756E-16 0 -0.008"
-            rpy="0 0 0"
-            mass="0.40503"
-            ixx="0.0008273"
-            ixy="-2.5374E-19"
-            ixz="1.6905E-22"
-            iyy="0.0008273"
-            iyz="-2.1817E-22"
-            izz="0.0016373"
+        <xacro:link_with_inertial name="${arm_id}_base1_link"
+            xyz="2.7756E-16 2.2204E-16 -0.008"
+            rpy="0 0 0"
+            mass="3.1592"
+            ixx="0.0064529"
+            ixy="-1.9807E-18"
+            ixz="1.3186E-21"
+            iyy="0.0064529"
+            iyz="-1.7017E-21"
+            izz="0.012771"
             visual_mesh="package://frcobot_description/meshes/fr5v6/visual/plant_link.DAE"
             collision_mesh="package://frcobot_description/meshes/fr5v6/collision/plant_link.STL" />
@@ -65,5 +66,5 @@
             <parent link="${arm_id}_base0_link" />
             <child link="${arm_id}_base1_link" />
-            <origin xyz="-0.00031408 0.00046097 0.41799" rpy="0 0 0" />
+            <origin xyz="0 0 0.487" rpy="0 0 0" />
         </joint>
         <xacro:link_with_inertial name="${arm_id}_base2_link" xyz="-0.00031896 -0.00029673 0.042463"

Commit message: 20250402 修改机械臂library，优化启动文件

File: catkin_ws/src/frcobot_description/urdf/fr5v6_library.xacro (robot description, xacro)
@@ -13,4 +13,10 @@
         <xacro:property name="color" value="0.89804 0.91765 0.92941 1" />
         <xacro:property name="material_name" value="" />
+        <xacro:if value="${tool_name == 'none'}">
+            <xacro:property name="tool_mass" value="0.1"/>
+        </xacro:if>
+        <xacro:unless value="${tool_name == 'none'}">
+            <xacro:property name="tool_mass" value="${tool_config['mass']}"/>
+        </xacro:unless>
         <xacro:macro name="link_with_inertial"
             params="name xyz rpy mass ixx ixy ixz iyy iyz izz visual_mesh collision_mesh scale:='1 1 1'">
@@ -218,12 +224,20 @@
             <inertial>
                 <origin xyz="0 0 0" rpy="0 0 0"/>
-                <mass value="${(tool_name == 'none') * 0.1 + (tool_name != 'none') * tool_config['mass']}" />
-                <inertia
-                    ixx="${(tool_name == 'none') * 0.1 + (tool_name != 'none') * tool_config['inertia']['ixx']}"
-                    ixy="${(tool_name == 'none') * 0.0 + (tool_name != 'none') * tool_config['inertia']['ixy']}"
-                    ixz="${(tool_name == 'none') * 0.0 + (tool_name != 'none') * tool_config['inertia']['ixz']}"
-                    iyy="${(tool_name == 'none') * 0.1 + (tool_name != 'none') * tool_config['inertia']['iyy']}"
-                    iyz="${(tool_name == 'none') * 0.0 + (tool_name != 'none') * tool_config['inertia']['iyz']}"
-                    izz="${(tool_name == 'none') * 0.1 + (tool_name != 'none') * tool_config['inertia']['izz']}" />
+                <xacro:if value="${tool_name == 'none'}">
+                    <mass value="0.1" />
+                    <inertia
+                        ixx="0.1" ixy="0.0" ixz="0.0"
+                        iyy="0.1" iyz="0.0" izz="0.1" />
+                </xacro:if>
+                <xacro:unless value="${tool_name == 'none'}">
+                    <mass value="${tool_config['mass']}" />
+                    <inertia
+                        ixx="${tool_config['inertia']['ixx']}"
+                        ixy="${tool_config['inertia']['ixy']}"
+                        ixz="${tool_config['inertia']['ixz']}"
+                        iyy="${tool_config['inertia']['iyy']}"
+                        iyz="${tool_config['inertia']['iyz']}"
+                        izz="${tool_config['inertia']['izz']}" />
+                </xacro:unless>
             </inertial>
         </link>

Commit message: 修改了末端工具连接的link为tool_link

File: catkin_ws/src/frcobot_description/urdf/fr5v6_library.xacro (robot description, xacro)
@@ -198,6 +198,24 @@
         <!-- 检查是否使用工具包系统 -->
         <xacro:property name="use_tool_package" value="${'tool_type' in tool_config}"/>
-        <!-- 如果使用工具包系统，使用新的工具加载器 -->
+        <!-- 如果使用工具包系统，先创建tool_link作为中间链接 -->
         <xacro:if value="${use_tool_package and tool_name != 'none'}">
+            <!-- 创建tool_link（连接到j6_link） -->
+            <link name="${arm_id}_tool_link">
+                <inertial>
+                    <origin xyz="0 0 0" rpy="0 0 0"/>
+                    <mass value="0.1" />
+                    <inertia
+                        ixx="0.1" ixy="0.0" ixz="0.0"
+                        iyy="0.1" iyz="0.0" izz="0.1" />
+                </inertial>
+            </link>
+            <!-- 创建从j6_link到tool_link的关节 -->
+            <joint name="${arm_id}_tool_joint" type="fixed">
+                <parent link="${arm_id}_j6_link" />
+                <child link="${arm_id}_tool_link" />
+                <!-- 先应用固定的法兰偏移 -->
+                <origin xyz="0 0 0.1" rpy="0 0 0" />
+            </joint>
+            <!-- 使用新的工具加载器，工具将连接到tool_link -->
             <xacro:load_tool arm_id="${arm_id}" tool_name="${tool_name}" tool_config="${tool_config}"/>
         </xacro:if>

File: catkin_ws/src/frcobot_description/urdf/tool_loader.xacro (robot description, xacro)
@@ -39,6 +39,6 @@
             <xacro:property name="collision_mesh_path" value="${tool_collision.get('mesh_path', '')}"/>
             <xacro:property name="collision_scale" value="${tool_collision.get('scale', [1,1,1])}"/>
-            <!-- 创建工具链接 -->
-            <link name="${arm_id}_tool_link">
+            <!-- 创建工具链接（使用工具名称作为链接名，避免与tool_link冲突） -->
+            <link name="${arm_id}_${tool_name}_link">
                 <!-- 可视化 -->
                 <xacro:if value="${visual_mesh_path}">
@@ -78,11 +78,12 @@
                 </inertial>
             </link>
-            <!-- 创建工具关节（连接到j6_link） -->
-            <joint name="${arm_id}_tool_joint" type="fixed">
-                <parent link="${arm_id}_j6_link" />
-                <child link="${arm_id}_tool_link" />
-                <!-- 先应用固定的法兰偏移（0.1m），然后加上工具偏移 -->
+            <!-- 创建工具关节（连接到tool_link，而不是j6_link） -->
+            <!-- 注意：tool_link已经在fr5v6_library.xacro中创建并连接到j6_link -->
+            <joint name="${arm_id}_${tool_name}_joint" type="fixed">
+                <parent link="${arm_id}_tool_link" />
+                <child link="${arm_id}_${tool_name}_link" />
+                <!-- 工具偏移（tool_link已经包含了0.1m的法兰偏移） -->
                 <origin
-                    xyz="${0.1 + tool_origin_xyz[0]} ${tool_origin_xyz[1]} ${tool_origin_xyz[2]}"
+                    xyz="${tool_origin_xyz[0]} ${tool_origin_xyz[1]} ${tool_origin_xyz[2]}"
                     rpy="${tool_origin_rpy[0]} ${tool_origin_rpy[1]} ${tool_origin_rpy[2]}" />
             </joint>
@@ -100,5 +101,5 @@
             </link>
             <joint name="${arm_id}_tcp_joint" type="fixed">
-                <parent link="${arm_id}_tool_link" />
+                <parent link="${arm_id}_${tool_name}_link" />
                 <child link="${arm_id}_tcp_link" />
                 <origin
@@ -115,17 +116,19 @@
             <xacro:property name="mount_offset" value="${urdf_config['mount_offset']}"/>
             <!-- 构建URDF文件路径 -->
-            <xacro:property name="tool_package_path" value="package://frcobot_tools/tools/${tool_name}"/>
+            <!-- 使用$(find)来解析package路径 -->
+            <xacro:property name="tool_package_path" value="$(find frcobot_tools)/tools/${tool_name}"/>
             <xacro:property name="full_urdf_path" value="${tool_package_path}/${urdf_file}"/>
             <!-- 加载外部URDF文件 -->
             <xacro:include filename="${full_urdf_path}"/>
-            <!-- 创建从j6_link到工具根链接的关节 -->
-            <joint name="${arm_id}_tool_joint" type="fixed">
-                <parent link="${arm_id}_j6_link" />
+            <!-- 创建从tool_link到工具根链接的关节（而不是j6_link） -->
+            <!-- 注意：tool_link已经在fr5v6_library.xacro中创建并连接到j6_link -->
+            <joint name="${arm_id}_${tool_name}_joint" type="fixed">
+                <parent link="${arm_id}_tool_link" />
                 <child link="${root_link_name}" />
-                <!-- 法兰偏移 + 工具安装偏移 -->
+                <!-- 工具安装偏移（tool_link已经包含了0.1m的法兰偏移） -->
                 <xacro:property name="mount_xyz" value="${mount_offset['xyz']}"/>
                 <xacro:property name="mount_rpy" value="${mount_offset['rpy']}"/>
                 <origin
-                    xyz="${0.1 + mount_xyz[0]} ${mount_xyz[1]} ${mount_xyz[2]}"
+                    xyz="${mount_xyz[0]} ${mount_xyz[1]} ${mount_xyz[2]}"
                     rpy="${mount_rpy[0]} ${mount_rpy[1]} ${mount_rpy[2]}" />
             </joint>

File: catkin_ws/src/frcobot_tools/tools/permanent_magnet/urdf/permanent_magnet.urdf (robot description, URDF)
Before this commit: robot permanent_magnet, 2 links, 1 joints
Links:
- removed link base_link
- removed link tcp_link
- added link pm_base_link, mass 0.136; collision mesh filename=package://permanent_magnet/meshes/pm_base_link.STL; visual mesh filename=package://permanent_magnet/meshes/pm_base_link.STL
- added link pm_tcp_link, mass 0.136; collision mesh filename=package://permanent_magnet/meshes/pm_tcp_link.STL; visual mesh filename=package://permanent_magnet/meshes/pm_tcp_link.STL
Joints:
- joint permanent_magnet: child tcp_link -> pm_tcp_link; parent base_link -> pm_base_link

Commit message: refactor: 更新工具配置加载逻辑，移除旧的tools.yaml支持
- 修改tool_config_loader.xacro和load_tool_config.py，工具配置现在仅从工具包加载
- 更新fr5v6_library.xacro，简化末端工具链接的创建逻辑
- 移除与旧配置的兼容性代码，确保系统使用新的工具包管理方式

File: catkin_ws/src/frcobot_description/urdf/fr5v6_library.xacro (robot description, xacro)
@@ -220,87 +220,21 @@
             <xacro:load_tool arm_id="${arm_id}" tool_name="${tool_name}" tool_config="${tool_config}"/>
         </xacro:if>
-        <!-- 否则使用旧的工具配置方式（向后兼容） -->
-        <xacro:unless value="${use_tool_package}">
-            <!-- 添加工具链接 - 始终创建 -->
+        <!-- 如果工具名称为none，创建空的ee_link -->
+        <xacro:if value="${tool_name == 'none'}">
             <link name="${arm_id}_ee_link">
-                <xacro:if value="${tool_name != 'none'}">
-                    <visual>
-                        <origin
-                            xyz="${tool_config['origin']['xyz'][0]}
-                                ${tool_config['origin']['xyz'][1]}
-                                ${tool_config['origin']['xyz'][2]}"
-                            rpy="${tool_config['origin']['rpy'][0]}
-                                ${tool_config['origin']['rpy'][1]}
-                                ${tool_config['origin']['rpy'][2]}" />
-                        <geometry>
-                            <mesh filename="${tool_config['mesh_path']}" scale="0.001 0.001 0.001" />
-                        </geometry>
-                    </visual>
-                    <collision>
-                        <origin
-                            xyz="${tool_config['origin']['xyz'][0]}
-                                ${tool_config['origin']['xyz'][1]}
-                                ${tool_config['origin']['xyz'][2]}"
-                            rpy="${tool_config['origin']['rpy'][0]}
-                                ${tool_config['origin']['rpy'][1]}
-                                ${tool_config['origin']['rpy'][2]}" />
-                        <geometry>
-                            <mesh filename="${tool_config['collision_mesh']}" scale="0.001 0.001 0.001" />
-                        </geometry>
-                    </collision>
-                </xacro:if>
                 <inertial>
                     <origin xyz="0 0 0" rpy="0 0 0"/>
-                    <xacro:if value="${tool_name == 'none'}">
-                        <mass value="0.1" />
-                        <inertia
-                            ixx="0.1" ixy="0.0" ixz="0.0"
-                            iyy="0.1" iyz="0.0" izz="0.1" />
-                    </xacro:if>
-                    <xacro:unless value="${tool_name == 'none'}">
-                        <mass value="${tool_config['mass']}" />
-                        <inertia
-                            ixx="${tool_config['inertia']['ixx']}"
-                            ixy="${tool_config['inertia']['ixy']}"
-                            ixz="${tool_config['inertia']['ixz']}"
-                            iyy="${tool_config['inertia']['iyy']}"
-                            iyz="${tool_config['inertia']['iyz']}"
-                            izz="${tool_config['inertia']['izz']}" />
-                    </xacro:unless>
+                    <mass value="0.1" />
+                    <inertia
+                        ixx="0.1" ixy="0.0" ixz="0.0"
+                        iyy="0.1" iyz="0.0" izz="0.1" />
                 </inertial>
             </link>
-            <!-- 总是创建工具关节 -->
             <joint name="${arm_id}_ee_joint" type="fixed">
                 <parent link="${arm_id}_j6_link" />
                 <child link="${arm_id}_ee_link" />
-                <!-- 先应用固定的法兰偏移 -->
                 <origin xyz="0 0 0.1" rpy="0 0 0" />
             </joint>
-            <!-- 只在有tool时创建TCP链接和关节 -->
-            <xacro:if value="${tool_name != 'none'}">
-                <link name="${arm_id}_tcp_link">
-                    <visual>
-                        <origin xyz="0 0 0" rpy="0 0 0" />
-                        <geometry>
-                            <sphere radius="0.005" />
-                        </geometry>
-                        <material name="">
-                            <color rgba="1 0 0 1" />
-                        </material>
-                    </visual>
-                </link>
-                <joint name="${arm_id}_tcp_joint" type="fixed">
-                    <parent link="${arm_id}_ee_link" />
-                    <child link="${arm_id}_tcp_link" />
-                    <origin
-                        xyz="${tool_config['tcp']['xyz'][0]}
-                            ${tool_config['tcp']['xyz'][1]}
-                            ${tool_config['tcp']['xyz'][2]}"
-                        rpy="${tool_config['tcp']['rpy'][0]}
-                            ${tool_config['tcp']['rpy'][1]}
-                            ${tool_config['tcp']['rpy'][2]}" />
-                </joint>
-            </xacro:if>
-        </xacro:unless>
+        </xacro:if>
     </xacro:macro>
     <xacro:macro name="gazebo-joint" params="joint ">

File: catkin_ws/src/frcobot_description/urdf/tool_config_loader.xacro (robot description, xacro)
@@ -2,5 +2,5 @@
 <!--
     工具配置加载器
-    优先从工具包加载配置，如果不存在则从旧的tools.yaml加载
+    从工具包加载配置
 -->
 <robot xmlns:xacro="http://www.ros.org/wiki/xacro">
@@ -13,10 +13,7 @@
     <xacro:macro name="load_tool_config" params="tool_name">
         <xacro:property name="tool_config_result" value="${None}"/>
-        <!-- 首先尝试从工具包加载 -->
+        <!-- 从工具包加载 -->
         <xacro:property name="tool_package_config_path"
                         value="$(find frcobot_tools)/tools/${tool_name}/config/tool.yaml"/>
-        <!-- 检查工具包配置文件是否存在 -->
-        <!-- 注意：xacro无法直接检查文件是否存在，所以我们先尝试加载 -->
-        <!-- 如果失败，会在下面的unless分支中处理 -->
         <xacro:try>
             <xacro:property name="tool_package_config"
@@ -26,12 +23,11 @@
         </xacro:try>
         <xacro:catch>
-            <!-- 如果工具包不存在，尝试从旧的tools.yaml加载 -->
-            <xacro:property name="old_tools_config_path"
-                            value="$(find frcobot_description)/config/tools.yaml"/>
-            <xacro:property name="old_tools_config"
-                            value="${xacro.load_yaml(old_tools_config_path)}"/>
-            <xacro:property name="tool_config_result"
-                            value="${old_tools_config['tools'][tool_name]}"/>
-            <xacro:property name="config_source" value="legacy"/>
+            <!-- 如果工具包不存在，返回空配置 -->
+            <xacro:property name="tool_config_result" value="{
+                'tool_type': 'simple',
+                'origin': {'xyz': [0,0,0], 'rpy': [0,0,0]},
+                'tcp': {'xyz': [0,0,0], 'rpy': [0,0,0]},
+                'physical_properties': {'mass': 0.1, 'inertia': {'ixx': 0.1, 'ixy': 0.0, 'ixz': 0.0, 'iyy': 0.1, 'iyz': 0.0, 'izz': 0.1}}
+            }"/>
         </xacro:catch>
         <!-- 如果工具名称为none，返回空配置 -->
