Commit message: 20250303 配置moveit基座

File: catkin_ws/src/fr5v6_dual_moveit_config/config/gazebo_fr5v6_dual_arms.urdf (robot description, URDF)
Before this commit: robot fr5v6_dual_arms, 16 links, 15 joints
Links:
- removed link base
- added link robot1_extra_base_link, mass 6.8715; collision mesh filename=package://frcobot_description/meshes/fr5v6/collision/extra_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; visual mesh filename=package://frcobot_description/meshes/fr5v6/visual/extra_bas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
- added link robot1_plant_link, mass 0.40503; collision mesh filename=package://frcobot_description/meshes/fr5v6/collision/plant_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; visual mesh filename=package://frcobot_description/meshes/fr5v6/visual/plant_lin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
- added link robot2_extra_base_link, mass 6.8715; collision mesh filename=package://frcobot_description/meshes/fr5v6/collision/extra_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; visual mesh filename=package://frcobot_description/meshes/fr5v6/visual/extra_bas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
- added link robot2_plant_link, mass 0.40503; collision mesh filename=package://frcobot_description/meshes/fr5v6/collision/plant_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; visual mesh filename=package://frcobot_description/meshes/fr5v6/visual/plant_lin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
Joints:
- removed joint base_to_world
- added joint robot1_extra_base_to_plant: type fixed, parent robot1_extra_base_link, child robot1_plant_link, origin xyz=-0.00031408 0.00046097 0.41799 rpy=0 0 0
- added joint robot1_extra_plant_to_base: type fixed, parent robot1_plant_link, child robot1_base_link, origin xyz=0 0 0.0001 rpy=0 0 0
- added joint robot2_extra_base_to_plant: type fixed, parent robot2_extra_base_link, child robot2_plant_link, origin xyz=-0.00031408 0.00046097 0.41799 rpy=0 0 0
- added joint robot2_extra_plant_to_base: type fixed, parent robot2_plant_link, child robot2_base_link, origin xyz=0 0 0.0001 rpy=0 0 0
- joint robot1_joint_base: child robot1_base_link -> robot1_extra_base_link; origin xyz=0 -0.5 1 rpy=0 0 0 -> xyz=0 -0.5 0 rpy=0 0 0; parent base -> world
- joint robot2_joint_base: child robot2_base_link -> robot2_extra_base_link; origin xyz=0 0.5 1 rpy=0 0 0 -> xyz=0 0.5 0 rpy=0 0 0; parent base -> world

File: catkin_ws/src/fr5v6_single_moveit_config/config/gazebo_fr5v6_single_arm.urdf (robot description, URDF)
Before this commit: robot fr5v6_single_arm, 8 links, 7 joints
Links:
- added link fr5v6_extra_base_link, mass 6.8715; collision mesh filename=package://frcobot_description/meshes/fr5v6/collision/extra_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; visual mesh filename=package://frcobot_description/meshes/fr5v6/visual/extra_bas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
- added link fr5v6_plant_link, mass 0.40503; collision mesh filename=package://frcobot_description/meshes/fr5v6/collision/plant_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; visual mesh filename=package://frcobot_description/meshes/fr5v6/visual/plant_lin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
Joints:
- added joint fr5v6_extra_base_to_plant: type fixed, parent fr5v6_extra_base_link, child fr5v6_plant_link, origin xyz=-0.00031408 0.00046097 0.41799 rpy=0 0 0
- added joint fr5v6_extra_plant_to_base: type fixed, parent fr5v6_plant_link, child fr5v6_base_link, origin xyz=0 0 0.0001 rpy=0 0 0
- joint fr5v6_joint_base: child fr5v6_base_link -> fr5v6_extra_base_link

File: catkin_ws/src/frcobot_description/urdf/fr5v6_dual_arms.xacro (robot description, xacro)
@@ -12,5 +12,5 @@
     <link name="world" />
     <!-- box shaped table as base for the 2 Pandas -->
-    <link name="base">
+    <!-- <link name="base">
         <visual>
             <origin xyz="0 0 0.5" rpy="0 0 0" />
@@ -33,10 +33,10 @@
             <inertia ixx="0.001" ixy="0.0" ixz="0.001" iyy="0.0" iyz="0.0" izz="0.001" />
         </inertial>
-    </link>
-    <joint name="base_to_world" type="fixed">
+    </link> -->
+    <!-- <joint name="base_to_world" type="fixed">
         <parent link="world" />
         <child link="base" />
         <origin xyz="0.0 0.0 0.0" rpy="0.0 0.0 0.0" />
-    </joint>
+    </joint> -->
     <!-- right arm with gripper -->
     <!-- <xacro:fr5v6_arm arm_id="$(arg arm_id_1)" connected_to="base" xyz="0 -0.5 1"
@@ -53,6 +53,6 @@
     <!-- <xacro:franka_hand arm_id="$(arg arm_id_2)" rpy="0 0 ${-pi/4}"
         connected_to="$(arg arm_id_2)_link8" gazebo="true" safety_distance="0.03" /> -->
-    <xacro:fr5v6_arm arm_id="$(arg arm_id_1)" connected_to="base" xyz="0 -0.5 1" />
-    <xacro:fr5v6_arm arm_id="$(arg arm_id_2)" connected_to="base" xyz="0 0.5 1" />
+    <xacro:fr5v6_arm arm_id="$(arg arm_id_1)" connected_to="world" xyz="0 -0.5 0" />
+    <xacro:fr5v6_arm arm_id="$(arg arm_id_2)" connected_to="world" xyz="0 0.5 0" />
     <!-- right arm joints control interface -->
     <xacro:gazebo-joint joint="$(arg arm_id_1)_j1" />
