Commit message: 20250308 修正实际机械臂的启动问题，重新配置moveit

File: catkin_ws/src/fr5v6_dual_moveit_config/config/gazebo_fr5v6_dual_arms.urdf (robot description, URDF)
Before this commit: robot fr5v6_dual_arms, 19 links, 18 joints
Links:
- removed link robot1_base_link
- removed link robot1_extra_base_link
- removed link robot1_j1_Link
- removed link robot1_j2_Link
- removed link robot1_j3_Link
- removed link robot1_j4_Link
- removed link robot1_j5_Link
- removed link robot1_j6_Link
- removed link robot1_plant_link
- removed link robot2_base_link
- removed link robot2_extra_base_link
- removed link robot2_j1_Link
- removed link robot2_j2_Link
- removed link robot2_j3_Link
- removed link robot2_j4_Link
- removed link robot2_j5_Link
- removed link robot2_j6_Link
- removed link robot2_plant_link
- added link robot1_base0_link, mass 6.8715; collision mesh filename=package://frcobot_description/meshes/fr5v6/collision/extra_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 scale=1 1 1; visual mesh filename=package://frcobot_description/meshes/fr5v6/visual/extra_bas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 scale=1 1 1
- added link robot1_base1_link, mass 0.40503; collision mesh filename=package://frcobot_description/meshes/fr5v6/collision/plant_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 scale=1 1 1; visual mesh filename=package://frcobot_description/meshes/fr5v6/visual/plant_lin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 scale=1 1 1
- added link robot1_base2_link, mass 1.6185; collision mesh filename=package://frcobot_description/meshes/fr5v6/collision/base_l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 scale=1 1 1; visual mesh filename=package://frcobot_description/meshes/fr5v6/visual/base_link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 scale=1 1 1
- added link robot1_j1_link, mass 4.3771; collision mesh filename=package://frcobot_description/meshes/fr5v6/collision/j1_lin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 scale=1 1 1; visual mesh filename=package://frcobot_description/meshes/fr5v6/visual/j1_link.D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 scale=1 1 1
- added link robot1_j2_link, mass 14.458; collision mesh filename=package://frcobot_description/meshes/fr5v6/collision/j2_lin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 scale=1 1 1; visual mesh filename=package://frcobot_description/meshes/fr5v6/visual/j2_link.D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 scale=1 1 1
- added link robot1_j3_link, mass 7.6737; collision mesh filename=package://frcobot_description/meshes/fr5v6/collision/j3_lin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 scale=1 1 1; visual mesh filename=package://frcobot_description/meshes/fr5v6/visual/j3_link.D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 scale=1 1 1
- added link robot1_j4_link, mass 1.6266; collision mesh filename=package://frcobot_description/meshes/fr5v6/collision/j4_lin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 scale=1 1 1; visual mesh filename=package://frcobot_description/meshes/fr5v6/visual/j4_link.D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 scale=1 1 1
- added link robot1_j5_link, mass 1.5812; collision mesh filename=package://frcobot_description/meshes/fr5v6/collision/j5_lin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 scale=1 1 1; visual mesh filename=package://frcobot_description/meshes/fr5v6/visual/j5_link.D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 scale=1 1 1
- added link robot1_j6_link, mass 0.52542; collision mesh filename=package://frcobot_description/meshes/fr5v6/collision/j6_lin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 scale=1 1 1; visual mesh filename=package://frcobot_description/meshes/fr5v6/visual/j6_link.D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 scale=1 1 1
- added link robot1_tool_link, mass 0.05; collision mesh filename=package://frcobot_description/meshes/fr5v6/collision/toolA-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 scale=0.001 0.001 0.001; visual mesh filename=package://frcobot_description/meshes/fr5v6/visual/toolA-250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 scale=0.001 0.001 0.001
- added link robot1_tool_tcp_link, mass 0.001; collision sphere radius=0.005; visual sphere radius=0.005
- added link robot2_base0_link, mass 6.8715; collision mesh filename=package://frcobot_description/meshes/fr5v6/collision/extra_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 scale=1 1 1; visual mesh filename=package://frcobot_description/meshes/fr5v6/visual/extra_bas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 scale=1 1 1
- added link robot2_base1_link, mass 0.40503; collision mesh filename=package://frcobot_description/meshes/fr5v6/collision/plant_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 scale=1 1 1; visual mesh filename=package://frcobot_description/meshes/fr5v6/visual/plant_lin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 scale=1 1 1
- added link robot2_base2_link, mass 1.6185; collision mesh filename=package://frcobot_description/meshes/fr5v6/collision/base_l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 scale=1 1 1; visual mesh filename=package://frcobot_description/meshes/fr5v6/visual/base_link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 scale=1 1 1
- added link robot2_j1_link, mass 4.3771; collision mesh filename=package://frcobot_description/meshes/fr5v6/collision/j1_lin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 scale=1 1 1; visual mesh filename=package://frcobot_description/meshes/fr5v6/visual/j1_link.D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 scale=1 1 1
- added link robot2_j2_link, mass 14.458; collision mesh filename=package://frcobot_description/meshes/fr5v6/collision/j2_lin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 scale=1 1 1; visual mesh filename=package://frcobot_description/meshes/fr5v6/visual/j2_link.D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 scale=1 1 1
- added link robot2_j3_link, mass 7.6737; collision mesh filename=package://frcobot_description/meshes/fr5v6/collision/j3_lin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 scale=1 1 1; visual mesh filename=package://frcobot_description/meshes/fr5v6/visual/j3_link.D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 scale=1 1 1
- added link robot2_j4_link, mass 1.6266; collision mesh filename=package://frcobot_description/meshes/fr5v6/collision/j4_lin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 scale=1 1 1; visual mesh filename=package://frcobot_description/meshes/fr5v6/visual/j4_link.D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 scale=1 1 1
- added link robot2_j5_link, mass 1.5812; collision mesh filename=package://frcobot_description/meshes/fr5v6/collision/j5_lin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 scale=1 1 1; visual mesh filename=package://frcobot_description/meshes/fr5v6/visual/j5_link.D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 scale=1 1 1
- added link robot2_j6_link, mass 0.52542; collision mesh filename=package://frcobot_description/meshes/fr5v6/collision/j6_lin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 scale=1 1 1; visual mesh filename=package://frcobot_description/meshes/fr5v6/visual/j6_link.D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 scale=1 1 1
- added link robot2_tool_link, mass 0.05; collision mesh filename=package://frcobot_description/meshes/fr5v6/collision/toolA-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 scale=0.001 0.001 0.001; visual mesh filename=package://frcobot_description/meshes/fr5v6/visual/toolA-250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 scale=0.001 0.001 0.001
- added link robot2_tool_tcp_link, mass 0.001; collision sphere radius=0.005; visual sphere radius=0.005
Joints:
- removed joint robot1_extra_base_to_plant
- removed joint robot1_extra_plant_to_base
- removed joint robot2_extra_base_to_plant
- removed joint robot2_extra_plant_to_base
- added joint robot1_base0_to_base1: type fixed, parent robot1_base0_link, child robot1_base1_link, origin xyz=-0.00031408 0.00046097 0.41799 rpy=0 0 0
- added joint robot1_base1_to_base2: type fixed, parent robot1_base1_link, child robot1_base2_link, origin xyz=0 0 0.0001 rpy=0 0 0
- added joint robot1_tcp_joint: type fixed, parent robot1_tool_link, child robot1_tool_tcp_link, origin xyz=0 0 0.25 rpy=0 0 0
- added joint robot1_tool_joint: type fixed, parent robot1_j6_link, child robot1_tool_link, origin xyz=0 0 0.1 rpy=0 0 0, axis 0 0 1, limit lower=0 upper=0 effort=0 velocity=0
- added joint robot2_base0_to_base1: type fixed, parent robot2_base0_link, child robot2_base1_link, origin xyz=-0.00031408 0.00046097 0.41799 rpy=0 0 0
- added joint robot2_base1_to_base2: type fixed, parent robot2_base1_link, child robot2_base2_link, origin xyz=0 0 0.0001 rpy=0 0 0
- added joint robot2_tcp_joint: type fixed, parent robot2_tool_link, child robot2_tool_tcp_link, origin xyz=0 0 0.25 rpy=0 0 0
- added joint robot2_tool_joint: type fixed, parent robot2_j6_link, child robot2_tool_link, origin xyz=0 0 0.1 rpy=0 0 0, axis 0 0 1, limit lower=0 upper=0 effort=0 velocity=0
- joint robot1_j1: child robot1_j1_Link -> robot1_j1_link; parent robot1_base_link -> robot1_base2_link
- joint robot1_j2: child robot1_j2_Link -> robot1_j2_link; parent robot1_j1_Link -> robot1_j1_link
- joint robot1_j3: child robot1_j3_Link -> robot1_j3_link; parent robot1_j2_Link -> robot1_j2_link
- joint robot1_j4: child robot1_j4_Link -> robot1_j4_link; parent robot1_j3_Link -> robot1_j3_link
- joint robot1_j5: child robot1_j5_Link -> robot1_j5_link; parent robot1_j4_Link -> robot1_j4_link
- joint robot1_j6: child robot1_j6_Link -> robot1_j6_link; parent robot1_j5_Link -> robot1_j5_link
- joint robot1_joint_base: child robot1_extra_base_link -> robot1_base0_link
- joint robot2_j1: child robot2_j1_Link -> robot2_j1_link; parent robot2_base_link -> robot2_base2_link
- joint robot2_j2: child robot2_j2_Link -> robot2_j2_link; parent robot2_j1_Link -> robot2_j1_link
- joint robot2_j3: child robot2_j3_Link -> robot2_j3_link; parent robot2_j2_Link -> robot2_j2_link
- joint robot2_j4: child robot2_j4_Link -> robot2_j4_link; parent robot2_j3_Link -> robot2_j3_link
- joint robot2_j5: child robot2_j5_Link -> robot2_j5_link; parent robot2_j4_Link -> robot2_j4_link
- joint robot2_j6: child robot2_j6_Link -> robot2_j6_link; parent robot2_j5_Link -> robot2_j5_link
- joint robot2_joint_base: child robot2_extra_base_link -> robot2_base0_link

File: catkin_ws/src/fr5v6_single_moveit_config/config/gazebo_fr5v6_single_arm.urdf (robot description, URDF)
Before this commit: robot fr5v6_single_arm, 12 links, 11 joints
Links:
- removed link fr5v6_base_link
- removed link fr5v6_extra_base_link
- removed link fr5v6_j1_link
- removed link fr5v6_j2_link
- removed link fr5v6_j3_link
- removed link fr5v6_j4_link
- removed link fr5v6_j5_link
- removed link fr5v6_j6_link
- removed link fr5v6_plant_link
- removed link fr5v6_tool_link
- removed link fr5v6_tool_tcp_link
- removed link world
- added link frrobot_base0_link, mass 6.8715; collision mesh filename=package://frcobot_description/meshes/fr5v6/collision/extra_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 scale=1 1 1; visual mesh filename=package://frcobot_description/meshes/fr5v6/visual/extra_bas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 scale=1 1 1
- added link frrobot_base1_link, mass 0.40503; collision mesh filename=package://frcobot_description/meshes/fr5v6/collision/plant_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 scale=1 1 1; visual mesh filename=package://frcobot_description/meshes/fr5v6/visual/plant_lin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 scale=1 1 1
- added link frrobot_base2_link, mass 1.6185; collision mesh filename=package://frcobot_description/meshes/fr5v6/collision/base_l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 scale=1 1 1; visual mesh filename=package://frcobot_description/meshes/fr5v6/visual/base_link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 scale=1 1 1
- added link frrobot_j1_link, mass 4.3771; collision mesh filename=package://frcobot_description/meshes/fr5v6/collision/j1_lin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 scale=1 1 1; visual mesh filename=package://frcobot_description/meshes/fr5v6/visual/j1_link.D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 scale=1 1 1
- added link frrobot_j2_link, mass 14.458; collision mesh filename=package://frcobot_description/meshes/fr5v6/collision/j2_lin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 scale=1 1 1; visual mesh filename=package://frcobot_description/meshes/fr5v6/visual/j2_link.D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 scale=1 1 1
- added link frrobot_j3_link, mass 7.6737; collision mesh filename=package://frcobot_description/meshes/fr5v6/collision/j3_lin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 scale=1 1 1; visual mesh filename=package://frcobot_description/meshes/fr5v6/visual/j3_link.D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 scale=1 1 1
- added link frrobot_j4_link, mass 1.6266; collision mesh filename=package://frcobot_description/meshes/fr5v6/collision/j4_lin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 scale=1 1 1; visual mesh filename=package://frcobot_description/meshes/fr5v6/visual/j4_link.D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 scale=1 1 1
- added link frrobot_j5_link, mass 1.5812; collision mesh filename=package://frcobot_description/meshes/fr5v6/collision/j5_lin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 scale=1 1 1; visual mesh filename=package://frcobot_description/meshes/fr5v6/visual/j5_link.D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 scale=1 1 1
- added link frrobot_j6_link, mass 0.52542; collision mesh filename=package://frcobot_description/meshes/fr5v6/collision/j6_lin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 scale=1 1 1; visual mesh filename=package://frcobot_description/meshes/fr5v6/visual/j6_link.D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 scale=1 1 1
- added link frrobot_tool_link, mass 0.05; collision mesh filename=package://frcobot_description/meshes/fr5v6/collision/toolA-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 scale=0.001 0.001 0.001; visual mesh filename=package://frcobot_description/meshes/fr5v6/visual/toolA-250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 scale=0.001 0.001 0.001
- added link frrobot_tool_tcp_link, mass 0.001; collision sphere radius=0.005; visual sphere radius=0.005
- added link robot_base
Joints:
- removed joint fr5v6_extra_base_to_plant
- removed joint fr5v6_extra_plant_to_base
- removed joint fr5v6_j1
- removed joint fr5v6_j2
- removed joint fr5v6_j3
- removed joint fr5v6_j4
- removed joint fr5v6_j5
- removed joint fr5v6_j6
- removed joint fr5v6_joint_base
- removed joint fr5v6_tool
- removed joint fr5v6_tool_tcp_joint
- added joint frrobot_base0_to_base1: type fixed, parent frrobot_base0_link, child frrobot_base1_link, origin xyz=-0.00031408 0.00046097 0.41799 rpy=0 0 0
- added joint frrobot_base1_to_base2: type fixed, parent frrobot_base1_link, child frrobot_base2_link, origin xyz=0 0 0.0001 rpy=0 0 0
- added joint frrobot_j1: type revolute, parent frrobot_base2_link, child frrobot_j1_link, origin xyz=0 0 0 rpy=0 0 0, axis 0 0 1, limit lower=-3.0543 upper=3.0543 effort=150 velocity=3.15
- added joint frrobot_j2: type revolute, parent frrobot_j1_link, child frrobot_j2_link, origin xyz=0 0 0.152 rpy=1.5708 0 0, axis 0 0 1, limit lower=-4.6251 upper=1.4835 effort=150 velocity=3.15
- added joint frrobot_j3: type revolute, parent frrobot_j2_link, child frrobot_j3_link, origin xyz=-0.425 0 0 rpy=0 0 0, axis 0 0 1, limit lower=-2.8274 upper=2.8274 effort=150 velocity=3.15
- added joint frrobot_j4: type revolute, parent frrobot_j3_link, child frrobot_j4_link, origin xyz=-0.39501 0 0 rpy=0 0 0, axis 0 0 1, limit lower=-4.6251 upper=1.4835 effort=28 velocity=3.2
- added joint frrobot_j5: type revolute, parent frrobot_j4_link, child frrobot_j5_link, origin xyz=0 0 0.1021 rpy=1.5708 0 0, axis 0 0 1, limit lower=-3.0543 upper=3.0543 effort=28 velocity=3.2
- added joint frrobot_j6: type revolute, parent frrobot_j5_link, child frrobot_j6_link, origin xyz=0 0 0.102 rpy=-1.5708 0 0, axis 0 0 1, limit lower=-3.0543 upper=3.0543 effort=28 velocity=3.2
- added joint frrobot_joint_base: type fixed, parent robot_base, child frrobot_base0_link, origin xyz=0 0 0 rpy=0 0 0
- added joint frrobot_tcp_joint: type fixed, parent frrobot_tool_link, child frrobot_tool_tcp_link, origin xyz=0 0 0.25 rpy=0 0 0
- added joint frrobot_tool_joint: type fixed, parent frrobot_j6_link, child frrobot_tool_link, origin xyz=0 0 0.1 rpy=0 0 0, axis 0 0 1, limit lower=0 upper=0 effort=0 velocity=0

File: catkin_ws/src/frcobot_description/urdf/fr5v6_dual_arms.xacro (robot description, xacro)
@@ -1,56 +1,11 @@
 <?xml version="1.0"?>
 <robot name="fr5v6_dual_arms" xmlns:xacro="http://ros.org/wiki/xacro">
-    <!-- add arms names prefixes -->
+    <!-- 定义参数 -->
     <xacro:arg name="arm_id_1" default="robot1" />
     <xacro:arg name="arm_id_2" default="robot2" />
-    <!-- load arm/hand models and utils (which adds the robot inertia tags to be Gazebo-simulation
-    ready) -->
-    <!-- <xacro:include filename="$(find franka_description)/robots/common/utils.xacro" /> -->
-    <!-- <xacro:include filename="$(find franka_description)/robots/common/franka_arm.xacro" /> -->
-    <!-- <xacro:include filename="$(find franka_description)/robots/common/franka_hand.xacro" /> -->
+    <!-- 添加虚拟根链接 -->
     <xacro:include filename="$(find frcobot_description)/urdf/fr5v6_library.xacro" />
+    <!-- 添加虚拟根链接 -->
     <link name="world" />
-    <!-- box shaped table as base for the 2 Pandas -->
-    <!-- <link name="base">
-        <visual>
-            <origin xyz="0 0 0.5" rpy="0 0 0" />
-            <geometry>
-                <box size="1 2 1" />
-            </geometry>
-            <material name="White">
-                <color rgba="1.0 1.0 1.0 1.0" />
-            </material>
-        </visual>
-        <collision>
-            <origin xyz="0 0 0.5" rpy="0 0 0" />
-            <geometry>
-                <box size="1 2 1" />
-            </geometry>
-        </collision>
-        <inertial>
-            <origin xyz="0.0 0.0 0.0" rpy="0.0 0.0 0.0" />
-            <mass value="10.0" />
-            <inertia ixx="0.001" ixy="0.0" ixz="0.001" iyy="0.0" iyz="0.0" izz="0.001" />
-        </inertial>
-    </link> -->
-    <!-- <joint name="base_to_world" type="fixed">
-        <parent link="world" />
-        <child link="base" />
-        <origin xyz="0.0 0.0 0.0" rpy="0.0 0.0 0.0" />
-    </joint> -->
-    <!-- right arm with gripper -->
-    <!-- <xacro:fr5v6_arm arm_id="$(arg arm_id_1)" connected_to="base" xyz="0 -0.5 1"
-        gazebo="true"
-        safety_distance="0.03"
-        joint_limits="${xacro.load_yaml('$(find fr5v6_moveit_config)/config/joint_limits.yaml')}"
-        /> -->
-    <!-- <xacro:franka_hand arm_id="$(arg arm_id_1)" rpy="0 0 ${-pi/4}"
-        connected_to="$(arg arm_id_1)_link8" gazebo="true" safety_distance="0.03" /> -->
-    <!-- left arm with gripper -->
-    <!-- <xacro:fr5v6_arm arm_id="$(arg arm_id_2)" connected_to="base" xyz="0 0.5 1" gazebo="true"
-        safety_distance="0.03"
-        joint_limits="${xacro.load_yaml('$(find fr5v6_moveit_config)/config/joint_limits.yaml')}" /> -->
-    <!-- <xacro:franka_hand arm_id="$(arg arm_id_2)" rpy="0 0 ${-pi/4}"
-        connected_to="$(arg arm_id_2)_link8" gazebo="true" safety_distance="0.03" /> -->
     <xacro:fr5v6_arm arm_id="$(arg arm_id_1)" connected_to="world" xyz="0 -0.5 0" />
     <xacro:fr5v6_arm arm_id="$(arg arm_id_2)" connected_to="world" xyz="0 0.5 0" />

File: catkin_ws/src/frcobot_description/urdf/fr5v6_library.xacro (robot description, xacro)
@@ -6,5 +6,5 @@
             <joint name="${arm_id}_joint_base" type="fixed">
                 <parent link="${connected_to}" />
-                <child link="${arm_id}_extra_base_link" />
+                <child link="${arm_id}_base0_link" />
                 <origin rpy="${rpy}" xyz="${xyz}" />
             </joint>
@@ -25,5 +25,5 @@
                     <origin xyz="0 0 0" rpy="0 0 0" />
                     <geometry>
-                        <mesh filename="${visual_mesh}" scale="${scale}"/>
+                        <mesh filename="${visual_mesh}" scale="${scale}" />
                     </geometry>
                     <material name="${material_name}">
@@ -34,10 +34,10 @@
                     <origin xyz="0 0 0" rpy="0 0 0" />
                     <geometry>
-                        <mesh filename="${collision_mesh}" scale="${scale}"/>
+                        <mesh filename="${collision_mesh}" scale="${scale}" />
                     </geometry>
                 </collision>
             </link>
         </xacro:macro>
-        <xacro:link_with_inertial name="${arm_id}_extra_base_link"
+        <xacro:link_with_inertial name="${arm_id}_base0_link"
             xyz="-0.00035477 0.0011738 0.038422"
             rpy="0 0 0"
@@ -51,10 +51,5 @@
             visual_mesh="package://frcobot_description/meshes/fr5v6/visual/extra_base_link.DAE"
             collision_mesh="package://frcobot_description/meshes/fr5v6/collision/extra_base_link.STL" />
-        <joint name="${arm_id}_extra_base_to_plant" type="fixed">
-            <parent link="${arm_id}_extra_base_link" />
-            <child link="${arm_id}_plant_link" />
-            <origin xyz="-0.00031408 0.00046097 0.41799" rpy="0 0 0" />
-        </joint>
-        <xacro:link_with_inertial name="${arm_id}_plant_link" xyz="2.7756E-16 0 -0.008"
+        <xacro:link_with_inertial name="${arm_id}_base1_link" xyz="2.7756E-16 0 -0.008"
             rpy="0 0 0"
             mass="0.40503"
@@ -67,10 +62,10 @@
             visual_mesh="package://frcobot_description/meshes/fr5v6/visual/plant_link.DAE"
             collision_mesh="package://frcobot_description/meshes/fr5v6/collision/plant_link.STL" />
-        <joint name="${arm_id}_extra_plant_to_base" type="fixed">
-            <parent link="${arm_id}_plant_link" />
-            <child link="${arm_id}_base_link" />
-            <origin xyz="0 0 0.0001" rpy="0 0 0" />
-        </joint>
-        <xacro:link_with_inertial name="${arm_id}_base_link" xyz="-0.00031896 -0.00029673 0.042463"
+        <joint name="${arm_id}_base0_to_base1" type="fixed">
+            <parent link="${arm_id}_base0_link" />
+            <child link="${arm_id}_base1_link" />
+            <origin xyz="-0.00031408 0.00046097 0.41799" rpy="0 0 0" />
+        </joint>
+        <xacro:link_with_inertial name="${arm_id}_base2_link" xyz="-0.00031896 -0.00029673 0.042463"
             rpy="0 0 0"
             mass="1.6185"
@@ -79,4 +74,9 @@
             visual_mesh="package://frcobot_description/meshes/fr5v6/visual/base_link.DAE"
             collision_mesh="package://frcobot_description/meshes/fr5v6/collision/base_link.STL" />
+        <joint name="${arm_id}_base1_to_base2" type="fixed">
+            <parent link="${arm_id}_base1_link" />
+            <child link="${arm_id}_base2_link" />
+            <origin xyz="0 0 0.0001" rpy="0 0 0" />
+        </joint>
         <xacro:link_with_inertial name="${arm_id}_j1_link" xyz="5.0029E-07 -0.0040922 0.14629"
             rpy="0 0 0"
@@ -88,5 +88,5 @@
         <joint name="${arm_id}_j1" type="revolute">
             <origin xyz="0 0 0" rpy="0 0 0" />
-            <parent link="${arm_id}_base_link" />
+            <parent link="${arm_id}_base2_link" />
             <child link="${arm_id}_j1_link" />
             <axis xyz="0 0 1" />
@@ -195,5 +195,5 @@
             collision_mesh="package://frcobot_description/meshes/fr5v6/collision/toolA-250mm.STL"
             scale="0.001 0.001 0.001" />
-        <joint name="${arm_id}_tool" type="fixed">
+        <joint name="${arm_id}_tool_joint" type="fixed">
             <origin xyz="0 0 0.1" rpy="0 0 0" />
             <parent link="${arm_id}_j6_link" />
@@ -230,5 +230,5 @@
             </collision>
         </link>
-        <joint name="${arm_id}_tool_tcp_joint" type="fixed">
+        <joint name="${arm_id}_tcp_joint" type="fixed">
             <origin xyz="0 0 0.25" rpy="0 0 0" />
             <parent link="${arm_id}_tool_link" />

File: catkin_ws/src/frcobot_description/urdf/fr5v6_single_arm.xacro (robot description, xacro)
@@ -1,11 +1,21 @@
-<?xml version="1.0" encoding="utf-8"?>
+<?xml version="1.0"?>
 <robot name="fr5v6_single_arm" xmlns:xacro="http://www.ros.org/wiki/xacro">
     <!-- 定义参数 -->
-    <xacro:property name="arm_id" value="fr5v6" />
-    <!-- 引用库文件 -->
+    <xacro:arg name="arm_id" default="frrobot" />
+    <!-- 添加虚拟根链接 -->
     <xacro:include filename="$(find frcobot_description)/urdf/fr5v6_library.xacro" />
     <!-- 添加虚拟根链接 -->
-    <link name="world" />
+    <link name="robot_base" />
     <!-- 实例化机械臂 -->
-    <xacro:fr5v6_arm arm_id="${arm_id}" connected_to="world" xyz="0 0 0" rpy="0 0 0" />
+    <xacro:fr5v6_arm arm_id="$(arg arm_id)" connected_to="robot_base" xyz="0 0 0" rpy="0 0 0" />
+    <xacro:gazebo-joint joint="$(arg arm_id)_j1" />
+    <xacro:gazebo-joint joint="$(arg arm_id)_j2" />
+    <xacro:gazebo-joint joint="$(arg arm_id)_j3" />
+    <xacro:gazebo-joint joint="$(arg arm_id)_j4" />
+    <xacro:gazebo-joint joint="$(arg arm_id)_j5" />
+    <xacro:gazebo-joint joint="$(arg arm_id)_j6" />
+    <!-- load ros_control plugin -->
+    <gazebo>
+        <plugin name="gazebo_ros_control" filename="libgazebo_ros_control.so" />
+    </gazebo>
 </robot>
