Commit message: 20250402 进行了双臂标定，仍有些许误差

File: catkin_ws/src/fr5v6_dual_moveit_config/config/gazebo_fr5v6_dual_arms.urdf (robot description, URDF)
Before this commit: robot fr5v6_dual_arms, 23 links, 22 joints
Links:
- removed link robot1_tool_tcp_link
- removed link robot2_tool_tcp_link
- link robot1_base0_link: mass 6.8715 -> 50.058
- link robot1_base1_link: mass 0.40503 -> 3.1592
- link robot1_tool_link: mass 0.05 -> 0.1; geometry 
- link robot2_base0_link: mass 6.8715 -> 50.058
- link robot2_base1_link: mass 0.40503 -> 3.1592
- link robot2_tool_link: mass 0.05 -> 0.1; geometry 
Joints:
- removed joint robot1_joint_base
- removed joint robot1_tcp_joint
- removed joint robot2_joint_base
- removed joint robot2_tcp_joint
- added joint robot1_to_robot2: type fixed, parent robot1_base0_link, child robot2_base0_link, origin xyz=-0.0313854 0.753229 0.00827339 rpy=0.0523678 0.0233265 -0.133503
- added joint world_to_robot1: type fixed, parent world, child robot1_base0_link, origin xyz=0 0 0 rpy=0 0 0
- joint robot1_base0_to_base1: origin xyz=-0.00031408 0.00046097 0.41799 rpy=0 0 0 -> xyz=0 0 0.487 rpy=0 0 0
- joint robot1_tool_joint: axis 0 0 1 -> (none); limit lower=0 upper=0 effort=0 velocity=0 -> (none)
- joint robot2_base0_to_base1: origin xyz=-0.00031408 0.00046097 0.41799 rpy=0 0 0 -> xyz=0 0 0.487 rpy=0 0 0
- joint robot2_tool_joint: axis 0 0 1 -> (none); limit lower=0 upper=0 effort=0 velocity=0 -> (none)

File: catkin_ws/src/frcobot_description/urdf/fr5v6_dual_arms.xacro (robot description, xacro)
@@ -1,13 +1,52 @@
 <?xml version="1.0"?>
-<robot name="fr5v6_dual_arms" xmlns:xacro="http://ros.org/wiki/xacro">
+<robot name="fr5v6_dual_arms" xmlns:xacro="http://www.ros.org/wiki/xacro">
     <!-- 定义参数 -->
     <xacro:arg name="arm_id_1" default="robot1" />
     <xacro:arg name="arm_id_2" default="robot2" />
+    <!-- 定义工具参数 -->
+    <xacro:arg name="robot1_tool" default="none"/>
+    <xacro:arg name="robot2_tool" default="none"/>
+    <!-- 导入标定参数 -->
+    <xacro:property name="calibration_file" value="$(find frcobot_description)/config/dual_arm_calibration.yaml"/>
+    <xacro:property name="calib" value="${xacro.load_yaml(calibration_file)}"/>
+    <!-- 加载工具配置文件 -->
+    <xacro:property name="tools_config" value="$(find frcobot_description)/config/tools.yaml"/>
+    <xacro:property name="tools" value="${xacro.load_yaml(tools_config)}"/>
+    <!-- 获取标定参数 -->
+    <xacro:property name="trans_x" value="${calib['left_to_right_transform']['translation']['x']}"/>
+    <xacro:property name="trans_y" value="${calib['left_to_right_transform']['translation']['y']}"/>
+    <xacro:property name="trans_z" value="${calib['left_to_right_transform']['translation']['z']}"/>
+    <xacro:property name="roll" value="${calib['left_to_right_transform']['rpy']['roll']}"/>
+    <xacro:property name="pitch" value="${calib['left_to_right_transform']['rpy']['pitch']}"/>
+    <xacro:property name="yaw" value="${calib['left_to_right_transform']['rpy']['yaw']}"/>
+    <!-- 获取工具配置 -->
+    <xacro:property name="robot1_tool_config" value="${tools['tools']['$(arg robot1_tool)']}"/>
+    <xacro:property name="robot2_tool_config" value="${tools['tools']['$(arg robot2_tool)']}"/>
     <!-- 添加虚拟根链接 -->
     <xacro:include filename="$(find frcobot_description)/urdf/fr5v6_library.xacro" />
-    <!-- 添加虚拟根链接 -->
-    <link name="world" />
-    <xacro:fr5v6_arm arm_id="$(arg arm_id_1)" connected_to="world" xyz="0 -0.5 0" />
-    <xacro:fr5v6_arm arm_id="$(arg arm_id_2)" connected_to="world" xyz="0 0.5 0" />
+    <!-- 创建世界链接作为唯一根链接 -->
+    <link name="world"/>
+    <!-- 连接世界链接到左臂基座 -->
+    <joint name="world_to_robot1" type="fixed">
+        <parent link="world"/>
+        <child link="robot1_base0_link"/>
+        <origin xyz="0 0 0" rpy="0 0 0"/>
+    </joint>
+    <!-- 创建左臂（机器人1） -->
+    <xacro:fr5v6_arm
+        arm_id="robot1"
+        tool_name="$(arg robot1_tool)"
+        tool_config="${robot1_tool_config}"/>
+    <!-- 连接左臂到右臂 - 使用标定参数 -->
+    <joint name="robot1_to_robot2" type="fixed">
+        <parent link="robot1_base0_link"/>
+        <child link="robot2_base0_link"/>
+        <origin xyz="${trans_x} ${trans_y} ${trans_z}" rpy="${roll} ${pitch} ${yaw}"/>
+    </joint>
+    <!-- 添加机器人2 -->
+    <xacro:fr5v6_arm
+        arm_id="robot2"
+        tool_name="$(arg robot2_tool)"
+        tool_config="${robot2_tool_config}"/>
     <!-- right arm joints control interface -->
     <xacro:gazebo-joint joint="$(arg arm_id_1)_j1" />

File: catkin_ws/src/frcobot_description/urdf/fr5v6_library.xacro (robot description, xacro)
@@ -2,5 +2,5 @@
 <robot name="fr5v6" xmlns:xacro="http://www.ros.org/wiki/xacro">
     <xacro:macro name="fr5v6_arm"
-        params="arm_id:='fr5v6' connected_to:='' xyz:='0 0 0' rpy:='0 0 0'">
+        params="arm_id:='fr5v6' connected_to:='' xyz:='0 0 0' rpy:='0 0 0' tool_name:='none' tool_config:='{}'">
         <xacro:unless value="${not connected_to}">
             <joint name="${arm_id}_joint_base" type="fixed">
@@ -188,52 +188,76 @@
                 k_velocity="10" />
         </joint>
-        <!-- Uncomment and modify the following section if you have a tool link -->
-        <xacro:link_with_inertial name="${arm_id}_tool_link" xyz="0.24412 0.079181 -0.126"
-            rpy="0 0 0"
-            mass="0.05"
-            ixx="5.82E-7" ixy="0" ixz="0.0" iyy="1.15E-8" iyz="0.0" izz="5.82E-7"
-            visual_mesh="package://frcobot_description/meshes/fr5v6/visual/toolA-250mm.DAE"
-            collision_mesh="package://frcobot_description/meshes/fr5v6/collision/toolA-250mm.STL"
-            scale="0.001 0.001 0.001" />
+        <!-- 添加工具链接 - 始终创建 -->
+        <link name="${arm_id}_tool_link">
+            <xacro:if value="${tool_name != 'none'}">
+                <visual>
+                    <origin
+                        xyz="${tool_config['origin']['xyz'][0]}
+                            ${tool_config['origin']['xyz'][1]}
+                            ${tool_config['origin']['xyz'][2]}"
+                        rpy="${tool_config['origin']['rpy'][0]}
+                            ${tool_config['origin']['rpy'][1]}
+                            ${tool_config['origin']['rpy'][2]}" />
+                    <geometry>
+                        <mesh filename="${tool_config['mesh_path']}" scale="0.001 0.001 0.001" />
+                    </geometry>
+                </visual>
+                <collision>
+                    <origin
+                        xyz="${tool_config['origin']['xyz'][0]}
+                            ${tool_config['origin']['xyz'][1]}
+                            ${tool_config['origin']['xyz'][2]}"
+                        rpy="${tool_config['origin']['rpy'][0]}
+                            ${tool_config['origin']['rpy'][1]}
+                            ${tool_config['origin']['rpy'][2]}" />
+                    <geometry>
+                        <mesh filename="${tool_config['collision_mesh']}" scale="0.001 0.001 0.001" />
+                    </geometry>
+                </collision>
+            </xacro:if>
+            <inertial>
+                <origin xyz="0 0 0" rpy="0 0 0"/>
+                <mass value="${(tool_name == 'none') * 0.1 + (tool_name != 'none') * tool_config['mass']}" />
+                <inertia
+                    ixx="${(tool_name == 'none') * 0.1 + (tool_name != 'none') * tool_config['inertia']['ixx']}"
+                    ixy="${(tool_name == 'none') * 0.0 + (tool_name != 'none') * tool_config['inertia']['ixy']}"
+                    ixz="${(tool_name == 'none') * 0.0 + (tool_name != 'none') * tool_config['inertia']['ixz']}"
+                    iyy="${(tool_name == 'none') * 0.1 + (tool_name != 'none') * tool_config['inertia']['iyy']}"
+                    iyz="${(tool_name == 'none') * 0.0 + (tool_name != 'none') * tool_config['inertia']['iyz']}"
+                    izz="${(tool_name == 'none') * 0.1 + (tool_name != 'none') * tool_config['inertia']['izz']}" />
+            </inertial>
+        </link>
+        <!-- 总是创建工具关节 -->
         <joint name="${arm_id}_tool_joint" type="fixed">
-            <origin xyz="0 0 0.1" rpy="0 0 0" />
             <parent link="${arm_id}_j6_link" />
             <child link="${arm_id}_tool_link" />
-            <axis xyz="0 0 1" />
-            <limit lower="0" upper="0" effort="0" velocity="0" />
-            <calibration rising="0" falling="0" />
-            <dynamics damping="0" friction="0" />
-            <safety_controller soft_lower_limit="0" soft_upper_limit="0" k_position="0"
-                k_velocity="0" />
-        </joint>
-        <!-- 添加工具末端TCP坐标系（使用基本几何体） -->
-        <link name="${arm_id}_tool_tcp_link">
-            <inertial>
-                <origin xyz="0 0 0" rpy="0 0 0" />
-                <mass value="0.001" />
-                <inertia ixx="0.0000001" ixy="0" ixz="0" iyy="0.0000001" iyz="0" izz="0.0000001" />
-            </inertial>
-            <visual>
-                <origin xyz="0 0 0" rpy="0 0 0" />
-                <geometry>
-                    <sphere radius="0.005"/>
-                </geometry>
-                <material name="">
-                    <color rgba="1 0 0 1" />
-                </material>
-            </visual>
-            <!-- 添加碰撞几何体 -->
-            <collision>
-                <origin xyz="0 0 0" rpy="0 0 0" />
-                <geometry>
-                    <sphere radius="0.005"/>
-                </geometry>
-            </collision>
-        </link>
-        <joint name="${arm_id}_tcp_joint" type="fixed">
-            <origin xyz="0 0 0.25" rpy="0 0 0" />
-            <parent link="${arm_id}_tool_link" />
-            <child link="${arm_id}_tool_tcp_link" />
-        </joint>
+            <!-- 先应用固定的法兰偏移 -->
+            <origin xyz="0 0 0.1" rpy="0 0 0" />
+        </joint>
+        <!-- 只在有tool时创建TCP链接和关节 -->
+        <xacro:if value="${tool_name != 'none'}">
+            <link name="${arm_id}_tcp_link">
+                <visual>
+                    <origin xyz="0 0 0" rpy="0 0 0" />
+                    <geometry>
+                        <sphere radius="0.005" />
+                    </geometry>
+                    <material name="">
+                        <color rgba="1 0 0 1" />
+                    </material>
+                </visual>
+            </link>
+            <joint name="${arm_id}_tcp_joint" type="fixed">
+                <parent link="${arm_id}_tool_link" />
+                <child link="${arm_id}_tcp_link" />
+                <origin
+                    xyz="${tool_config['tcp']['xyz'][0]}
+                        ${tool_config['tcp']['xyz'][1]}
+                        ${tool_config['tcp']['xyz'][2]}"
+                    rpy="${tool_config['tcp']['rpy'][0]}
+                        ${tool_config['tcp']['rpy'][1]}
+                        ${tool_config['tcp']['rpy'][2]}" />
+            </joint>
+        </xacro:if>
     </xacro:macro>
     <xacro:macro name="gazebo-joint" params="joint ">

Commit message: feat: 将tool_link统一改为ee_link，并添加permanent_magnet和electronic_magnet工具支持
- 将机器人本体末端链接从tool_link统一改为ee_link
- 更新所有相关配置文件（URDF、SRDF、RViz配置等）
- 为permanent_magnet和electronic_magnet工具创建配置文件
- 更新工具URDF中的mesh路径为frcobot_tools包路径
- 创建collision和visual子文件夹并组织mesh文件
- 添加单臂可视化launch文件

File: catkin_ws/src/fr5v6_dual_moveit_config/config/gazebo_fr5v6_dual_arms.urdf (robot description, URDF)
Before this commit: robot fr5v6_dual_arms, 21 links, 20 joints
Links:
- removed link robot1_tool_link
- removed link robot2_tool_link
- added link robot1_ee_link, mass 0.1
- added link robot2_ee_link, mass 0.1
Joints:
- removed joint robot1_tool_joint
- removed joint robot2_tool_joint
- added joint robot1_ee_joint: type fixed, parent robot1_j6_link, child robot1_ee_link, origin xyz=0 0 0.1 rpy=0 0 0
- added joint robot2_ee_joint: type fixed, parent robot2_j6_link, child robot2_ee_link, origin xyz=0 0 0.1 rpy=0 0 0

File: catkin_ws/src/fr5v6_single_moveit_config/config/gazebo_fr5v6_single_arm.urdf (robot description, URDF)
Before this commit: robot fr5v6_single_arm, 11 links, 10 joints
Links:
- removed link frrobot_tool_link
- added link frrobot_ee_link, mass 0.1
Joints:
- removed joint frrobot_tool_joint
- added joint frrobot_ee_joint: type fixed, parent frrobot_j6_link, child frrobot_ee_link, origin xyz=0 0 0.1 rpy=0 0 0

File: catkin_ws/src/frcobot_description/urdf/fr5v6_library.xacro (robot description, xacro)
@@ -198,8 +198,8 @@
         <!-- 检查是否使用工具包系统 -->
         <xacro:property name="use_tool_package" value="${'tool_type' in tool_config}"/>
-        <!-- 如果使用工具包系统，先创建tool_link作为中间链接 -->
+        <!-- 如果使用工具包系统，先创建ee_link作为中间链接 -->
         <xacro:if value="${use_tool_package and tool_name != 'none'}">
-            <!-- 创建tool_link（连接到j6_link） -->
-            <link name="${arm_id}_tool_link">
+            <!-- 创建ee_link（连接到j6_link） -->
+            <link name="${arm_id}_ee_link">
                 <inertial>
                     <origin xyz="0 0 0" rpy="0 0 0"/>
@@ -210,12 +210,12 @@
                 </inertial>
             </link>
-            <!-- 创建从j6_link到tool_link的关节 -->
-            <joint name="${arm_id}_tool_joint" type="fixed">
+            <!-- 创建从j6_link到ee_link的关节 -->
+            <joint name="${arm_id}_ee_joint" type="fixed">
                 <parent link="${arm_id}_j6_link" />
-                <child link="${arm_id}_tool_link" />
+                <child link="${arm_id}_ee_link" />
                 <!-- 先应用固定的法兰偏移 -->
                 <origin xyz="0 0 0.1" rpy="0 0 0" />
             </joint>
-            <!-- 使用新的工具加载器，工具将连接到tool_link -->
+            <!-- 使用新的工具加载器，工具将连接到ee_link -->
             <xacro:load_tool arm_id="${arm_id}" tool_name="${tool_name}" tool_config="${tool_config}"/>
         </xacro:if>
@@ -223,5 +223,5 @@
         <xacro:unless value="${use_tool_package}">
             <!-- 添加工具链接 - 始终创建 -->
-            <link name="${arm_id}_tool_link">
+            <link name="${arm_id}_ee_link">
                 <xacro:if value="${tool_name != 'none'}">
                     <visual>
@@ -271,7 +271,7 @@
             </link>
             <!-- 总是创建工具关节 -->
-            <joint name="${arm_id}_tool_joint" type="fixed">
+            <joint name="${arm_id}_ee_joint" type="fixed">
                 <parent link="${arm_id}_j6_link" />
-                <child link="${arm_id}_tool_link" />
+                <child link="${arm_id}_ee_link" />
                 <!-- 先应用固定的法兰偏移 -->
                 <origin xyz="0 0 0.1" rpy="0 0 0" />
@@ -291,5 +291,5 @@
                 </link>
                 <joint name="${arm_id}_tcp_joint" type="fixed">
-                    <parent link="${arm_id}_tool_link" />
+                    <parent link="${arm_id}_ee_link" />
                     <child link="${arm_id}_tcp_link" />
                     <origin

File: catkin_ws/src/frcobot_description/urdf/tool_loader.xacro (robot description, xacro)
@@ -39,5 +39,5 @@
             <xacro:property name="collision_mesh_path" value="${tool_collision.get('mesh_path', '')}"/>
             <xacro:property name="collision_scale" value="${tool_collision.get('scale', [1,1,1])}"/>
-            <!-- 创建工具链接（使用工具名称作为链接名，避免与tool_link冲突） -->
+            <!-- 创建工具链接（使用工具名称作为链接名，避免与ee_link冲突） -->
             <link name="${arm_id}_${tool_name}_link">
                 <!-- 可视化 -->
@@ -78,10 +78,10 @@
                 </inertial>
             </link>
-            <!-- 创建工具关节（连接到tool_link，而不是j6_link） -->
-            <!-- 注意：tool_link已经在fr5v6_library.xacro中创建并连接到j6_link -->
+            <!-- 创建工具关节（连接到ee_link，而不是j6_link） -->
+            <!-- 注意：ee_link已经在fr5v6_library.xacro中创建并连接到j6_link -->
             <joint name="${arm_id}_${tool_name}_joint" type="fixed">
-                <parent link="${arm_id}_tool_link" />
+                <parent link="${arm_id}_ee_link" />
                 <child link="${arm_id}_${tool_name}_link" />
-                <!-- 工具偏移（tool_link已经包含了0.1m的法兰偏移） -->
+                <!-- 工具偏移（ee_link已经包含了0.1m的法兰偏移） -->
                 <origin
                     xyz="${tool_origin_xyz[0]} ${tool_origin_xyz[1]} ${tool_origin_xyz[2]}"
@@ -121,10 +121,10 @@
             <!-- 加载外部URDF文件 -->
             <xacro:include filename="${full_urdf_path}"/>
-            <!-- 创建从tool_link到工具根链接的关节（而不是j6_link） -->
-            <!-- 注意：tool_link已经在fr5v6_library.xacro中创建并连接到j6_link -->
+            <!-- 创建从ee_link到工具根链接的关节（而不是j6_link） -->
+            <!-- 注意：ee_link已经在fr5v6_library.xacro中创建并连接到j6_link -->
             <joint name="${arm_id}_${tool_name}_joint" type="fixed">
-                <parent link="${arm_id}_tool_link" />
+                <parent link="${arm_id}_ee_link" />
                 <child link="${root_link_name}" />
-                <!-- 工具安装偏移（tool_link已经包含了0.1m的法兰偏移） -->
+                <!-- 工具安装偏移（ee_link已经包含了0.1m的法兰偏移） -->
                 <xacro:property name="mount_xyz" value="${mount_offset['xyz']}"/>
                 <xacro:property name="mount_rpy" value="${mount_offset['rpy']}"/>

File: catkin_ws/src/frcobot_tools/tools/electronic_magnet/urdf/electronic_magnet.urdf (robot description, URDF)
Before this commit: robot electronic_magnet, 3 links, 2 joints
Links:
- link em_base_link: geometry collision mesh filename=package://frcobot_tools/tools/electronic_magnet/meshes/coll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; visual mesh filename=package://frcobot_tools/tools/electronic_magnet/meshes/visu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
- link em_ee_link: geometry collision mesh filename=package://frcobot_tools/tools/electronic_magnet/meshes/coll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; visual mesh filename=package://frcobot_tools/tools/electronic_magnet/meshes/visu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
- link em_tcp_link: geometry collision mesh filename=package://frcobot_tools/tools/electronic_magnet/meshes/coll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; visual mesh filename=package://frcobot_tools/tools/electronic_magnet/meshes/visu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

File: catkin_ws/src/frcobot_tools/tools/permanent_magnet/urdf/permanent_magnet.urdf (robot description, URDF)
Before this commit: robot permanent_magnet, 2 links, 1 joints
Links:
- link pm_base_link: geometry collision mesh filename=package://frcobot_tools/tools/permanent_magnet/meshes/colli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; visual mesh filename=package://frcobot_tools/tools/permanent_magnet/meshes/visua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
- link pm_tcp_link: geometry collision mesh filename=package://frcobot_tools/tools/permanent_magnet/meshes/colli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; visual mesh filename=package://frcobot_tools/tools/permanent_magnet/meshes/visua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
