Commit message: 20251212 完成测试

File: src/zlab_arm_description/tools/electronic_magnet/urdf/electronic_magnet.urdf (robot description, URDF)
Before this commit: robot electronic_magnet, 3 links, 2 joints
Links:
- link em_base_link: geometry collision mesh filename=package://zlab_arm_description/tools/electronic_magnet/mesh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; visual mesh filename=package://zlab_arm_description/tools/electronic_magnet/mesh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
- link em_ee_link: geometry collision mesh filename=package://zlab_arm_description/tools/electronic_magnet/mesh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; visual mesh filename=package://zlab_arm_description/tools/electronic_magnet/mesh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
- link em_tcp_link: geometry collision mesh filename=package://zlab_arm_description/tools/electronic_magnet/mesh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; visual mesh filename=package://zlab_arm_description/tools/electronic_magnet/mesh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

File: src/zlab_arm_description/tools/magnetic_sensor_bracket/urdf/bracket.urdf.xacro (robot description, xacro)
@@ -5,7 +5,8 @@
 <robot xmlns:xacro="http://www.ros.org/wiki/xacro"
   name="bracket">
-  <!-- 参数定义：允许外部指定链接名前缀 -->
-  <xacro:arg name="link_prefix" default=""/>
-  <xacro:property name="prefix" value="$(arg link_prefix)"/>
+  <!-- Arm ID: 从父xacro文件传递的全局变量tool_arm_id -->
+  <!-- 直接使用tool_arm_id作为前缀，避免循环定义 -->
+  <!-- Prefix for link names to avoid conflicts in dual arm setup -->
+  <xacro:property name="prefix" value="${tool_arm_id}_"/>
   <link name="${prefix}bracket_base_link">
     <inertial>

File: src/zlab_arm_description/zlab_arm/urdf/tool_loader.xacro (robot description, xacro)
@@ -111,67 +111,26 @@
             <xacro:property name="root_link_name" value="${urdf_config['root_link_name']}"/>
             <xacro:property name="tcp_link_name" value="${urdf_config['tcp_link_name']}"/>
-            <!-- 从配置中提取参数 -->
-            <xacro:property name="tool_origin_xyz" value="${tool_config['origin']['xyz']}"/>
-            <xacro:property name="tool_origin_rpy" value="${tool_config['origin']['rpy']}"/>
-            <xacro:property name="tool_tcp_xyz" value="${tool_config['tcp']['xyz']}"/>
-            <xacro:property name="tool_tcp_rpy" value="${tool_config['tcp']['rpy']}"/>
-            <xacro:property name="tool_mass" value="${tool_config['physical_properties']['mass']}"/>
-            <xacro:property name="tool_inertia" value="${tool_config['physical_properties']['inertia']}"/>
-            <xacro:property name="tool_inertia_ixx" value="${tool_inertia['ixx']}"/>
-            <xacro:property name="tool_inertia_ixy" value="${tool_inertia['ixy']}"/>
-            <xacro:property name="tool_inertia_ixz" value="${tool_inertia['ixz']}"/>
-            <xacro:property name="tool_inertia_iyy" value="${tool_inertia['iyy']}"/>
-            <xacro:property name="tool_inertia_iyz" value="${tool_inertia['iyz']}"/>
-            <xacro:property name="tool_inertia_izz" value="${tool_inertia['izz']}"/>
             <!-- 获取安装偏移配置 -->
             <xacro:property name="mount_offset" value="${urdf_config['mount_offset']}"/>
-            <!-- 直接从配置文件读取网格文件路径 -->
-            <xacro:property name="visual_path" value="${tool_config['visual_mesh']}"/>
-            <xacro:property name="collision_path" value="${tool_config['collision_mesh']}"/>
-            <!-- 完整网格文件路径 -->
-            <xacro:property name="visual_mesh_path" value="package://zlab_arm_description/tools/${tool_name}/${visual_path}"/>
-            <xacro:property name="collision_mesh_path" value="package://zlab_arm_description/tools/${tool_name}/${collision_path}"/>
-            <!-- 内联定义工具链接以避免命名冲突 -->
-            <link name="${arm_id}_${root_link_name}">
-                <inertial>
-                    <origin xyz="${tool_origin_xyz[0]} ${tool_origin_xyz[1]} ${tool_origin_xyz[2]}" rpy="${tool_origin_rpy[0]} ${tool_origin_rpy[1]} ${tool_origin_rpy[2]}" />
-                    <mass value="${tool_mass}" />
-                    <inertia ixx="${tool_inertia_ixx}" ixy="${tool_inertia_ixy}" ixz="${tool_inertia_ixz}" iyy="${tool_inertia_iyy}" iyz="${tool_inertia_iyz}" izz="${tool_inertia_izz}" />
-                </inertial>
-                <visual>
-                    <origin xyz="0 0 0" rpy="0 0 0" />
-                    <geometry>
-                        <mesh filename="${visual_mesh_path}" />
-                    </geometry>
-                    <material name="">
-                        <color rgba="1 1 1 1" />
-                    </material>
-                </visual>
-                <collision>
-                    <origin xyz="0 0 0" rpy="0 0 0" />
-                    <geometry>
-                        <mesh filename="${collision_mesh_path}" />
-                    </geometry>
-                </collision>
-            </link>
-            <link name="${arm_id}_${tcp_link_name}">
-                <inertial>
-                    <origin xyz="${tool_tcp_xyz[0]} ${tool_tcp_xyz[1]} ${tool_tcp_xyz[2]}" rpy="${tool_tcp_rpy[0]} ${tool_tcp_rpy[1]} ${tool_tcp_rpy[2]}" />
-                    <mass value="0.001" />
-                    <inertia ixx="1e-6" ixy="0.0" ixz="0.0" iyy="1e-6" iyz="0.0" izz="1e-6" />
-                </inertial>
-                <!-- TCP链接不显示任何可视化内容，只用于运动学计算 -->
-            </link>
-            <joint name="${arm_id}_${tcp_link_name}_joint" type="fixed">
-                <parent link="${arm_id}_${root_link_name}" />
-                <child link="${arm_id}_${tcp_link_name}" />
-                <origin xyz="${tool_tcp_xyz[0]} ${tool_tcp_xyz[1]} ${tool_tcp_xyz[2]}" rpy="${tool_tcp_rpy[0]} ${tool_tcp_rpy[1]} ${tool_tcp_rpy[2]}" />
-            </joint>
+            <xacro:property name="mount_xyz" value="${mount_offset['xyz']}"/>
+            <xacro:property name="mount_rpy" value="${mount_offset['rpy']}"/>
+            <!-- 构建工具文件路径 -->
+            <xacro:property name="tool_file_path" value="$(find zlab_arm_description)/tools/${tool_name}/${urdf_file}"/>
+            <!-- 设置全局变量供工具xacro文件使用 -->
+            <xacro:property name="tool_arm_id" value="${arm_id}"/>
+            <!-- 加载工具URDF/xacro文件 -->
+            <!-- 如果配置文件指定的是.urdf.xacro文件，直接include（它会使用tool_arm_id变量） -->
+            <xacro:if value="${urdf_file.endswith('.urdf.xacro')}">
+                <!-- 使用xacro include，工具xacro文件会从tool_arm_id变量获取arm_id -->
+                <xacro:include filename="${tool_file_path}"/>
+            </xacro:if>
+            <xacro:unless value="${urdf_file.endswith('.urdf.xacro')}">
+                <!-- 如果是.urdf文件，直接include（不支持arm_id前缀，会有命名冲突） -->
+                <xacro:include filename="${tool_file_path}"/>
+            </xacro:unless>
             <!-- 创建从ee_link到工具根链接的关节 -->
             <joint name="${arm_id}_${tool_name}_joint" type="fixed">
                 <parent link="${arm_id}_ee_link" />
                 <child link="${arm_id}_${root_link_name}" />
-                <xacro:property name="mount_xyz" value="${mount_offset['xyz']}"/>
-                <xacro:property name="mount_rpy" value="${mount_offset['rpy']}"/>
                 <origin
                     xyz="${mount_xyz[0]} ${mount_xyz[1]} ${mount_xyz[2]}"

File: src/zlab_arm_dual_moveit_config/config/zlab_dual_arms.srdf.xacro (robot description, xacro)
@@ -4,5 +4,8 @@
     A URDF file must exist for this robot as well, where the joints and the links that are referenced are defined
 -->
-<robot name="zlab_dual_arms">
+<robot name="zlab_dual_arms" xmlns:xacro="http://www.ros.org/wiki/xacro">
+    <!-- Tool parameters for dynamic collision disable configuration -->
+    <xacro:arg name="arm1_tool" default="none"/>
+    <xacro:arg name="arm2_tool" default="none"/>
     <!--GROUPS: Representation of a set of joints and links. This can be useful for specifying DOF to plan for, defining arms, end effectors, etc-->
     <!--LINKS: When a link is specified, the parent joint of that link (if it exists) is automatically included-->
@@ -196,5 +199,65 @@
     <disable_collisions link1="arm2_j4_link" link2="arm2_j6_link" reason="Never"/>
     <disable_collisions link1="arm2_j5_link" link2="arm2_j6_link" reason="Adjacent"/>
-    <!-- Tool collision disable - will be dynamically added based on tool_name parameter -->
-    <!-- These will be handled by the launch file based on the tool being used -->
+    <!-- Tool collision disable - dynamically loaded from tool configuration files -->
+    <!-- Macro to generate disable_collisions from tool config -->
+    <xacro:macro name="generate_tool_collision_disable" params="arm_id tool_name">
+        <xacro:unless value="${tool_name == 'none'}">
+            <xacro:property name="tool_config_path"
+                            value="$(find zlab_arm_description)/tools/${tool_name}/config/tool.yaml"/>
+            <xacro:property name="tool_config"
+                            value="${xacro.load_yaml(tool_config_path)}"/>
+            <!-- Check if collision_disable configuration exists -->
+            <xacro:if value="${'collision_disable' in tool_config}">
+                <xacro:property name="collision_disable_list" value="${tool_config['collision_disable']}"/>
+                <!-- Generate disable_collisions for each link pair -->
+                <!-- Note: xacro doesn't support while loops, so we need to handle each item individually -->
+                <!-- For tools with multiple link pairs, we'll handle up to 10 pairs (should be enough) -->
+                <xacro:property name="collision_count" value="${len(collision_disable_list)}"/>
+                <!-- Handle up to 10 collision pairs -->
+                <xacro:if value="${collision_count > 0}">
+                    <xacro:property name="pair0" value="${collision_disable_list[0]}"/>
+                    <disable_collisions link1="${arm_id}_${pair0['link1']}" link2="${arm_id}_${pair0['link2']}" reason="${pair0.get('reason', 'Adjacent')}"/>
+                </xacro:if>
+                <xacro:if value="${collision_count > 1}">
+                    <xacro:property name="pair1" value="${collision_disable_list[1]}"/>
+                    <disable_collisions link1="${arm_id}_${pair1['link1']}" link2="${arm_id}_${pair1['link2']}" reason="${pair1.get('reason', 'Adjacent')}"/>
+                </xacro:if>
+                <xacro:if value="${collision_count > 2}">
+                    <xacro:property name="pair2" value="${collision_disable_list[2]}"/>
+                    <disable_collisions link1="${arm_id}_${pair2['link1']}" link2="${arm_id}_${pair2['link2']}" reason="${pair2.get('reason', 'Adjacent')}"/>
+                </xacro:if>
+                <xacro:if value="${collision_count > 3}">
+                    <xacro:property name="pair3" value="${collision_disable_list[3]}"/>
+                    <disable_collisions link1="${arm_id}_${pair3['link1']}" link2="${arm_id}_${pair3['link2']}" reason="${pair3.get('reason', 'Adjacent')}"/>
+                </xacro:if>
+                <xacro:if value="${collision_count > 4}">
+                    <xacro:property name="pair4" value="${collision_disable_list[4]}"/>
+                    <disable_collisions link1="${arm_id}_${pair4['link1']}" link2="${arm_id}_${pair4['link2']}" reason="${pair4.get('reason', 'Adjacent')}"/>
+                </xacro:if>
+                <xacro:if value="${collision_count > 5}">
+                    <xacro:property name="pair5" value="${collision_disable_list[5]}"/>
+                    <disable_collisions link1="${arm_id}_${pair5['link1']}" link2="${arm_id}_${pair5['link2']}" reason="${pair5.get('reason', 'Adjacent')}"/>
+                </xacro:if>
+                <xacro:if value="${collision_count > 6}">
+                    <xacro:property name="pair6" value="${collision_disable_list[6]}"/>
+                    <disable_collisions link1="${arm_id}_${pair6['link1']}" link2="${arm_id}_${pair6['link2']}" reason="${pair6.get('reason', 'Adjacent')}"/>
+                </xacro:if>
+                <xacro:if value="${collision_count > 7}">
+                    <xacro:property name="pair7" value="${collision_disable_list[7]}"/>
+                    <disable_collisions link1="${arm_id}_${pair7['link1']}" link2="${arm_id}_${pair7['link2']}" reason="${pair7.get('reason', 'Adjacent')}"/>
+                </xacro:if>
+                <xacro:if value="${collision_count > 8}">
+                    <xacro:property name="pair8" value="${collision_disable_list[8]}"/>
+                    <disable_collisions link1="${arm_id}_${pair8['link1']}" link2="${arm_id}_${pair8['link2']}" reason="${pair8.get('reason', 'Adjacent')}"/>
+                </xacro:if>
+                <xacro:if value="${collision_count > 9}">
+                    <xacro:property name="pair9" value="${collision_disable_list[9]}"/>
+                    <disable_collisions link1="${arm_id}_${pair9['link1']}" link2="${arm_id}_${pair9['link2']}" reason="${pair9.get('reason', 'Adjacent')}"/>
+                </xacro:if>
+            </xacro:if>
+        </xacro:unless>
+    </xacro:macro>
+    <!-- Generate collision disables for arm1 and arm2 tools -->
+    <xacro:generate_tool_collision_disable arm_id="arm1" tool_name="$(arg arm1_tool)"/>
+    <xacro:generate_tool_collision_disable arm_id="arm2" tool_name="$(arg arm2_tool)"/>
 </robot>
