Commit message: 20251221更新magnetometer_array，更新三臂协作bringup

File: src/zlab_robots_descriptions/zlab_tools_description/magnetometer_array/urdf/magnetometer_array_macro.xacro (robot description, xacro)
@@ -5,11 +5,11 @@
       <parent link="${parent}"/>
       <child link="${prefix}magnetometer_base_link"/>
-      <origin xyz="0 0 0" rpy="0 0 0"/>
+      <origin xyz="0 0 0" rpy="0 0 ${pi/2}"/>
     </joint>
     <link name="${prefix}magnetometer_base_link">
       <inertial>
-        <origin xyz="-2.07166456524356E-07 0.0021604655211999 0.0362476651991424" rpy="0 0 0" />
-        <mass value="0.0332054242847689" />
-        <inertia ixx="5.63055976294825E-05" ixy="5.92198383575024E-12" ixz="6.68013595190353E-10" iyy="5.96936991935191E-05" iyz="-2.03045562894017E-06" izz="1.14540668478137E-05" />
+        <origin xyz="2.0717E-07 0.0021605 -0.036248" rpy="0 0 0" />
+        <mass value="0.033205" />
+        <inertia ixx="5.6306E-05" ixy="-5.922E-12" ixz="6.6801E-10" iyy="5.9694E-05" iyz="2.0305E-06" izz="1.1454E-05" />
       </inertial>
       <visual>
@@ -31,7 +31,7 @@
     <link name="${prefix}magnetometer_tcp_link">
       <inertial>
-        <origin xyz="-1.2355E-05 0.0019209 -0.1507" rpy="0 0 0" />
-        <mass value="0.035468" />
-        <inertia ixx="7.6653E-05" ixy="1.9231E-11" ixz="3.8778E-08" iyy="8.0393E-05" iyz="-2.0188E-06" izz="1.1822E-05" />
+        <origin xyz="-0.00019067 0.0018908 -0.060443" rpy="0 0 0" />
+        <mass value="0.0022623" />
+        <inertia ixx="3.3502E-07" ixy="6.2726E-20" ixz="-6.8291E-10" iyy="4.1094E-07" iyz="1.8218E-19" izz="8.7172E-08" />
       </inertial>
       <visual>
@@ -41,5 +41,5 @@
         </geometry>
         <material name="">
-          <color rgba="1 1 1 1" />
+          <color rgba="0.75294 0.75294 0.75294 1" />
         </material>
       </visual>
@@ -51,6 +51,6 @@
       </collision>
     </link>
-    <joint name="${prefix}magnetometer_tcp_joint" type="fixed">
-      <origin xyz="0 0.00023753 0.19309" rpy="0 0 0" />
+    <joint name="${prefix}magnetometer_joint" type="fixed">
+      <origin xyz="0 0.00023753 -0.19309" rpy="3.1416 0 3.1416" />
       <parent link="${prefix}magnetometer_base_link" />
       <child link="${prefix}magnetometer_tcp_link" />
