Commit message: 20251229 修复工具前缀问题

File: src/zlab_robots_descriptions/zlab_tools_description/tools/electronic_magnet/urdf/electronic_magnet.urdf (robot description, URDF)
Before this commit: robot electronic_magnet, 3 links, 2 joints
Links:
- link em_base_link: geometry collision mesh filename=package://zlab_tools_description/tools/electronic_magnet/me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; visual mesh filename=package://zlab_tools_description/tools/electronic_magnet/me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
- link em_ee_link: geometry collision mesh filename=package://zlab_tools_description/tools/electronic_magnet/me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; visual mesh filename=package://zlab_tools_description/tools/electronic_magnet/me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
- link em_tcp_link: geometry collision mesh filename=package://zlab_tools_description/tools/electronic_magnet/me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; visual mesh filename=package://zlab_tools_description/tools/electronic_magnet/me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

File: src/zlab_robots_descriptions/zlab_tools_description/tools/electronic_magnet/urdf/electronic_magnet.urdf.xacro (robot description, xacro)
@@ -29,5 +29,5 @@
       <geometry>
         <mesh
-          filename="package://zlab_tools_description/electronic_magnet/meshes/visual/em_base_link.STL" />
+          filename="package://zlab_tools_description/tools/electronic_magnet/meshes/visual/em_base_link.STL" />
       </geometry>
       <material
@@ -43,5 +43,5 @@
       <geometry>
         <mesh
-          filename="package://zlab_tools_description/electronic_magnet/meshes/collision/em_base_link.STL" />
+          filename="package://zlab_tools_description/tools/electronic_magnet/meshes/collision/em_base_link.STL" />
       </geometry>
     </collision>
@@ -68,5 +68,5 @@
       <geometry>
         <mesh
-          filename="package://zlab_tools_description/electronic_magnet/meshes/visual/em_tcp_link.STL" />
+          filename="package://zlab_tools_description/tools/electronic_magnet/meshes/visual/em_tcp_link.STL" />
       </geometry>
       <material
@@ -82,5 +82,5 @@
       <geometry>
         <mesh
-          filename="package://zlab_tools_description/electronic_magnet/meshes/collision/em_tcp_link.STL" />
+          filename="package://zlab_tools_description/tools/electronic_magnet/meshes/collision/em_tcp_link.STL" />
       </geometry>
     </collision>
@@ -118,5 +118,5 @@
       <geometry>
         <mesh
-          filename="package://zlab_tools_description/electronic_magnet/meshes/visual/em_ee_link.STL" />
+          filename="package://zlab_tools_description/tools/electronic_magnet/meshes/visual/em_ee_link.STL" />
       </geometry>
       <material
@@ -132,5 +132,5 @@
       <geometry>
         <mesh
-          filename="package://zlab_tools_description/electronic_magnet/meshes/collision/em_ee_link.STL" />
+          filename="package://zlab_tools_description/tools/electronic_magnet/meshes/collision/em_ee_link.STL" />
       </geometry>
     </collision>

File: src/zlab_robots_descriptions/zlab_tools_description/tools/electronic_magnet/urdf/electronic_magnet_macro.xacro (robot description, xacro)
@@ -16,5 +16,5 @@
         <origin xyz="0 0 0" rpy="0 0 0" />
         <geometry>
-          <mesh filename="package://zlab_tools_description/electronic_magnet/meshes/visual/em_base_link.STL" />
+          <mesh filename="package://zlab_tools_description/tools/electronic_magnet/meshes/visual/em_base_link.STL" />
         </geometry>
         <material name="">
@@ -25,5 +25,5 @@
         <origin xyz="0 0 0" rpy="0 0 0" />
         <geometry>
-          <mesh filename="package://zlab_tools_description/electronic_magnet/meshes/collision/em_base_link.STL" />
+          <mesh filename="package://zlab_tools_description/tools/electronic_magnet/meshes/collision/em_base_link.STL" />
         </geometry>
       </collision>
@@ -38,5 +38,5 @@
         <origin xyz="0 0 0" rpy="0 0 0" />
         <geometry>
-          <mesh filename="package://zlab_tools_description/electronic_magnet/meshes/visual/em_tcp_link.STL" />
+          <mesh filename="package://zlab_tools_description/tools/electronic_magnet/meshes/visual/em_tcp_link.STL" />
         </geometry>
         <material name="">
@@ -47,5 +47,5 @@
         <origin xyz="0 0 0" rpy="0 0 0" />
         <geometry>
-          <mesh filename="package://zlab_tools_description/electronic_magnet/meshes/collision/em_tcp_link.STL" />
+          <mesh filename="package://zlab_tools_description/tools/electronic_magnet/meshes/collision/em_tcp_link.STL" />
         </geometry>
       </collision>
@@ -65,5 +65,5 @@
         <origin xyz="0 0 0" rpy="0 0 0" />
         <geometry>
-          <mesh filename="package://zlab_tools_description/electronic_magnet/meshes/visual/em_ee_link.STL" />
+          <mesh filename="package://zlab_tools_description/tools/electronic_magnet/meshes/visual/em_ee_link.STL" />
         </geometry>
         <material name="">
@@ -74,5 +74,5 @@
         <origin xyz="0 0 0" rpy="0 0 0" />
         <geometry>
-          <mesh filename="package://zlab_tools_description/electronic_magnet/meshes/collision/em_ee_link.STL" />
+          <mesh filename="package://zlab_tools_description/tools/electronic_magnet/meshes/collision/em_ee_link.STL" />
         </geometry>
       </collision>

File: src/zlab_robots_descriptions/zlab_tools_description/tools/magnetic_sensor_bracket/urdf/bracket.urdf.xacro (robot description, xacro)
@@ -18,5 +18,5 @@
       <origin xyz="0 0 0" rpy="0 0 0" />
       <geometry>
-        <mesh filename="package://zlab_tools_description/magnetic_sensor_bracket/meshes/bracket_base_link.STL" />
+        <mesh filename="package://zlab_tools_description/tools/magnetic_sensor_bracket/meshes/bracket_base_link.STL" />
       </geometry>
       <material name="">
@@ -27,5 +27,5 @@
       <origin xyz="0 0 0" rpy="0 0 0" />
       <geometry>
-        <mesh filename="package://zlab_tools_description/magnetic_sensor_bracket/meshes/bracket_base_link.STL" />
+        <mesh filename="package://zlab_tools_description/tools/magnetic_sensor_bracket/meshes/bracket_base_link.STL" />
       </geometry>
     </collision>

File: src/zlab_robots_descriptions/zlab_tools_description/tools/magnetic_sensor_bracket/urdf/bracket_macro.xacro (robot description, xacro)
@@ -16,5 +16,5 @@
         <origin xyz="0 0 0" rpy="0 0 0" />
         <geometry>
-          <mesh filename="package://zlab_tools_description/magnetic_sensor_bracket/meshes/bracket_base_link.STL" />
+          <mesh filename="package://zlab_tools_description/tools/magnetic_sensor_bracket/meshes/bracket_base_link.STL" />
         </geometry>
         <material name="">
@@ -25,5 +25,5 @@
         <origin xyz="0 0 0" rpy="0 0 0" />
         <geometry>
-          <mesh filename="package://zlab_tools_description/magnetic_sensor_bracket/meshes/bracket_base_link.STL" />
+          <mesh filename="package://zlab_tools_description/tools/magnetic_sensor_bracket/meshes/bracket_base_link.STL" />
         </geometry>
       </collision>

File: src/zlab_robots_descriptions/zlab_tools_description/tools/magnetometer_array/urdf/magnetometer_array.urdf.xacro (robot description, xacro)
@@ -1,5 +1,5 @@
 <?xml version="1.0" encoding="utf-8"?>
 <robot name="magnetometer_array" xmlns:xacro="http://www.ros.org/wiki/xacro">
-  <xacro:include filename="$(find zlab_tools_description)/magnetometer_array/urdf/magnetometer_array_macro.xacro"/>
+  <xacro:include filename="$(find zlab_tools_description)/tools/magnetometer_array/urdf/magnetometer_array_macro.xacro"/>
   <link name="world"/>
   <xacro:magnetometer_array prefix="" parent="world"/>

File: src/zlab_robots_descriptions/zlab_tools_description/tools/magnetometer_array/urdf/magnetometer_array_macro.xacro (robot description, xacro)
@@ -16,5 +16,5 @@
         <origin xyz="0 0 0" rpy="0 0 0" />
         <geometry>
-          <mesh filename="package://zlab_tools_description/magnetometer_array/meshes/magnetometer_base_link.STL" />
+          <mesh filename="package://zlab_tools_description/tools/magnetometer_array/meshes/magnetometer_base_link.STL" />
         </geometry>
         <material name="">
@@ -25,5 +25,5 @@
         <origin xyz="0 0 0" rpy="0 0 0" />
         <geometry>
-          <mesh filename="package://zlab_tools_description/magnetometer_array/meshes/magnetometer_base_link.STL" />
+          <mesh filename="package://zlab_tools_description/tools/magnetometer_array/meshes/magnetometer_base_link.STL" />
         </geometry>
       </collision>
@@ -38,5 +38,5 @@
         <origin xyz="0 0 0" rpy="0 0 0" />
         <geometry>
-          <mesh filename="package://zlab_tools_description/magnetometer_array/meshes/magnetometer_tcp_link.STL" />
+          <mesh filename="package://zlab_tools_description/tools/magnetometer_array/meshes/magnetometer_tcp_link.STL" />
         </geometry>
         <material name="">
@@ -47,5 +47,5 @@
         <origin xyz="0 0 0" rpy="0 0 0" />
         <geometry>
-          <mesh filename="package://zlab_tools_description/magnetometer_array/meshes/magnetometer_tcp_link.STL" />
+          <mesh filename="package://zlab_tools_description/tools/magnetometer_array/meshes/magnetometer_tcp_link.STL" />
         </geometry>
       </collision>

File: src/zlab_robots_descriptions/zlab_tools_description/tools/permanent_magnet/urdf/permanent_magnet_macro.xacro (robot description, xacro)
@@ -16,5 +16,5 @@
         <origin xyz="0 0 0" rpy="0 0 0" />
         <geometry>
-          <mesh filename="package://zlab_tools_description/permanent_magnet/meshes/visual/pm_base_link.STL" />
+          <mesh filename="package://zlab_tools_description/tools/permanent_magnet/meshes/visual/pm_base_link.STL" />
         </geometry>
         <material name="">
@@ -25,5 +25,5 @@
         <origin xyz="0 0 0" rpy="0 0 0" />
         <geometry>
-          <mesh filename="package://zlab_tools_description/permanent_magnet/meshes/collision/pm_base_link.STL" />
+          <mesh filename="package://zlab_tools_description/tools/permanent_magnet/meshes/collision/pm_base_link.STL" />
         </geometry>
       </collision>
@@ -38,5 +38,5 @@
         <origin xyz="0 0 0" rpy="0 0 0" />
         <geometry>
-          <mesh filename="package://zlab_tools_description/permanent_magnet/meshes/visual/pm_tcp_link.STL" />
+          <mesh filename="package://zlab_tools_description/tools/permanent_magnet/meshes/visual/pm_tcp_link.STL" />
         </geometry>
         <material name="">
@@ -47,5 +47,5 @@
         <origin xyz="0 0 0" rpy="0 0 0" />
         <geometry>
-          <mesh filename="package://zlab_tools_description/permanent_magnet/meshes/collision/pm_tcp_link.STL" />
+          <mesh filename="package://zlab_tools_description/tools/permanent_magnet/meshes/collision/pm_tcp_link.STL" />
         </geometry>
       </collision>

File: src/zlab_robots_descriptions/zlab_tools_description/urdf/tool_loader.xacro (robot description, xacro)
@@ -116,5 +116,5 @@
             <xacro:property name="mount_rpy" value="${mount_offset['rpy']}"/>
             <!-- 构建工具文件路径 -->
-            <xacro:property name="tool_file_path" value="$(find zlab_tools_description)/${tool_name}/${urdf_file}"/>
+            <xacro:property name="tool_file_path" value="$(find zlab_tools_description)/tools/${tool_name}/${urdf_file}"/>
             <!-- 设置全局变量供工具xacro文件使用 -->
             <xacro:property name="tool_arm_id" value="${arm_id}"/>

File: src/zlab_robots_descriptions/zlab_tools_description/urdf/zlab_tools.xacro (robot description, xacro)
@@ -1,29 +1,27 @@
 <?xml version="1.0" encoding="utf-8"?>
 <robot xmlns:xacro="http://www.ros.org/wiki/xacro">
-  <!-- Include all tool macros -->
-  <xacro:include filename="$(find zlab_tools_description)/electronic_magnet/urdf/electronic_magnet_macro.xacro"/>
-  <xacro:include filename="$(find zlab_tools_description)/permanent_magnet/urdf/permanent_magnet_macro.xacro"/>
-  <xacro:include filename="$(find zlab_tools_description)/magnetic_sensor_bracket/urdf/bracket_macro.xacro"/>
-  <xacro:include filename="$(find zlab_tools_description)/magnetometer_array/urdf/magnetometer_array_macro.xacro"/>
+  <!--
+    工具加载系统 - 基于配置文件的动态加载
+    新增工具时，只需在工具目录下创建 config/tool.yaml 配置文件即可
+    无需修改此文件
+  -->
+  <!-- 加载工具加载器 -->
+  <xacro:include filename="$(find zlab_tools_description)/urdf/tool_loader.xacro" />
   <!-- Main macro to load a tool based on name -->
+  <!-- 此宏从工具配置文件自动加载工具，支持动态扩展 -->
   <xacro:macro name="load_tool" params="tool_name prefix parent">
-    <!-- Check for predefined tools -->
-    <xacro:if value="${tool_name == 'electronic_magnet'}">
-       <xacro:electronic_magnet prefix="${prefix}" parent="${parent}"/>
+    <xacro:if value="${tool_name == 'none'}">
+      <!-- No tool loaded -->
     </xacro:if>
-    <xacro:unless value="${tool_name == 'electronic_magnet'}">
-      <xacro:if value="${tool_name == 'permanent_magnet'}">
-         <xacro:permanent_magnet prefix="${prefix}" parent="${parent}"/>
-      </xacro:if>
-      <xacro:unless value="${tool_name == 'permanent_magnet'}">
-        <xacro:if value="${tool_name == 'magnetic_sensor_bracket'}">
-           <xacro:magnetic_sensor_bracket prefix="${prefix}" parent="${parent}"/>
-        </xacro:if>
-        <xacro:unless value="${tool_name == 'magnetic_sensor_bracket'}">
-          <xacro:if value="${tool_name == 'magnetometer_array'}">
-             <xacro:magnetometer_array prefix="${prefix}" parent="${parent}"/>
-          </xacro:if>
-        </xacro:unless>
-      </xacro:unless>
+    <xacro:unless value="${tool_name == 'none'}">
+      <!-- 加载工具配置文件 -->
+      <xacro:property name="tool_config_file" value="$(find zlab_tools_description)/tools/${tool_name}/config/tool.yaml"/>
+      <xacro:property name="tool_config" value="${xacro.load_yaml(tool_config_file)}"/>
+      <!-- 使用配置加载工具 -->
+      <xacro:load_tool_from_config
+          arm_id="${prefix}"
+          tool_name="${tool_name}"
+          tool_config="${tool_config}"
+          parent="${parent}" />
     </xacro:unless>
   </xacro:macro>
