Commit message: 20251220修复fr5单臂工具，fr5双臂工具，diana7工具还待修复

File: src/zlab_robots_descriptions/diana7_description/urdf/diana7.urdf.xacro (robot description, xacro)
@@ -1,4 +1,8 @@
 <?xml version="1.0" encoding="utf-8"?>
 <robot xmlns:xacro="http://wiki.ros.org/xacro" name="diana7">
+  <!-- Tool Argument -->
+  <xacro:arg name="tool_name" default="none"/>
+  <!-- Include Tool Library -->
+  <xacro:include filename="$(find zlab_tools_description)/urdf/tools_library.xacro" />
   <link name="world">
       <origin
@@ -374,3 +378,5 @@
       velocity="3.14" />
   </joint>
+  <!-- Load Tool -->
+  <xacro:load_tool tool_name="$(arg tool_name)" prefix="" parent="link_7"/>
 </robot>

File: src/zlab_robots_descriptions/fr5_description/fr5_description/urdf/fr.xacro (robot description, xacro)
@@ -6,19 +6,8 @@
     <!-- 定义工具参数 -->
     <xacro:arg name="tool_name" default="none"/>
-    <!-- 加载工具配置 -->
-    <!-- 从工具包加载工具配置 -->
-    <!-- 如果tool_name为"none"，则不加载工具配置，使用空字典 -->
-    <xacro:property name="tool_name_arg" value="$(arg tool_name)"/>
-    <xacro:property name="tool_config" value="{}"/>
-    <!-- 只有当tool_name不为"none"时才加载工具配置 -->
-    <xacro:unless value="${tool_name_arg == 'none'}">
-        <!-- 从工具包加载工具配置 -->
-        <xacro:property name="tool_package_path"
-                        value="$(find fr5_description)/tools/${tool_name_arg}/config/tool.yaml"/>
-        <xacro:property name="tool_config"
-                        value="${xacro.load_yaml(tool_package_path)}"/>
-    </xacro:unless>
-    <!-- 添加虚拟根链接 -->
-    <xacro:include filename="$(find fr5_description)/fr/urdf/fr5_library.xacro" />
+    <!-- 加载工具库 -->
+    <xacro:include filename="$(find zlab_tools_description)/urdf/tools_library.xacro" />
+    <!-- 加载机械臂库 -->
+    <xacro:include filename="$(find fr5_description)/fr5_description/urdf/fr5_library.xacro" />
     <!-- 添加虚拟根链接 -->
     <link name="world" />
@@ -29,6 +18,8 @@
         xyz="0 0 0"
         rpy="0 0 0"
-        tool_name="$(arg tool_name)"
-        tool_config="${tool_config}" />
+        tool_name="none"
+        tool_config="{}" />
+    <!-- 加载工具 -->
+    <xacro:load_tool tool_name="$(arg tool_name)" prefix="$(arg arm_id)_" parent="$(arg arm_id)_ee_link"/>
     <xacro:gazebo-joint joint="$(arg arm_id)_j1" />
     <xacro:gazebo-joint joint="$(arg arm_id)_j2" />

File: src/zlab_robots_descriptions/fr5_description/fr5_description/urdf/tool_loader.xacro (robot description, xacro)
@@ -116,5 +116,5 @@
             <xacro:property name="mount_rpy" value="${mount_offset['rpy']}"/>
             <!-- 构建工具文件路径 -->
-            <xacro:property name="tool_file_path" value="$(find fr5_description)/tools/${tool_name}/${urdf_file}"/>
+            <xacro:property name="tool_file_path" value="$(find zlab_tools_description)/${tool_name}/${urdf_file}"/>
             <!-- 设置全局变量供工具xacro文件使用 -->
             <xacro:property name="tool_arm_id" value="${arm_id}"/>

File: src/zlab_robots_descriptions/fr5_description/fr5_description/urdf/zlab_dual_arms.xacro (robot description, xacro)
@@ -13,25 +13,9 @@
     <xacro:arg name="arm2_rpy" default=""/>
     <!-- 加载机械臂库 -->
-    <xacro:include filename="$(find fr5_description)/fr/urdf/fr5_library.xacro" />
+    <xacro:include filename="$(find fr5_description)/fr5_description/urdf/fr5_library.xacro" />
+    <!-- 加载工具库 -->
+    <xacro:include filename="$(find zlab_tools_description)/urdf/tools_library.xacro" />
     <!-- 创建世界坐标系 -->
     <link name="world" />
-    <!-- ========== 加载 arm1 工具配置 ========== -->
-    <xacro:property name="arm1_tool_name_arg" value="$(arg arm1_tool)"/>
-    <xacro:property name="arm1_tool_config" value="{}"/>
-    <xacro:unless value="${arm1_tool_name_arg == 'none'}">
-        <xacro:property name="arm1_tool_package_path"
-                        value="$(find fr5_description)/tools/${arm1_tool_name_arg}/config/tool.yaml"/>
-        <xacro:property name="arm1_tool_config"
-                        value="${xacro.load_yaml(arm1_tool_package_path)}"/>
-    </xacro:unless>
-    <!-- ========== 加载 arm2 工具配置 ========== -->
-    <xacro:property name="arm2_tool_name_arg" value="$(arg arm2_tool)"/>
-    <xacro:property name="arm2_tool_config" value="{}"/>
-    <xacro:unless value="${arm2_tool_name_arg == 'none'}">
-        <xacro:property name="arm2_tool_package_path"
-                        value="$(find fr5_description)/tools/${arm2_tool_name_arg}/config/tool.yaml"/>
-        <xacro:property name="arm2_tool_config"
-                        value="${xacro.load_yaml(arm2_tool_package_path)}"/>
-    </xacro:unless>
     <!-- ========== 设置arm2位置 ========== -->
     <!-- 默认值：arm1在原点，arm2在右边1米处 -->
@@ -72,6 +56,8 @@
         xyz="$(arg arm1_xyz)"
         rpy="$(arg arm1_rpy)"
-        tool_name="$(arg arm1_tool)"
-        tool_config="${arm1_tool_config}" />
+        tool_name="none"
+        tool_config="{}" />
+    <!-- 加载 arm1 工具 -->
+    <xacro:load_tool tool_name="$(arg arm1_tool)" prefix="arm1_" parent="arm1_ee_link"/>
     <xacro:gazebo-joint joint="arm1_j1" />
     <xacro:gazebo-joint joint="arm1_j2" />
@@ -86,6 +72,8 @@
         xyz="${arm2_xyz_final}"
         rpy="${arm2_rpy_final}"
-        tool_name="$(arg arm2_tool)"
-        tool_config="${arm2_tool_config}" />
+        tool_name="none"
+        tool_config="{}" />
+    <!-- 加载 arm2 工具 -->
+    <xacro:load_tool tool_name="$(arg arm2_tool)" prefix="arm2_" parent="arm2_ee_link"/>
     <xacro:gazebo-joint joint="arm2_j1" />
     <xacro:gazebo-joint joint="arm2_j2" />

File: src/zlab_robots_descriptions/fr5_description/fr5_description/urdf/zlab_triple_arms.xacro (robot description, xacro)
@@ -11,7 +11,12 @@
     <xacro:arg name="arm2_xyz" default="1.5 0.4 0"/>
     <xacro:arg name="arm2_rpy" default="0 0 0"/>
+    <!-- Arguments for tools -->
+    <xacro:arg name="arm1_tool" default="none"/>
+    <xacro:arg name="arm2_tool" default="none"/>
+    <xacro:arg name="diana7_tool" default="none"/>
     <!-- Include Macros -->
     <xacro:include filename="$(find fr5_description)/fr5_description/urdf/fr5_library.xacro" />
     <xacro:include filename="$(find diana7_description)/urdf/diana7_macro.xacro" />
+    <xacro:include filename="$(find zlab_tools_description)/urdf/tools_library.xacro" />
     <!-- World Link -->
     <link name="world" />
@@ -20,7 +25,13 @@
         <origin xyz="$(arg diana7_xyz)" rpy="$(arg diana7_rpy)"/>
     </xacro:diana7_robot>
+    <!-- Load Tool for Diana7 -->
+    <xacro:load_tool tool_name="$(arg diana7_tool)" prefix="diana7_" parent="diana7_link_7"/>
     <!-- Instantiate FR5 Arm 1 -->
-    <xacro:fr arm_id="arm1" connected_to="world" xyz="$(arg arm1_xyz)" rpy="$(arg arm1_rpy)"/>
+    <xacro:fr arm_id="arm1" connected_to="world" xyz="$(arg arm1_xyz)" rpy="$(arg arm1_rpy)" tool_name="none"/>
+    <!-- Load Tool for Arm 1 -->
+    <xacro:load_tool tool_name="$(arg arm1_tool)" prefix="arm1_" parent="arm1_ee_link"/>
     <!-- Instantiate FR5 Arm 2 -->
-    <xacro:fr arm_id="arm2" connected_to="world" xyz="$(arg arm2_xyz)" rpy="$(arg arm2_rpy)"/>
+    <xacro:fr arm_id="arm2" connected_to="world" xyz="$(arg arm2_xyz)" rpy="$(arg arm2_rpy)" tool_name="none"/>
+    <!-- Load Tool for Arm 2 -->
+    <xacro:load_tool tool_name="$(arg arm2_tool)" prefix="arm2_" parent="arm2_ee_link"/>
 </robot>

File: src/zlab_robots_moveit_config/fr5_dual_moveit_config/config/zlab_dual_arms.srdf.xacro (robot description, xacro)
@@ -204,5 +204,5 @@
         <xacro:unless value="${tool_name == 'none'}">
             <xacro:property name="tool_config_path"
-                            value="$(find fr5_description)/tools/${tool_name}/config/tool.yaml"/>
+                            value="$(find zlab_tools_description)/${tool_name}/config/tool.yaml"/>
             <xacro:property name="tool_config"
                             value="${xacro.load_yaml(tool_config_path)}"/>

File: src/zlab_robots_moveit_config/fr5_single_moveit_config/config/fr.srdf.xacro (robot description, xacro)
@@ -93,5 +93,5 @@
         <xacro:unless value="${tool_name == 'none'}">
             <xacro:property name="tool_config_path"
-                            value="$(find fr5_description)/tools/${tool_name}/config/tool.yaml"/>
+                            value="$(find zlab_tools_description)/${tool_name}/config/tool.yaml"/>
             <xacro:property name="tool_config"
                             value="${xacro.load_yaml(tool_config_path)}"/>

Commit message: 20251221新增diana7底座和camera_calibration

File: src/zlab_robots_descriptions/diana7_description/urdf/diana7.urdf.xacro (robot description, xacro)
@@ -10,4 +10,61 @@
         rpy="0 0 0" />
   </link>
+  <!-- Optional base assembly (default: included) -->
+  <link name="diana7_base_link">
+    <inertial>
+      <origin xyz="-0.0554345295309022 -0.000128426199742461 0.380705746455594" rpy="0 0 0" />
+      <mass value="94.0798220497049" />
+      <inertia ixx="11.6812698745749" ixy="0.000483119972220811" ixz="0.0946190239054891"
+              iyy="10.7627891849386" iyz="0.00470248742831138" izz="8.47191505976327" />
+    </inertial>
+    <visual>
+      <origin xyz="0 0 0" rpy="0 0 0" />
+      <geometry>
+        <mesh filename="package://diana7_description/meshes/base/diana7_base_link.STL" />
+      </geometry>
+      <material name="">
+        <color rgba="0.8 0.8 0.8 1" />
+      </material>
+    </visual>
+    <collision>
+      <origin xyz="0 0 0" rpy="0 0 0" />
+      <geometry>
+        <mesh filename="package://diana7_description/meshes/base/diana7_base_link.STL" />
+      </geometry>
+    </collision>
+  </link>
+  <link name="diana7_base_flange_link">
+    <inertial>
+      <origin xyz="-0.039655 0.021372 -0.3992" rpy="0 0 0" />
+      <mass value="94.08" />
+      <inertia ixx="11.681" ixy="0.00048312" ixz="0.094619" iyy="10.763"
+              iyz="0.0047025" izz="8.4719" />
+    </inertial>
+    <visual>
+      <origin xyz="0 0 0" rpy="0 0 0" />
+      <geometry>
+        <mesh filename="package://diana7_description/meshes/base/diana7_base_flange_link.STL" />
+      </geometry>
+      <material name="">
+        <color rgba="0.8 0.8 0.8 1" />
+      </material>
+    </visual>
+    <collision>
+      <origin xyz="0 0 0" rpy="0 0 0" />
+      <geometry>
+        <mesh filename="package://diana7_description/meshes/base/diana7_base_flange_link.STL" />
+      </geometry>
+    </collision>
+  </link>
+  <joint name="world_to_diana7_base" type="fixed">
+    <origin xyz="0 0 0" rpy="0 0 0" />
+    <parent link="world" />
+    <child link="diana7_base_link" />
+  </joint>
+  <joint name="diana7_base_to_flange" type="fixed">
+    <origin xyz="-0.015779 -0.0215 0.7799" rpy="0 0 0" />
+    <parent link="diana7_base_link" />
+    <child link="diana7_base_flange_link" />
+  </joint>
   <link name="base_link">
     <inertial>
@@ -45,6 +102,7 @@
   </link>
   <joint name="base_joint" type="fixed">
-    <parent link="world"/>
+    <parent link="diana7_base_flange_link"/>
     <child link="base_link"/>
+    <origin xyz="0 0 0" rpy="0 0 0" />
   </joint>
   <link name="link_1">

File: src/zlab_robots_descriptions/diana7_description/urdf/diana7_macro.xacro (robot description, xacro)
@@ -36,8 +36,64 @@
       </collision>
     </link>
+    <link name="${prefix}pedestal_link">
+      <inertial>
+        <origin xyz="-0.0554345295309022 -0.000128426199742461 0.380705746455594" rpy="0 0 0" />
+        <mass value="94.0798220497049" />
+        <inertia ixx="11.6812698745749" ixy="0.000483119972220811" ixz="0.0946190239054891"
+              iyy="10.7627891849386" iyz="0.00470248742831138" izz="8.47191505976327" />
+      </inertial>
+      <visual>
+        <origin xyz="0 0 0" rpy="0 0 0" />
+        <geometry>
+          <mesh filename="package://diana7_description/meshes/base/diana7_base_link.STL" />
+        </geometry>
+        <material name="">
+          <color rgba="0.8 0.8 0.8 1" />
+        </material>
+      </visual>
+      <collision>
+        <origin xyz="0 0 0" rpy="0 0 0" />
+        <geometry>
+          <mesh filename="package://diana7_description/meshes/base/diana7_base_link.STL" />
+        </geometry>
+      </collision>
+    </link>
+    <link name="${prefix}pedestal_flange_link">
+      <inertial>
+        <origin xyz="-0.039655 0.021372 -0.3992" rpy="0 0 0" />
+        <mass value="94.08" />
+        <inertia ixx="11.681" ixy="0.00048312" ixz="0.094619" iyy="10.763"
+              iyz="0.0047025" izz="8.4719" />
+      </inertial>
+      <visual>
+        <origin xyz="0 0 0" rpy="0 0 0" />
+        <geometry>
+          <mesh filename="package://diana7_description/meshes/base/diana7_base_flange_link.STL" />
+        </geometry>
+        <material name="">
+          <color rgba="0.8 0.8 0.8 1" />
+        </material>
+      </visual>
+      <collision>
+        <origin xyz="0 0 0" rpy="0 0 0" />
+        <geometry>
+          <mesh filename="package://diana7_description/meshes/base/diana7_base_flange_link.STL" />
+        </geometry>
+      </collision>
+    </link>
+    <joint name="${prefix}pedestal_joint" type="fixed">
+      <parent link="${parent}"/>
+      <child link="${prefix}pedestal_link"/>
+      <xacro:insert_block name="origin" />
+    </joint>
+    <joint name="${prefix}pedestal_to_flange" type="fixed">
+      <origin xyz="-0.015779 -0.0215 0.7799" rpy="0 0 0" />
+      <parent link="${prefix}pedestal_link" />
+      <child link="${prefix}pedestal_flange_link" />
+    </joint>
     <joint name="${prefix}base_joint" type="fixed">
-      <parent link="${parent}"/>
+      <parent link="${prefix}pedestal_flange_link"/>
       <child link="${prefix}base_link"/>
-      <xacro:insert_block name="origin" />
+      <origin xyz="0 0 0" rpy="0 0 0" />
     </joint>
     <link name="${prefix}link_1">

File: src/zlab_robots_moveit_config/triple_arm_moveit_config/config/zlab_triple_arms.srdf.xacro (robot description, xacro)
@@ -124,4 +124,7 @@
     <disable_collisions link1="arm2_j5_link" link2="arm2_j6_link" reason="Adjacent"/>
     <!-- Diana7 Internal -->
+    <disable_collisions link1="diana7_pedestal_link" link2="diana7_pedestal_flange_link" reason="Adjacent" />
+    <disable_collisions link1="diana7_pedestal_flange_link" link2="diana7_base_link" reason="Adjacent" />
+    <disable_collisions link1="diana7_pedestal_link" link2="diana7_base_link" reason="User" />
     <disable_collisions link1="diana7_base_link" link2="diana7_link_1" reason="Adjacent" />
     <disable_collisions link1="diana7_link_1" link2="diana7_link_2" reason="Adjacent" />

Commit message: 20251221新增了diana7的底座

File: src/zlab_robots_descriptions/diana7_description/urdf/diana7.urdf.xacro (robot description, xacro)
@@ -13,8 +13,8 @@
   <link name="diana7_base_link">
     <inertial>
-      <origin xyz="-0.0554345295309022 -0.000128426199742461 0.380705746455594" rpy="0 0 0" />
-      <mass value="94.0798220497049" />
-      <inertia ixx="11.6812698745749" ixy="0.000483119972220811" ixz="0.0946190239054891"
-              iyy="10.7627891849386" iyz="0.00470248742831138" izz="8.47191505976327" />
+      <origin xyz="-0.042824 -0.00012843 0.38233" rpy="0 0 0" />
+      <mass value="94.08" />
+      <inertia ixx="11.684" ixy="0.00063824" ixz="-0.011577"
+              iyy="10.763" iyz="0.004684" izz="8.4692" />
     </inertial>
     <visual>
@@ -36,8 +36,8 @@
   <link name="diana7_base_flange_link">
     <inertial>
-      <origin xyz="-0.039655 0.021372 -0.3992" rpy="0 0 0" />
+      <origin xyz="-0.052824 0.021372 -0.39767" rpy="0 0 0" />
       <mass value="94.08" />
-      <inertia ixx="11.681" ixy="0.00048312" ixz="0.094619" iyy="10.763"
-              iyz="0.0047025" izz="8.4719" />
+      <inertia ixx="11.684" ixy="0.00063824" ixz="-0.011577" iyy="10.763"
+              iyz="0.004684" izz="8.4692" />
     </inertial>
     <visual>
@@ -63,5 +63,5 @@
   </joint>
   <joint name="diana7_base_to_flange" type="fixed">
-    <origin xyz="-0.015779 -0.0215 0.7799" rpy="0 0 0" />
+    <origin xyz="0.01 -0.0215 0.78" rpy="0 0 0" />
     <parent link="diana7_base_link" />
     <child link="diana7_base_flange_link" />

File: src/zlab_robots_descriptions/diana7_description/urdf/diana7_macro.xacro (robot description, xacro)
@@ -38,8 +38,8 @@
     <link name="${prefix}pedestal_link">
       <inertial>
-        <origin xyz="-0.0554345295309022 -0.000128426199742461 0.380705746455594" rpy="0 0 0" />
-        <mass value="94.0798220497049" />
-        <inertia ixx="11.6812698745749" ixy="0.000483119972220811" ixz="0.0946190239054891"
-              iyy="10.7627891849386" iyz="0.00470248742831138" izz="8.47191505976327" />
+        <origin xyz="-0.042824 -0.00012843 0.38233" rpy="0 0 0" />
+        <mass value="94.08" />
+        <inertia ixx="11.684" ixy="0.00063824" ixz="-0.011577"
+              iyy="10.763" iyz="0.004684" izz="8.4692" />
       </inertial>
       <visual>
@@ -61,8 +61,8 @@
     <link name="${prefix}pedestal_flange_link">
       <inertial>
-        <origin xyz="-0.039655 0.021372 -0.3992" rpy="0 0 0" />
+        <origin xyz="-0.052824 0.021372 -0.39767" rpy="0 0 0" />
         <mass value="94.08" />
-        <inertia ixx="11.681" ixy="0.00048312" ixz="0.094619" iyy="10.763"
-              iyz="0.0047025" izz="8.4719" />
+        <inertia ixx="11.684" ixy="0.00063824" ixz="-0.011577" iyy="10.763"
+              iyz="0.004684" izz="8.4692" />
       </inertial>
       <visual>
@@ -88,5 +88,5 @@
     </joint>
     <joint name="${prefix}pedestal_to_flange" type="fixed">
-      <origin xyz="-0.015779 -0.0215 0.7799" rpy="0 0 0" />
+      <origin xyz="0.01 -0.0215 0.78" rpy="0 0 0" />
       <parent link="${prefix}pedestal_link" />
       <child link="${prefix}pedestal_flange_link" />

Commit message: 20251225 修复三臂启动问题

File: src/zlab_robots_descriptions/diana7_description/urdf/diana7.urdf.xacro (robot description, xacro)
@@ -140,5 +140,5 @@
     </collision>
   </link>
-  <joint name="joint_1" type="revolute">
+  <joint name="diana7_j1" type="revolute">
     <origin
       xyz="0.0 -2.9150689157e-12 0.2856"
@@ -187,5 +187,5 @@
     </collision>
   </link>
-  <joint name="joint_2" type="revolute">
+  <joint name="diana7_j2" type="revolute">
     <origin
       xyz="0.0 -0.0 0.0"
@@ -235,5 +235,5 @@
     </collision>
   </link>
-  <joint name="joint_3" type="revolute">
+  <joint name="diana7_j3" type="revolute">
     <origin
       xyz="0.0 -0.4586 -2.24557565126e-12"
@@ -282,5 +282,5 @@
     </collision>
   </link>
-  <joint name="joint_4" type="revolute">
+  <joint name="diana7_j4" type="revolute">
     <origin
       xyz="0.065 -0.0 0.0"
@@ -329,5 +329,5 @@
     </collision>
   </link>
-  <joint name="joint_5" type="revolute">
+  <joint name="diana7_j5" type="revolute">
     <origin
       xyz="-0.0528 -0.4554 -2.22990656691e-12"
@@ -376,5 +376,5 @@
     </collision>
   </link>
-  <joint name="joint_6" type="revolute">
+  <joint name="diana7_j6" type="revolute">
     <origin
       xyz="-0.0122 0.0 0.0"
@@ -423,5 +423,5 @@
     </collision>
   </link>
-  <joint name="joint_7" type="revolute">
+  <joint name="diana7_j7" type="revolute">
     <origin
       xyz="0.087 -0.1169 -5.72411237751e-13"

File: src/zlab_robots_descriptions/diana7_description/urdf/diana7_macro.xacro (robot description, xacro)
@@ -131,5 +131,5 @@
       </collision>
     </link>
-    <joint name="${prefix}joint_1" type="revolute">
+    <joint name="${prefix}j1" type="revolute">
       <origin
         xyz="0.0 -2.9150689157e-12 0.2856"
@@ -178,5 +178,5 @@
       </collision>
     </link>
-    <joint name="${prefix}joint_2" type="revolute">
+    <joint name="${prefix}j2" type="revolute">
       <origin
         xyz="0.0 -0.0 0.0"
@@ -226,5 +226,5 @@
       </collision>
     </link>
-    <joint name="${prefix}joint_3" type="revolute">
+    <joint name="${prefix}j3" type="revolute">
       <origin
         xyz="0.0 -0.4586 -2.24557565126e-12"
@@ -273,5 +273,5 @@
       </collision>
     </link>
-    <joint name="${prefix}joint_4" type="revolute">
+    <joint name="${prefix}j4" type="revolute">
       <origin
         xyz="0.065 -0.0 0.0"
@@ -320,5 +320,5 @@
       </collision>
     </link>
-    <joint name="${prefix}joint_5" type="revolute">
+    <joint name="${prefix}j5" type="revolute">
       <origin
         xyz="-0.0528 -0.4554 -2.22990656691e-12"
@@ -367,5 +367,5 @@
       </collision>
     </link>
-    <joint name="${prefix}joint_6" type="revolute">
+    <joint name="${prefix}j6" type="revolute">
       <origin
         xyz="-0.0122 0.0 0.0"
@@ -414,5 +414,5 @@
       </collision>
     </link>
-    <joint name="${prefix}joint_7" type="revolute">
+    <joint name="${prefix}j7" type="revolute">
       <origin
         xyz="0.087 -0.1169 -5.72411237751e-13"

File: src/zlab_robots_moveit_config/triple_arm_moveit_config/config/zlab_triple_arms.srdf.xacro (robot description, xacro)
@@ -54,11 +54,11 @@
     <!-- Diana7 States -->
     <group_state name="home" group="diana7">
-        <joint name="diana7_joint_1" value="0"/>
-        <joint name="diana7_joint_2" value="0"/>
-        <joint name="diana7_joint_3" value="0"/>
-        <joint name="diana7_joint_4" value="0"/>
-        <joint name="diana7_joint_5" value="0"/>
-        <joint name="diana7_joint_6" value="0"/>
-        <joint name="diana7_joint_7" value="0"/>
+        <joint name="diana7_j1" value="0"/>
+        <joint name="diana7_j2" value="0"/>
+        <joint name="diana7_j3" value="0"/>
+        <joint name="diana7_j4" value="0"/>
+        <joint name="diana7_j5" value="0"/>
+        <joint name="diana7_j6" value="0"/>
+        <joint name="diana7_j7" value="0"/>
     </group_state>
     <!-- Triple Arms States -->
@@ -76,11 +76,11 @@
         <joint name="arm2_j5" value="0"/>
         <joint name="arm2_j6" value="0"/>
-        <joint name="diana7_joint_1" value="0"/>
-        <joint name="diana7_joint_2" value="0"/>
-        <joint name="diana7_joint_3" value="0"/>
-        <joint name="diana7_joint_4" value="0"/>
-        <joint name="diana7_joint_5" value="0"/>
-        <joint name="diana7_joint_6" value="0"/>
-        <joint name="diana7_joint_7" value="0"/>
+        <joint name="diana7_j1" value="0"/>
+        <joint name="diana7_j2" value="0"/>
+        <joint name="diana7_j3" value="0"/>
+        <joint name="diana7_j4" value="0"/>
+        <joint name="diana7_j5" value="0"/>
+        <joint name="diana7_j6" value="0"/>
+        <joint name="diana7_j7" value="0"/>
     </group_state>
     <!-- VIRTUAL JOINTS -->
