Commit message: 20251225 统一bringup，添加位置加载

File: src/zlab_robots_descriptions/diana7_description/urdf/diana7.urdf.xacro (robot description, xacro)
@@ -1,13 +1,20 @@
 <?xml version="1.0" encoding="utf-8"?>
 <robot xmlns:xacro="http://wiki.ros.org/xacro" name="diana7">
+  <!-- Layout configuration file -->
+  <xacro:arg name="layout_config" default=""/>
+  <xacro:property name="layout" value="${xacro.load_yaml(arg('layout_config')) if arg('layout_config') else dict()}"/>
+  <!-- Position Arguments -->
+  <xacro:arg name="xyz" default="0 0 0"/>
+  <xacro:arg name="rpy" default="0 0 0"/>
   <!-- Tool Argument -->
   <xacro:arg name="tool_name" default="none"/>
   <!-- Include Tool Library -->
   <xacro:include filename="$(find zlab_tools_description)/urdf/tools_library.xacro" />
-  <link name="world">
-      <origin
-        xyz="0 0 0"
-        rpy="0 0 0" />
-  </link>
+  <link name="world" />
+  <!-- Resolve position with priority: 1. CLI/Launch > 2. Layout YAML > 3. Default -->
+  <xacro:property name="xyz_arg" value="$(arg xyz)"/>
+  <xacro:property name="rpy_arg" value="$(arg rpy)"/>
+  <xacro:property name="xyz_final" value="${xyz_arg if xyz_arg != '0 0 0' else (layout['diana7']['xyz'] if 'diana7' in layout and 'xyz' in layout['diana7'] else '0 0 0')}"/>
+  <xacro:property name="rpy_final" value="${rpy_arg if rpy_arg != '0 0 0' else (layout['diana7']['rpy'] if 'diana7' in layout and 'rpy' in layout['diana7'] else '0 0 0')}"/>
   <!-- Optional base assembly (default: included) -->
   <link name="diana7_base_link">
@@ -58,5 +65,5 @@
   </link>
   <joint name="world_to_diana7_base" type="fixed">
-    <origin xyz="0 0 0" rpy="0 0 0" />
+    <origin xyz="${xyz_final}" rpy="${rpy_final}" />
     <parent link="world" />
     <child link="diana7_base_link" />

File: src/zlab_robots_descriptions/fr5_description/fr5_description/urdf/fr.xacro (robot description, xacro)
@@ -1,4 +1,7 @@
 <?xml version="1.0"?>
 <robot name="fr" xmlns:xacro="http://www.ros.org/wiki/xacro">
+    <!-- Layout configuration file -->
+    <xacro:arg name="layout_config" default=""/>
+    <xacro:property name="layout" value="${xacro.load_yaml(arg('layout_config')) if arg('layout_config') else dict()}"/>
     <!-- 定义参数 -->
     <!-- arm_id: 机械臂ID，可以是 arm1, arm2 等，默认为 arm1 -->
@@ -6,4 +9,7 @@
     <!-- 定义工具参数 -->
     <xacro:arg name="tool_name" default="none"/>
+    <!-- Position Arguments -->
+    <xacro:arg name="xyz" default="0 0 0"/>
+    <xacro:arg name="rpy" default="0 0 0"/>
     <!-- 加载工具库 -->
     <xacro:include filename="$(find zlab_tools_description)/urdf/tools_library.xacro" />
@@ -12,10 +18,16 @@
     <!-- 添加虚拟根链接 -->
     <link name="world" />
+    <!-- Resolve position with priority: 1. CLI/Launch > 2. Layout YAML > 3. Default -->
+    <xacro:property name="arm_id_str" value="$(arg arm_id)"/>
+    <xacro:property name="xyz_arg" value="$(arg xyz)"/>
+    <xacro:property name="rpy_arg" value="$(arg rpy)"/>
+    <xacro:property name="xyz_final" value="${xyz_arg if xyz_arg != '0 0 0' else (layout[arm_id_str]['xyz'] if arm_id_str in layout and 'xyz' in layout[arm_id_str] else '0 0 0')}"/>
+    <xacro:property name="rpy_final" value="${rpy_arg if rpy_arg != '0 0 0' else (layout[arm_id_str]['rpy'] if arm_id_str in layout and 'rpy' in layout[arm_id_str] else '0 0 0')}"/>
     <!-- 实例化机械臂 -->
     <xacro:fr
         arm_id="$(arg arm_id)"
         connected_to="world"
-        xyz="0 0 0"
-        rpy="0 0 0"
+        xyz="${xyz_final}"
+        rpy="${rpy_final}"
         tool_name="none"
         tool_config="{}" />

File: src/zlab_robots_descriptions/fr5_description/fr5_description/urdf/zlab_dual_arms.xacro (robot description, xacro)
@@ -1,4 +1,7 @@
 <?xml version="1.0"?>
 <robot name="zlab_dual_arms" xmlns:xacro="http://www.ros.org/wiki/xacro">
+    <!-- Layout configuration file -->
+    <xacro:arg name="layout_config" default=""/>
+    <xacro:property name="layout" value="${xacro.load_yaml(arg('layout_config')) if arg('layout_config') else dict()}"/>
     <!-- 定义参数 -->
     <!-- arm1 工具参数 -->
@@ -18,4 +21,9 @@
     <!-- 创建世界坐标系 -->
     <link name="world" />
+    <!-- ========== 设置arm1位置 ========== -->
+    <xacro:property name="a1_xyz_arg" value="$(arg arm1_xyz)"/>
+    <xacro:property name="a1_rpy_arg" value="$(arg arm1_rpy)"/>
+    <xacro:property name="arm1_xyz_final" value="${a1_xyz_arg if a1_xyz_arg != '' else (layout['arm1']['xyz'] if 'arm1' in layout and 'xyz' in layout['arm1'] else '0 0 0')}"/>
+    <xacro:property name="arm1_rpy_final" value="${a1_rpy_arg if a1_rpy_arg != '' else (layout['arm1']['rpy'] if 'arm1' in layout and 'rpy' in layout['arm1'] else '0 0 0')}"/>
     <!-- ========== 设置arm2位置 ========== -->
     <!-- 默认值：arm1在原点，arm2在右边1米处 -->
@@ -25,27 +33,24 @@
     <xacro:property name="arm2_xyz_arg" value="$(arg arm2_xyz)"/>
     <xacro:property name="arm2_rpy_arg" value="$(arg arm2_rpy)"/>
-    <!-- 如果arm2_xyz参数未指定（为空），尝试从标定文件加载 -->
-    <xacro:if value="${arm2_xyz_arg == ''}">
-        <xacro:property name="calibration_file_path"
-                        value="$(find fr5_description)/config/dual_arm_calibration.yaml"/>
-        <xacro:property name="calibration_config"
-                        value="${xacro.load_yaml(calibration_file_path)}"/>
-        <xacro:property name="transform" value="${calibration_config['arm1_to_arm2_transform']}"/>
-        <xacro:property name="translation" value="${transform['translation']}"/>
-        <xacro:property name="rpy" value="${transform['rpy']}"/>
-        <!-- 使用标定文件中的位置和姿态 -->
-        <xacro:property name="arm2_xyz_final"
-                        value="${translation['x']} ${translation['y']} ${translation['z']}"/>
-        <xacro:property name="arm2_rpy_final"
-                        value="${rpy['roll']} ${rpy['pitch']} ${rpy['yaw']}"/>
+    <!-- 优先级：1. CLI/Launch > 2. Layout YAML > 3. Calibration YAML > 4. Default -->
+    <xacro:if value="${arm2_xyz_arg != ''}">
+        <xacro:property name="arm2_xyz_final" value="${arm2_xyz_arg}"/>
+        <xacro:property name="arm2_rpy_final" value="${arm2_rpy_arg if arm2_rpy_arg != '' else arm2_rpy_default}"/>
     </xacro:if>
-    <!-- 如果arm2_xyz参数已指定，使用参数值 -->
-    <xacro:unless value="${arm2_xyz_arg == ''}">
-        <xacro:property name="arm2_xyz_final" value="${arm2_xyz_arg}"/>
-        <xacro:if value="${arm2_rpy_arg == ''}">
-            <xacro:property name="arm2_rpy_final" value="${arm2_rpy_default}"/>
+    <xacro:unless value="${arm2_xyz_arg != ''}">
+        <!-- 尝试从 Layout YAML 加载 -->
+        <xacro:if value="${layout and 'arm2' in layout and 'xyz' in layout['arm2']}">
+            <xacro:property name="arm2_xyz_final" value="${layout['arm2']['xyz']}"/>
+            <xacro:property name="arm2_rpy_final" value="${layout['arm2']['rpy'] if 'rpy' in layout['arm2'] else arm2_rpy_default}"/>
         </xacro:if>
-        <xacro:unless value="${arm2_rpy_arg == ''}">
-            <xacro:property name="arm2_rpy_final" value="${arm2_rpy_arg}"/>
+        <xacro:unless value="${layout and 'arm2' in layout and 'xyz' in layout['arm2']}">
+            <!-- 尝试从标定文件加载 -->
+            <xacro:property name="calibration_file_path" value="$(find fr5_description)/config/dual_arm_calibration.yaml"/>
+            <xacro:property name="calibration_config" value="${xacro.load_yaml(calibration_file_path)}"/>
+            <xacro:property name="transform" value="${calibration_config['arm1_to_arm2_transform']}"/>
+            <xacro:property name="translation" value="${transform['translation']}"/>
+            <xacro:property name="rpy" value="${transform['rpy']}"/>
+            <xacro:property name="arm2_xyz_final" value="${translation['x']} ${translation['y']} ${translation['z']}"/>
+            <xacro:property name="arm2_rpy_final" value="${rpy['roll']} ${rpy['pitch']} ${rpy['yaw']}"/>
         </xacro:unless>
     </xacro:unless>
@@ -54,6 +59,6 @@
         arm_id="arm1"
         connected_to="world"
-        xyz="$(arg arm1_xyz)"
-        rpy="$(arg arm1_rpy)"
+        xyz="${arm1_xyz_final}"
+        rpy="${arm1_rpy_final}"
         tool_name="none"
         tool_config="{}" />

File: src/zlab_robots_descriptions/fr5_description/fr5_description/urdf/zlab_triple_arms.xacro (robot description, xacro)
@@ -1,4 +1,7 @@
 <?xml version="1.0"?>
 <robot name="zlab_triple_arms" xmlns:xacro="http://www.ros.org/wiki/xacro">
+    <!-- Layout configuration file -->
+    <xacro:arg name="layout_config" default=""/>
+    <xacro:property name="layout" value="${xacro.load_yaml(arg('layout_config')) if arg('layout_config') else dict()}"/>
     <!-- Arguments for positions -->
     <!-- Diana7 (Center) -->
@@ -11,4 +14,17 @@
     <xacro:arg name="arm2_xyz" default="1.5 0.4 0"/>
     <xacro:arg name="arm2_rpy" default="0 0 0"/>
+    <!-- Resolve positions (Priority: CLI/Launch > YAML > Xacro Default) -->
+    <xacro:property name="d7_xyz_arg" value="$(arg diana7_xyz)"/>
+    <xacro:property name="d7_rpy_arg" value="$(arg diana7_rpy)"/>
+    <xacro:property name="diana7_xyz_final" value="${d7_xyz_arg if d7_xyz_arg != '' else (layout['diana7']['xyz'] if 'diana7' in layout and 'xyz' in layout['diana7'] else '0 0 0')}"/>
+    <xacro:property name="diana7_rpy_final" value="${d7_rpy_arg if d7_rpy_arg != '' else (layout['diana7']['rpy'] if 'diana7' in layout and 'rpy' in layout['diana7'] else '0 0 0')}"/>
+    <xacro:property name="a1_xyz_arg" value="$(arg arm1_xyz)"/>
+    <xacro:property name="a1_rpy_arg" value="$(arg arm1_rpy)"/>
+    <xacro:property name="arm1_xyz_final" value="${a1_xyz_arg if a1_xyz_arg != '' else (layout['arm1']['xyz'] if 'arm1' in layout and 'xyz' in layout['arm1'] else '1.5 -0.2 0')}"/>
+    <xacro:property name="arm1_rpy_final" value="${a1_rpy_arg if a1_rpy_arg != '' else (layout['arm1']['rpy'] if 'arm1' in layout and 'rpy' in layout['arm1'] else '0 0 0')}"/>
+    <xacro:property name="a2_xyz_arg" value="$(arg arm2_xyz)"/>
+    <xacro:property name="a2_rpy_arg" value="$(arg arm2_rpy)"/>
+    <xacro:property name="arm2_xyz_final" value="${a2_xyz_arg if a2_xyz_arg != '' else (layout['arm2']['xyz'] if 'arm2' in layout and 'xyz' in layout['arm2'] else '1.5 0.4 0')}"/>
+    <xacro:property name="arm2_rpy_final" value="${a2_rpy_arg if a2_rpy_arg != '' else (layout['arm2']['rpy'] if 'arm2' in layout and 'rpy' in layout['arm2'] else '0 0 0')}"/>
     <!-- Arguments for tools -->
     <xacro:arg name="arm1_tool" default="none"/>
@@ -23,14 +39,14 @@
     <!-- Instantiate Diana7 -->
     <xacro:diana7_robot prefix="diana7_" parent="world">
-        <origin xyz="$(arg diana7_xyz)" rpy="$(arg diana7_rpy)"/>
+        <origin xyz="${diana7_xyz_final}" rpy="${diana7_rpy_final}"/>
     </xacro:diana7_robot>
     <!-- Load Tool for Diana7 -->
     <xacro:load_tool tool_name="$(arg diana7_tool)" prefix="diana7_" parent="diana7_link_7"/>
     <!-- Instantiate FR5 Arm 1 -->
-    <xacro:fr arm_id="arm1" connected_to="world" xyz="$(arg arm1_xyz)" rpy="$(arg arm1_rpy)" tool_name="none"/>
+    <xacro:fr arm_id="arm1" connected_to="world" xyz="${arm1_xyz_final}" rpy="${arm1_rpy_final}" tool_name="none"/>
     <!-- Load Tool for Arm 1 -->
     <xacro:load_tool tool_name="$(arg arm1_tool)" prefix="arm1_" parent="arm1_ee_link"/>
     <!-- Instantiate FR5 Arm 2 -->
-    <xacro:fr arm_id="arm2" connected_to="world" xyz="$(arg arm2_xyz)" rpy="$(arg arm2_rpy)" tool_name="none"/>
+    <xacro:fr arm_id="arm2" connected_to="world" xyz="${arm2_xyz_final}" rpy="${arm2_rpy_final}" tool_name="none"/>
     <!-- Load Tool for Arm 2 -->
     <xacro:load_tool tool_name="$(arg arm2_tool)" prefix="arm2_" parent="arm2_ee_link"/>
