Commit message: 20251230更新tool

File: src/zlab_robots_descriptions/diana7_description/urdf/diana7.urdf.xacro (robot description, xacro)
@@ -20,5 +20,5 @@
   <!-- Instantiate Diana7 -->
   <xacro:diana7_robot
-    prefix="diana7_"
+    prefix="diana7"
     parent="world"
     tool_name="$(arg tool_name)">

File: src/zlab_robots_descriptions/diana7_description/urdf/diana7_macro.xacro (robot description, xacro)
@@ -2,5 +2,5 @@
 <robot xmlns:xacro="http://wiki.ros.org/xacro">
   <xacro:macro name="diana7_robot" params="prefix:='' parent:='world' tool_name:='none' *origin">
-    <link name="${prefix}base_link">
+    <link name="${prefix}_base_link">
       <inertial>
         <origin
@@ -36,5 +36,5 @@
       </collision>
     </link>
-    <link name="${prefix}pedestal_link">
+    <link name="${prefix}_pedestal_link">
       <inertial>
         <origin xyz="-0.042824 -0.00012843 0.38233" rpy="0 0 0" />
@@ -59,5 +59,5 @@
       </collision>
     </link>
-    <link name="${prefix}pedestal_flange_link">
+    <link name="${prefix}_pedestal_flange_link">
       <inertial>
         <origin xyz="-0.052824 0.021372 -0.39767" rpy="0 0 0" />
@@ -82,20 +82,20 @@
       </collision>
     </link>
-    <joint name="${prefix}pedestal_joint" type="fixed">
+    <joint name="${prefix}_pedestal_joint" type="fixed">
       <parent link="${parent}"/>
-      <child link="${prefix}pedestal_link"/>
+      <child link="${prefix}_pedestal_link"/>
       <xacro:insert_block name="origin" />
     </joint>
-    <joint name="${prefix}pedestal_to_flange" type="fixed">
+    <joint name="${prefix}_pedestal_to_flange" type="fixed">
       <origin xyz="0.01 -0.0215 0.78" rpy="0 0 0" />
-      <parent link="${prefix}pedestal_link" />
-      <child link="${prefix}pedestal_flange_link" />
-    </joint>
-    <joint name="${prefix}base_joint" type="fixed">
-      <parent link="${prefix}pedestal_flange_link"/>
-      <child link="${prefix}base_link"/>
+      <parent link="${prefix}_pedestal_link" />
+      <child link="${prefix}_pedestal_flange_link" />
+    </joint>
+    <joint name="${prefix}_base_joint" type="fixed">
+      <parent link="${prefix}_pedestal_flange_link"/>
+      <child link="${prefix}_base_link"/>
       <origin xyz="0 0 0" rpy="0 0 0" />
     </joint>
-    <link name="${prefix}link_1">
+    <link name="${prefix}_link_1">
       <inertial>
         <origin
@@ -131,10 +131,10 @@
       </collision>
     </link>
-    <joint name="${prefix}joint_1" type="revolute">
+    <joint name="${prefix}_joint_1" type="revolute">
       <origin
         xyz="0.0 -2.9150689157e-12 0.2856"
         rpy="-3.1415926535795866 0.0 -0.0" />
-      <parent link="${prefix}base_link" />
-      <child link="${prefix}link_1" />
+      <parent link="${prefix}_base_link" />
+      <child link="${prefix}_link_1" />
       <axis xyz="0 0 1" />
       <limit
@@ -144,5 +144,5 @@
         velocity="2.61" />
     </joint>
-    <link name="${prefix}link_2">
+    <link name="${prefix}_link_2">
       <inertial>
         <origin
@@ -178,10 +178,10 @@
       </collision>
     </link>
-    <joint name="${prefix}joint_2" type="revolute">
+    <joint name="${prefix}_joint_2" type="revolute">
       <origin
         xyz="0.0 -0.0 0.0"
         rpy="1.57079632679 -0.0 0.0" />
-      <parent link="${prefix}link_1" />
-      <child link="${prefix}link_2" />
+      <parent link="${prefix}_link_1" />
+      <child link="${prefix}_link_2" />
       <axis xyz="0 0 1" />
       <limit
@@ -191,5 +191,5 @@
         velocity="2.618" />
     </joint>
-    <link name="${prefix}link_3">
+    <link name="${prefix}_link_3">
       <inertial>
         <origin
@@ -226,10 +226,10 @@
       </collision>
     </link>
-    <joint name="${prefix}joint_3" type="revolute">
+    <joint name="${prefix}_joint_3" type="revolute">
       <origin
         xyz="0.0 -0.4586 -2.24557565126e-12"
         rpy="-1.57079632679 0.0 0.0" />
-      <parent link="${prefix}link_2" />
-      <child link="${prefix}link_3" />
+      <parent link="${prefix}_link_2" />
+      <child link="${prefix}_link_3" />
       <axis xyz="0 0 1" />
       <limit
@@ -239,5 +239,5 @@
         velocity="2.61" />
     </joint>
-    <link name="${prefix}link_4">
+    <link name="${prefix}_link_4">
       <inertial>
         <origin
@@ -273,10 +273,10 @@
       </collision>
     </link>
-    <joint name="${prefix}joint_4" type="revolute">
+    <joint name="${prefix}_joint_4" type="revolute">
       <origin
         xyz="0.065 -0.0 0.0"
         rpy="1.57079632679 -0.0 0.0" />
-      <parent link="${prefix}link_3" />
-      <child link="${prefix}link_4" />
+      <parent link="${prefix}_link_3" />
+      <child link="${prefix}_link_4" />
       <axis xyz="0 0 1" />
       <limit
@@ -286,5 +286,5 @@
         velocity="2.61" />
     </joint>
-    <link name="${prefix}link_5">
+    <link name="${prefix}_link_5">
       <inertial>
         <origin
@@ -320,10 +320,10 @@
       </collision>
     </link>
-    <joint name="${prefix}joint_5" type="revolute">
+    <joint name="${prefix}_joint_5" type="revolute">
       <origin
         xyz="-0.0528 -0.4554 -2.22990656691e-12"
         rpy="-1.57079632679 0.0 0.0" />
-      <parent link="${prefix}link_4" />
-      <child link="${prefix}link_5" />
+      <parent link="${prefix}_link_4" />
+      <child link="${prefix}_link_5" />
       <axis xyz="0 0 1" />
       <limit
@@ -333,5 +333,5 @@
         velocity="3.14" />
     </joint>
-    <link name="${prefix}link_6">
+    <link name="${prefix}_link_6">
       <inertial>
         <origin
@@ -367,10 +367,10 @@
       </collision>
     </link>
-    <joint name="${prefix}joint_6" type="revolute">
+    <joint name="${prefix}_joint_6" type="revolute">
       <origin
         xyz="-0.0122 0.0 0.0"
         rpy="1.57079632679 -1.0206823934513925e-11 -3.141592653589793" />
-      <parent link="${prefix}link_5" />
-      <child link="${prefix}link_6" />
+      <parent link="${prefix}_link_5" />
+      <child link="${prefix}_link_6" />
       <axis xyz="0 0 1" />
       <limit
@@ -380,5 +380,5 @@
         velocity="3.14" />
     </joint>
-    <link name="${prefix}link_7">
+    <link name="${prefix}_link_7">
       <inertial>
         <origin
@@ -414,10 +414,10 @@
       </collision>
     </link>
-    <joint name="${prefix}joint_7" type="revolute">
+    <joint name="${prefix}_joint_7" type="revolute">
       <origin
         xyz="0.087 -0.1169 -5.72411237751e-13"
         rpy="-1.57079632679 0.0 0.0" />
-      <parent link="${prefix}link_6" />
-      <child link="${prefix}link_7" />
+      <parent link="${prefix}_link_6" />
+      <child link="${prefix}_link_7" />
       <axis xyz="0 0 1" />
       <limit
@@ -428,9 +428,9 @@
     </joint>
     <!-- End Effector Link -->
-    <link name="${prefix}ee_link" />
-    <joint name="${prefix}joint_ee" type="fixed">
-      <parent link="${prefix}link_7" />
-      <child link="${prefix}ee_link" />
-      <origin xyz="0 0 0" rpy="0 0 0" />
+    <link name="${prefix}_ee_link" />
+    <joint name="${prefix}_joint_ee" type="fixed">
+      <parent link="${prefix}_link_7" />
+      <child link="${prefix}_ee_link" />
+      <origin xyz="0 0 0" rpy="3.1415926531795866 0 1.5707963266" />
     </joint>
     <!-- Tool Loading -->
@@ -440,5 +440,5 @@
             tool_name="${tool_name}"
             prefix="${prefix}"
-            parent="${prefix}ee_link" />
+            parent="${prefix}_ee_link" />
     </xacro:unless>
   </xacro:macro>

File: src/zlab_robots_descriptions/fr5_description/urdf/zlab_triple_arms.xacro (robot description, xacro)
@@ -40,5 +40,5 @@
     <!-- Instantiate Diana7 -->
     <xacro:diana7_robot
-        prefix="diana7_"
+        prefix="diana7"
         parent="world"
         tool_name="$(arg diana7_tool)">

File: src/zlab_robots_descriptions/zlab_tools_description/tool_template/urdf/tool_template_macro.xacro (robot description, xacro)
@@ -1,10 +1,5 @@
 <?xml version="1.0"?>
 <robot xmlns:xacro="http://www.ros.org/wiki/xacro">
-  <xacro:macro name="tool_template" params="prefix parent">
-    <joint name="${prefix}tool_joint" type="fixed">
-      <parent link="${parent}"/>
-      <child link="${prefix}tool_base_link"/>
-      <origin xyz="0 0 0" rpy="0 0 0"/>
-    </joint>
+  <xacro:macro name="tool_template" params="prefix">
     <link name="${prefix}tool_base_link">
       <visual>

File: src/zlab_robots_descriptions/zlab_tools_description/tools/magnetometer_array/urdf/magnetometer_array.urdf.xacro (robot description, xacro)
@@ -1,6 +1,11 @@
 <?xml version="1.0" encoding="utf-8"?>
 <robot name="magnetometer_array" xmlns:xacro="http://www.ros.org/wiki/xacro">
+  <!--
+    此文件专门用于工具集成加载系统。
+    它会被 tool_loader.xacro 包含。
+    tool_loader.xacro 会预先定义 tool_arm_id 属性。
+  -->
   <xacro:include filename="$(find zlab_tools_description)/tools/magnetometer_array/urdf/magnetometer_array_macro.xacro"/>
-  <link name="world"/>
-  <xacro:magnetometer_array prefix="" parent="world"/>
+  <!-- 实例化 Links，使用机械臂前缀 -->
+  <xacro:magnetometer_array_links prefix="${tool_arm_id}_" />
 </robot>

File: src/zlab_robots_descriptions/zlab_tools_description/tools/magnetometer_array/urdf/magnetometer_array_macro.xacro (robot description, xacro)
@@ -1,15 +1,11 @@
 <?xml version="1.0" encoding="utf-8"?>
 <robot xmlns:xacro="http://www.ros.org/wiki/xacro">
-  <xacro:macro name="magnetometer_array" params="prefix parent">
-    <joint name="${prefix}tool_joint" type="fixed">
-      <parent link="${parent}"/>
-      <child link="${prefix}magnetometer_base_link"/>
-      <origin xyz="0 0 0" rpy="0 0 ${pi/2}"/>
-    </joint>
+  <!-- 仅定义 Links 的宏 -->
+  <xacro:macro name="magnetometer_array_links" params="prefix">
     <link name="${prefix}magnetometer_base_link">
       <inertial>
-        <origin xyz="2.0717E-07 0.0021605 -0.036248" rpy="0 0 0" />
-        <mass value="0.033205" />
-        <inertia ixx="5.6306E-05" ixy="-5.922E-12" ixz="6.6801E-10" iyy="5.9694E-05" iyz="2.0305E-06" izz="1.1454E-05" />
+        <origin xyz="-2.07166456525017E-07 0.0021604655211999 0.0362476651991424" rpy="0 0 0" />
+        <mass value="0.0332054242847689" />
+        <inertia ixx="5.63055976294825E-05" ixy="5.92198383565254E-12" ixz="6.68013595190661E-10" iyy="5.96936991935191E-05" iyz="-2.03045562894017E-06" izz="1.14540668478137E-05" />
       </inertial>
       <visual>
@@ -31,7 +27,7 @@
     <link name="${prefix}magnetometer_tcp_link">
       <inertial>
-        <origin xyz="-0.00019067 0.0018908 -0.060443" rpy="0 0 0" />
-        <mass value="0.0022623" />
-        <inertia ixx="3.3502E-07" ixy="6.2726E-20" ixz="-6.8291E-10" iyy="4.1094E-07" iyz="1.8218E-19" izz="8.7172E-08" />
+        <origin xyz="-0.000190659438675016 0.00189080741259228 -0.0604428602463941" rpy="0 0 0" />
+        <mass value="0.00226226919267647" />
+        <inertia ixx="3.35022731202412E-07" ixy="6.2725681636899E-20" ixz="-6.82910069048886E-10" iyy="4.1094183087163E-07" iyz="1.82178739960353E-19" izz="8.71724385779425E-08" />
       </inertial>
       <visual>
@@ -41,5 +37,5 @@
         </geometry>
         <material name="">
-          <color rgba="0.75294 0.75294 0.75294 1" />
+          <color rgba="0.752941176470588 0.752941176470588 0.752941176470588 1" />
         </material>
       </visual>
@@ -52,5 +48,5 @@
     </link>
     <joint name="${prefix}magnetometer_joint" type="fixed">
-      <origin xyz="0 0.00023753 -0.19309" rpy="3.1416 0 3.1416" />
+      <origin xyz="0 0.00023753 0.19309" rpy="0 0 0" />
       <parent link="${prefix}magnetometer_base_link" />
       <child link="${prefix}magnetometer_tcp_link" />
@@ -58,3 +54,12 @@
     </joint>
   </xacro:macro>
+  <!-- 完整定义的宏（包含与 parent 的连接） -->
+  <xacro:macro name="magnetometer_array" params="prefix parent">
+    <joint name="${prefix}tool_joint" type="fixed">
+      <parent link="${parent}"/>
+      <child link="${prefix}magnetometer_base_link"/>
+      <origin xyz="0 0 0" rpy="0 0 0"/>
+    </joint>
+    <xacro:magnetometer_array_links prefix="${prefix}" />
+  </xacro:macro>
 </robot>
