Commit message: 20251229 删除flange

File: src/zlab_robots_descriptions/diana7_description/urdf/diana7_macro.xacro (robot description, xacro)
@@ -427,14 +427,8 @@
         velocity="3.14" />
     </joint>
-    <!-- Flange and EE -->
-    <link name="${prefix}flange" />
-    <joint name="${prefix}joint_flange" type="fixed">
-      <parent link="${prefix}link_7" />
-      <child link="${prefix}flange" />
-      <origin xyz="0 0 0" rpy="0 0 0" />
-    </joint>
+    <!-- End Effector Link -->
     <link name="${prefix}ee_link" />
     <joint name="${prefix}joint_ee" type="fixed">
-      <parent link="${prefix}flange" />
+      <parent link="${prefix}link_7" />
       <child link="${prefix}ee_link" />
       <origin xyz="0 0 0" rpy="0 0 0" />

File: src/zlab_robots_descriptions/fr5_description/fr5_description/urdf/fr5_library.xacro (robot description, xacro)
@@ -1,5 +1,5 @@
 <?xml version="1.0" encoding="utf-8"?>
-<robot name="fr" xmlns:xacro="http://www.ros.org/wiki/xacro">
-    <xacro:macro name="fr"
+<robot name="fr5" xmlns:xacro="http://www.ros.org/wiki/xacro">
+    <xacro:macro name="fr5"
         params="arm_id:='fr1' connected_to:='' xyz:='0 0 0' rpy:='0 0 0' tool_name:='none' tool_config:='{}'">
         <xacro:unless value="${not connected_to}">
@@ -204,11 +204,4 @@
                 k_velocity="10" />
         </joint>
-        <!-- Flange Link -->
-        <link name="${arm_id}_flange" />
-        <joint name="${arm_id}_joint_flange" type="fixed">
-            <parent link="${arm_id}_link_6" />
-            <child link="${arm_id}_flange" />
-            <origin xyz="0 0 0.1" rpy="0 0 0" />
-        </joint>
         <!-- 如果工具名称为none，只创建ee_link，不加载工具 -->
         <xacro:if value="${tool_name == 'none'}">
@@ -223,7 +216,7 @@
             </link>
             <joint name="${arm_id}_ee_joint" type="fixed">
-                <parent link="${arm_id}_flange" />
+                <parent link="${arm_id}_link_6" />
                 <child link="${arm_id}_ee_link" />
-                <origin xyz="0 0 0" rpy="0 0 0" />
+                <origin xyz="0 0 0.1" rpy="0 0 0" />
             </joint>
         </xacro:if>
@@ -236,5 +229,5 @@
             <!-- 如果使用工具包系统，先创建ee_link作为中间链接 -->
             <xacro:if value="${use_tool_package}">
-                <!-- 创建ee_link（连接到flange） -->
+                <!-- 创建ee_link（连接到link_6） -->
                 <link name="${arm_id}_ee_link">
                     <inertial>
@@ -246,9 +239,9 @@
                     </inertial>
                 </link>
-                <!-- 创建从flange到ee_link的关节 -->
+                <!-- 创建从link_6到ee_link的关节 -->
                 <joint name="${arm_id}_ee_joint" type="fixed">
-                    <parent link="${arm_id}_flange" />
+                    <parent link="${arm_id}_link_6" />
                     <child link="${arm_id}_ee_link" />
-                    <origin xyz="0 0 0" rpy="0 0 0" />
+                    <origin xyz="0 0 0.1" rpy="0 0 0" />
                 </joint>
                 <!-- 使用新的工具加载器，工具将连接到ee_link -->

File: src/zlab_robots_descriptions/fr5_description/urdf/fr5.xacro (robot description, xacro)
@@ -1,4 +1,4 @@
 <?xml version="1.0"?>
-<robot name="fr" xmlns:xacro="http://www.ros.org/wiki/xacro">
+<robot name="fr5" xmlns:xacro="http://www.ros.org/wiki/xacro">
     <!-- Layout configuration file -->
     <xacro:arg name="layout_config" default=""/>
@@ -26,5 +26,5 @@
     <xacro:property name="rpy_final" value="${rpy_arg if rpy_arg != '0 0 0' else (layout[arm_id_str]['rpy'] if arm_id_str in layout and 'rpy' in layout[arm_id_str] else '0 0 0')}"/>
     <!-- 实例化机械臂 -->
-    <xacro:fr
+    <xacro:fr5
         arm_id="$(arg arm_id)"
         connected_to="world"

File: src/zlab_robots_descriptions/fr5_description/urdf/fr5_library.xacro (robot description, xacro)
@@ -1,5 +1,5 @@
 <?xml version="1.0" encoding="utf-8"?>
-<robot name="fr" xmlns:xacro="http://www.ros.org/wiki/xacro">
-    <xacro:macro name="fr"
+<robot name="fr5" xmlns:xacro="http://www.ros.org/wiki/xacro">
+    <xacro:macro name="fr5"
         params="arm_id:='fr1' connected_to:='' xyz:='0 0 0' rpy:='0 0 0' tool_name:='none'">
         <xacro:unless value="${not connected_to}">
@@ -198,19 +198,12 @@
                 k_velocity="10" />
         </joint>
-        <!-- Flange Link -->
-        <link name="${arm_id}_flange" />
-        <joint name="${arm_id}_joint_flange" type="fixed">
-            <parent link="${arm_id}_link_6" />
-            <child link="${arm_id}_flange" />
-            <origin xyz="0 0 0.1" rpy="0 0 0" />
-        </joint>
         <!-- Tool Loading -->
         <xacro:include filename="$(find zlab_tools_description)/urdf/zlab_tools.xacro" />
-        <!-- Always create ee_link as a reference point at the flange -->
+        <!-- Always create ee_link as a reference point at the end of link_6 -->
         <link name="${arm_id}_ee_link" />
         <joint name="${arm_id}_ee_joint" type="fixed">
-            <parent link="${arm_id}_flange" />
+            <parent link="${arm_id}_link_6" />
             <child link="${arm_id}_ee_link" />
-            <origin xyz="0 0 0" rpy="0 0 0" />
+            <origin xyz="0 0 0.1" rpy="0 0 0" />
         </joint>
         <xacro:unless value="${tool_name == 'none'}">

File: src/zlab_robots_descriptions/fr5_description/urdf/zlab_dual_arms.xacro (robot description, xacro)
@@ -57,5 +57,5 @@
     </xacro:unless>
     <!-- ========== 实例化 arm1 ========== -->
-    <xacro:fr
+    <xacro:fr5
         arm_id="arm1"
         connected_to="world"
@@ -70,5 +70,5 @@
     <xacro:gazebo-joint joint="arm1_joint_6" />
     <!-- ========== 实例化 arm2 ========== -->
-    <xacro:fr
+    <xacro:fr5
         arm_id="arm2"
         connected_to="world"

File: src/zlab_robots_descriptions/fr5_description/urdf/zlab_triple_arms.xacro (robot description, xacro)
@@ -7,12 +7,12 @@
     <!-- Arguments for positions -->
     <!-- Diana7 (Center) -->
-    <xacro:arg name="diana7_xyz" default="0 0 0"/>
-    <xacro:arg name="diana7_rpy" default="0 0 0"/>
+    <xacro:arg name="diana7_xyz" default=""/>
+    <xacro:arg name="diana7_rpy" default=""/>
     <!-- FR5 Arm 1 (Left) -->
-    <xacro:arg name="arm1_xyz" default="1.5 -0.2 0"/>
-    <xacro:arg name="arm1_rpy" default="0 0 0"/>
+    <xacro:arg name="arm1_xyz" default=""/>
+    <xacro:arg name="arm1_rpy" default=""/>
     <!-- FR5 Arm 2 (Right) -->
-    <xacro:arg name="arm2_xyz" default="1.5 0.4 0"/>
-    <xacro:arg name="arm2_rpy" default="0 0 0"/>
+    <xacro:arg name="arm2_xyz" default=""/>
+    <xacro:arg name="arm2_rpy" default=""/>
     <!-- Resolve positions (Priority: CLI/Launch > YAML > Xacro Default) -->
     <xacro:property name="d7_xyz_arg" value="$(arg diana7_xyz)"/>
@@ -46,5 +46,5 @@
     </xacro:diana7_robot>
     <!-- Instantiate FR5 Arm 1 -->
-    <xacro:fr
+    <xacro:fr5
         arm_id="arm1"
         connected_to="world"
@@ -53,5 +53,5 @@
         tool_name="$(arg arm1_tool)"/>
     <!-- Instantiate FR5 Arm 2 -->
-    <xacro:fr
+    <xacro:fr5
         arm_id="arm2"
         connected_to="world"

File: src/zlab_robots_moveit_config/fr5_single_moveit_config/config/fr5.srdf.xacro (robot description, xacro)
@@ -4,5 +4,5 @@
     A URDF file must exist for this robot as well, where the joints and the links that are referenced are defined
 -->
-<robot name="fr" xmlns:xacro="http://www.ros.org/wiki/xacro">
+<robot name="fr5" xmlns:xacro="http://www.ros.org/wiki/xacro">
     <!-- Arm ID parameter -->
     <xacro:arg name="arm_id" default="arm1" />
@@ -12,5 +12,5 @@
     <!--CHAINS: When a chain is specified, all the links along the chain (including endpoints) are included in the group. Additionally, all the joints that are parents to included links are also included. This means that joints along the chain and the parent joint of the base link are included in the group-->
     <!--SUBGROUPS: Groups can also be formed by referencing to already defined group names-->
-    <group name="fr">
+    <group name="fr5">
         <link name="$(arg arm_id)_ee_link"/>
         <link name="$(arg arm_id)_link_1"/>
@@ -28,5 +28,5 @@
     </group>
     <!--GROUP STATES: Purpose: Define a named state for a particular group, in terms of joint values. This is useful to define states like 'folded arms'-->
-    <group_state name="zero" group="fr">
+    <group_state name="zero" group="fr5">
         <joint name="$(arg arm_id)_joint_1" value="0"/>
         <joint name="$(arg arm_id)_joint_2" value="0"/>
@@ -36,5 +36,5 @@
         <joint name="$(arg arm_id)_joint_6" value="0"/>
     </group_state>
-        <group_state name="up" group="fr">
+        <group_state name="up" group="fr5">
         <joint name="$(arg arm_id)_joint_1" value="0"/>
         <joint name="$(arg arm_id)_joint_2" value="-1.570796"/>
@@ -44,5 +44,5 @@
         <joint name="$(arg arm_id)_joint_6" value="0"/>
     </group_state>
-    <group_state name="ready" group="fr">
+    <group_state name="ready" group="fr5">
         <joint name="$(arg arm_id)_joint_1" value="0"/>
         <joint name="$(arg arm_id)_joint_2" value="-1.4189"/>
@@ -52,5 +52,5 @@
         <joint name="$(arg arm_id)_joint_6" value="0"/>
     </group_state>
-    <group_state name="bow" group="fr">
+    <group_state name="bow" group="fr5">
         <joint name="$(arg arm_id)_joint_1" value="0"/>
         <joint name="$(arg arm_id)_joint_2" value="-1.570796"/>
@@ -60,5 +60,5 @@
         <joint name="$(arg arm_id)_joint_6" value="-3.1415926"/>
     </group_state>
-        <group_state name="endrotate" group="fr">
+        <group_state name="endrotate" group="fr5">
         <joint name="$(arg arm_id)_joint_1" value="0"/>
         <joint name="$(arg arm_id)_joint_2" value="-1.570796"/>
