Commit message: 20251230所有关于工具部分全部更新

File: src/zlab_robots_descriptions/diana7_description/urdf/diana7_macro.xacro (robot description, xacro)
@@ -432,5 +432,5 @@
       <parent link="${prefix}_link_7" />
       <child link="${prefix}_ee_link" />
-      <origin xyz="0 0 0" rpy="3.1415926531795866 0 1.5707963266" />
+      <origin xyz="0 0 0" rpy="3.1415926531795866 0 -1.5707963266" />
     </joint>
     <!-- Tool Loading -->

File: src/zlab_robots_descriptions/zlab_tools_description/tools/calibration_tool/urdf/calibration_tool.urdf.xacro (robot description, xacro)
@@ -1,77 +1,6 @@
 <?xml version="1.0" encoding="utf-8"?>
-<robot xmlns:xacro="http://www.ros.org/wiki/xacro" name="calibration_tool">
-  <!-- 1) 实体：只在一个 link 上保留 mesh/collision/inertial（这里选 base） -->
-  <link name="${tool_arm_id}_calibration_base_link">
-    <inertial>
-      <origin xyz="8.68737263231918E-11 0.0497527045553807 0.00249999998593278" rpy="0 0 0"/>
-      <mass value="0.031694702045305"/>
-      <inertia ixx="7.92231294487921E-05" ixy="3.02800948370523E-15" ixz="-4.01660599408829E-15"
-               iyy="1.01746769831227E-05" iyz="-6.07540568485497E-15" izz="8.28804530559537E-05"/>
-    </inertial>
-    <visual>
-      <origin xyz="0 0 0" rpy="0 0 0"/>
-      <geometry>
-        <mesh filename="package://zlab_tools_description/tools/calibration_tool/meshes/visual/calibration_base_link.STL"/>
-      </geometry>
-      <material name="">
-        <color rgba="1 1 1 1"/>
-      </material>
-    </visual>
-    <collision>
-      <origin xyz="0 0 0" rpy="0 0 0"/>
-      <geometry>
-        <mesh filename="package://zlab_tools_description/tools/calibration_tool/meshes/collision/calibration_base_link.STL"/>
-      </geometry>
-    </collision>
-  </link>
-  <!-- 2) frame-only：ee -->
-  <link name="${tool_arm_id}_calibration_ee_link"/>
-  <joint name="${tool_arm_id}_calibration_ee" type="fixed">
-    <origin xyz="0 0 0.005" rpy="0 0 0"/>
-    <parent link="${tool_arm_id}_calibration_base_link"/>
-    <child link="${tool_arm_id}_calibration_ee_link"/>
-  </joint>
-  <!-- 3) frame-only：tcp -->
-  <link name="${tool_arm_id}_calibration_tcp_link"/>
-  <joint name="${tool_arm_id}_calibration_tcp" type="fixed">
-    <origin xyz="0 0.0915 -0.0025" rpy="0 0 0"/>
-    <parent link="${tool_arm_id}_calibration_ee_link"/>
-    <child link="${tool_arm_id}_calibration_tcp_link"/>
-  </joint>
-  <!-- 五个tcp link -->
-  <!-- front_tag: z 朝前，与 tcp 同向 -->
-  <link name="${tool_arm_id}_front_tag"/>
-  <joint name="${tool_arm_id}_tcp_to_front_tag" type="fixed">
-    <origin xyz="0 0 0.02" rpy="0 0 0"/>
-    <parent link="${tool_arm_id}_calibration_tcp_link"/>
-    <child link="${tool_arm_id}_front_tag"/>
-  </joint>
-  <!-- back_tag: z 朝后，绕 y 轴转 pi -->
-  <link name="${tool_arm_id}_back_tag"/>
-  <joint name="${tool_arm_id}_tcp_to_back_tag" type="fixed">
-    <origin xyz="0 0 -0.02" rpy="0 3.141592653589793 0"/>
-    <parent link="${tool_arm_id}_calibration_tcp_link"/>
-    <child link="${tool_arm_id}_back_tag"/>
-  </joint>
-  <!-- left_tag: z 朝左（-x），绕 y 轴转 -pi/2 -->
-  <link name="${tool_arm_id}_left_tag"/>
-  <joint name="${tool_arm_id}_tcp_to_left_tag" type="fixed">
-    <origin xyz="-0.02 0 0" rpy="0 -1.5707963267948966 0"/>
-    <parent link="${tool_arm_id}_calibration_tcp_link"/>
-    <child link="${tool_arm_id}_left_tag"/>
-  </joint>
-  <!-- right_tag: z 朝右（+x），绕 y 轴转 +pi/2 -->
-  <link name="${tool_arm_id}_right_tag"/>
-  <joint name="${tool_arm_id}_tcp_to_right_tag" type="fixed">
-    <origin xyz="0.02 0 0" rpy="0 1.5707963267948966 0"/>
-    <parent link="${tool_arm_id}_calibration_tcp_link"/>
-    <child link="${tool_arm_id}_right_tag"/>
-  </joint>
-  <!-- top_tag: z 朝上（+y），绕 x 轴转 -pi/2 -->
-  <link name="${tool_arm_id}_top_tag"/>
-  <joint name="${tool_arm_id}_tcp_to_top_tag" type="fixed">
-    <origin xyz="0 0.02 0" rpy="-1.5707963267948966 0 0"/>
-    <parent link="${tool_arm_id}_calibration_tcp_link"/>
-    <child link="${tool_arm_id}_top_tag"/>
-  </joint>
+<robot name="calibration_tool" xmlns:xacro="http://www.ros.org/wiki/xacro">
+  <xacro:include filename="$(find zlab_tools_description)/tools/calibration_tool/urdf/calibration_tool_macro.xacro"/>
+  <!-- Instantiate Links using tool_arm_id prefix -->
+  <xacro:calibration_tool_links prefix="${tool_arm_id}" />
 </robot>

File: src/zlab_robots_descriptions/zlab_tools_description/tools/electronic_magnet/urdf/electronic_magnet.urdf (robot description, URDF)
Before this commit: robot electronic_magnet, 3 links, 2 joints
Links:
- removed link em_base_link
- removed link em_ee_link
- removed link em_tcp_link
- added link electronic_magnet_base_link, mass 0.12279; collision mesh filename=package://zlab_tools_description/tools/electronic_magnet/me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; visual mesh filename=package://zlab_tools_description/tools/electronic_magnet/me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
- added link electronic_magnet_ee_link, mass 4.7133; collision mesh filename=package://zlab_tools_description/tools/electronic_magnet/me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; visual mesh filename=package://zlab_tools_description/tools/electronic_magnet/me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
- added link electronic_magnet_tcp_link, mass 4.7133; collision mesh filename=package://zlab_tools_description/tools/electronic_magnet/me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; visual mesh filename=package://zlab_tools_description/tools/electronic_magnet/me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
Joints:
- joint electro_magnet: child em_tcp_link -> electronic_magnet_tcp_link; parent em_base_link -> electronic_magnet_base_link
- joint electromagnet_ee: child em_ee_link -> electronic_magnet_ee_link; parent em_tcp_link -> electronic_magnet_tcp_link

File: src/zlab_robots_descriptions/zlab_tools_description/tools/electronic_magnet/urdf/electronic_magnet.urdf.xacro (robot description, xacro)
@@ -1,151 +1,6 @@
 <?xml version="1.0" encoding="utf-8"?>
-<!-- This URDF was automatically created by SolidWorks to URDF Exporter! Originally created by Stephen Brawner (brawner@gmail.com)
-     Commit Version: 1.6.0-4-g7f85cfe  Build Version: 1.6.7995.38578
-     For more information, please see http://wiki.ros.org/sw_urdf_exporter -->
 <robot name="electronic_magnet" xmlns:xacro="http://www.ros.org/wiki/xacro">
-  <!-- Arm ID: 从父xacro文件传递的全局变量tool_arm_id -->
-  <!-- 直接使用tool_arm_id作为前缀，避免循环定义 -->
-  <!-- Prefix for link names to avoid conflicts in dual arm setup -->
-  <xacro:property name="prefix" value="${tool_arm_id}_"/>
-  <link name="${prefix}em_base_link">
-    <inertial>
-      <origin
-        xyz="-8.3267E-17 0.00012355 0.0077014"
-        rpy="0 0 0" />
-      <mass
-        value="0.12279" />
-      <inertia
-        ixx="2.413E-05"
-        ixy="-5.9292E-21"
-        ixz="6.5341E-20"
-        iyy="2.4481E-05"
-        iyz="-7.2797E-08"
-        izz="3.9841E-05" />
-    </inertial>
-    <visual>
-      <origin
-        xyz="0 0 0"
-        rpy="0 0 0" />
-      <geometry>
-        <mesh
-          filename="package://zlab_tools_description/tools/electronic_magnet/meshes/visual/em_base_link.STL" />
-      </geometry>
-      <material
-        name="">
-        <color
-          rgba="1 0.94902 0.89804 1" />
-      </material>
-    </visual>
-    <collision>
-      <origin
-        xyz="0 0 0"
-        rpy="0 0 0" />
-      <geometry>
-        <mesh
-          filename="package://zlab_tools_description/tools/electronic_magnet/meshes/collision/em_base_link.STL" />
-      </geometry>
-    </collision>
-  </link>
-  <link name="${prefix}em_tcp_link">
-    <inertial>
-      <origin
-        xyz="2.7756E-17 2.7756E-17 9.5087E-05"
-        rpy="0 0 0" />
-      <mass
-        value="4.7133" />
-      <inertia
-        ixx="0.024838"
-        ixy="0"
-        ixz="-1.1723E-18"
-        iyy="0.024838"
-        iyz="2.1387E-19"
-        izz="0.0017594" />
-    </inertial>
-    <visual>
-      <origin
-        xyz="0 0 0"
-        rpy="0 0 0" />
-      <geometry>
-        <mesh
-          filename="package://zlab_tools_description/tools/electronic_magnet/meshes/visual/em_tcp_link.STL" />
-      </geometry>
-      <material
-        name="">
-        <color
-          rgba="0.53725 0.34902 0.33725 1" />
-      </material>
-    </visual>
-    <collision>
-      <origin
-        xyz="0 0 0"
-        rpy="0 0 0" />
-      <geometry>
-        <mesh
-          filename="package://zlab_tools_description/tools/electronic_magnet/meshes/collision/em_tcp_link.STL" />
-      </geometry>
-    </collision>
-  </link>
-  <joint
-    name="${prefix}electro_magnet"
-    type="fixed">
-    <origin
-      xyz="0 0.00023753 0.145"
-      rpy="0 0 0" />
-    <parent
-      link="${prefix}em_base_link" />
-    <child
-      link="${prefix}em_tcp_link" />
-  </joint>
-  <link name="${prefix}em_ee_link">
-    <inertial>
-      <origin
-        xyz="2.7756E-17 2.7756E-17 -0.1249"
-        rpy="0 0 0" />
-      <mass
-        value="4.7133" />
-      <inertia
-        ixx="0.024838"
-        ixy="0"
-        ixz="-1.1723E-18"
-        iyy="0.024838"
-        iyz="2.1387E-19"
-        izz="0.0017594" />
-    </inertial>
-    <visual>
-      <origin
-        xyz="0 0 0"
-        rpy="0 0 0" />
-      <geometry>
-        <mesh
-          filename="package://zlab_tools_description/tools/electronic_magnet/meshes/visual/em_ee_link.STL" />
-      </geometry>
-      <material
-        name="">
-        <color
-          rgba="0.53725 0.34902 0.33725 1" />
-      </material>
-    </visual>
-    <collision>
-      <origin
-        xyz="0 0 0"
-        rpy="0 0 0" />
-      <geometry>
-        <mesh
-          filename="package://zlab_tools_description/tools/electronic_magnet/meshes/collision/em_ee_link.STL" />
-      </geometry>
-    </collision>
-  </link>
-  <joint
-    name="${prefix}electromagnet_ee"
-    type="fixed">
-    <origin
-      xyz="0 0 0.125"
-      rpy="0 0 0" />
-    <parent
-      link="${prefix}em_tcp_link" />
-    <child
-      link="${prefix}em_ee_link" />
-    <axis
-      xyz="0 0 0" />
-  </joint>
+  <xacro:include filename="$(find zlab_tools_description)/tools/electronic_magnet/urdf/electronic_magnet_macro.xacro"/>
+  <!-- Instantiate Links using tool_arm_id prefix -->
+  <xacro:electronic_magnet_links prefix="${tool_arm_id}" />
 </robot>

File: src/zlab_robots_descriptions/zlab_tools_description/tools/electronic_magnet/urdf/electronic_magnet_macro.xacro (robot description, xacro)
@@ -1,11 +1,7 @@
 <?xml version="1.0" encoding="utf-8"?>
 <robot xmlns:xacro="http://www.ros.org/wiki/xacro">
-  <xacro:macro name="electronic_magnet" params="prefix parent">
-    <joint name="${prefix}tool_joint" type="fixed">
-      <parent link="${parent}"/>
-      <child link="${prefix}em_base_link"/>
-      <origin xyz="0 0 0" rpy="0 0 0"/>
-    </joint>
-    <link name="${prefix}em_base_link">
+  <!-- Macro for Links and Internal Joints -->
+  <xacro:macro name="electronic_magnet_links" params="prefix">
+    <link name="${prefix}_electronic_magnet_base_link">
       <inertial>
         <origin xyz="-8.3267E-17 0.00012355 0.0077014" rpy="0 0 0" />
@@ -16,5 +12,5 @@
         <origin xyz="0 0 0" rpy="0 0 0" />
         <geometry>
-          <mesh filename="package://zlab_tools_description/tools/electronic_magnet/meshes/visual/em_base_link.STL" />
+          <mesh filename="package://zlab_tools_description/tools/electronic_magnet/meshes/visual/electronic_magnet_base_link.STL" />
         </geometry>
         <material name="">
@@ -25,9 +21,9 @@
         <origin xyz="0 0 0" rpy="0 0 0" />
         <geometry>
-          <mesh filename="package://zlab_tools_description/tools/electronic_magnet/meshes/collision/em_base_link.STL" />
+          <mesh filename="package://zlab_tools_description/tools/electronic_magnet/meshes/collision/electronic_magnet_base_link.STL" />
         </geometry>
       </collision>
     </link>
-    <link name="${prefix}em_tcp_link">
+    <link name="${prefix}_electronic_magnet_tcp_link">
       <inertial>
         <origin xyz="2.7756E-17 2.7756E-17 9.5087E-05" rpy="0 0 0" />
@@ -38,5 +34,5 @@
         <origin xyz="0 0 0" rpy="0 0 0" />
         <geometry>
-          <mesh filename="package://zlab_tools_description/tools/electronic_magnet/meshes/visual/em_tcp_link.STL" />
+          <mesh filename="package://zlab_tools_description/tools/electronic_magnet/meshes/visual/electronic_magnet_tcp_link.STL" />
         </geometry>
         <material name="">
@@ -47,40 +43,29 @@
         <origin xyz="0 0 0" rpy="0 0 0" />
         <geometry>
-          <mesh filename="package://zlab_tools_description/tools/electronic_magnet/meshes/collision/em_tcp_link.STL" />
+          <mesh filename="package://zlab_tools_description/tools/electronic_magnet/meshes/collision/electronic_magnet_tcp_link.STL" />
         </geometry>
       </collision>
     </link>
-    <joint name="${prefix}em_tcp_joint" type="fixed">
+    <joint name="${prefix}_electronic_magnet_tcp_joint" type="fixed">
       <origin xyz="0 0.00023753 0.145" rpy="0 0 0" />
-      <parent link="${prefix}em_base_link" />
-      <child link="${prefix}em_tcp_link" />
+      <parent link="${prefix}_electronic_magnet_base_link" />
+      <child link="${prefix}_electronic_magnet_tcp_link" />
     </joint>
-    <link name="${prefix}em_ee_link">
-      <inertial>
-        <origin xyz="2.7756E-17 2.7756E-17 -0.1249" rpy="0 0 0" />
-        <mass value="4.7133" />
-        <inertia ixx="0.024838" ixy="0" ixz="-1.1723E-18" iyy="0.024838" iyz="2.1387E-19" izz="0.0017594" />
-      </inertial>
-      <visual>
-        <origin xyz="0 0 0" rpy="0 0 0" />
-        <geometry>
-          <mesh filename="package://zlab_tools_description/tools/electronic_magnet/meshes/visual/em_ee_link.STL" />
-        </geometry>
-        <material name="">
-          <color rgba="0.53725 0.34902 0.33725 1" />
-        </material>
-      </visual>
-      <collision>
-        <origin xyz="0 0 0" rpy="0 0 0" />
-        <geometry>
-          <mesh filename="package://zlab_tools_description/tools/electronic_magnet/meshes/collision/em_ee_link.STL" />
-        </geometry>
-      </collision>
+    <link name="${prefix}_electronic_magnet_ee_link">
     </link>
-    <joint name="${prefix}em_ee_joint" type="fixed">
+    <joint name="${prefix}_electronic_magnet_ee_joint" type="fixed">
       <origin xyz="0 0 0.125" rpy="0 0 0" />
-      <parent link="${prefix}em_tcp_link" />
-      <child link="${prefix}em_ee_link" />
+      <parent link="${prefix}_electronic_magnet_tcp_link" />
+      <child link="${prefix}_electronic_magnet_ee_link" />
     </joint>
   </xacro:macro>
+  <!-- Macro for Full Tool (includes joint to parent) -->
+  <xacro:macro name="electronic_magnet" params="prefix parent">
+    <joint name="${prefix}_tool_joint" type="fixed">
+      <parent link="${parent}"/>
+      <child link="${prefix}_electronic_magnet_base_link"/>
+      <origin xyz="0 0 0" rpy="0 0 0"/>
+    </joint>
+    <xacro:electronic_magnet_links prefix="${prefix}" />
+  </xacro:macro>
 </robot>

File: src/zlab_robots_descriptions/zlab_tools_description/tools/magnetic_sensor_bracket/urdf/bracket_macro.xacro (robot description, xacro)
@@ -1,11 +1,7 @@
 <?xml version="1.0" encoding="utf-8"?>
 <robot xmlns:xacro="http://www.ros.org/wiki/xacro">
-  <xacro:macro name="magnetic_sensor_bracket" params="prefix parent">
-    <joint name="${prefix}tool_joint" type="fixed">
-      <parent link="${parent}"/>
-      <child link="${prefix}bracket_base_link"/>
-      <origin xyz="0 0 0" rpy="0 0 0"/>
-    </joint>
-    <link name="${prefix}bracket_base_link">
+  <!-- Macro for Links and Internal Joints -->
+  <xacro:macro name="magnetic_sensor_bracket_links" params="prefix">
+    <link name="${prefix}_magnetic_sensor_bracket_base_link">
       <inertial>
         <origin xyz="6.56146448854258E-18 0.000826414697970227 0.0706784267775077" rpy="0 0 0" />
@@ -29,5 +25,5 @@
       </collision>
     </link>
-    <link name="${prefix}bracket_tcp_link">
+    <link name="${prefix}_magnetic_sensor_bracket_tcp_link">
       <inertial>
         <origin xyz="0.036673 0.024999 -0.077722" rpy="0 0 0" />
@@ -37,10 +33,19 @@
       <!-- TCP link intentionally has no visual/collision geometry to avoid duplicating the tool mesh -->
     </link>
-    <joint name="${prefix}bracket_tcp_joint" type="fixed">
+    <joint name="${prefix}_magnetic_sensor_bracket_tcp_joint" type="fixed">
       <origin xyz="0 0 0.13" rpy="0 0 0" />
-      <parent link="${prefix}bracket_base_link" />
-      <child link="${prefix}bracket_tcp_link" />
+      <parent link="${prefix}_magnetic_sensor_bracket_base_link" />
+      <child link="${prefix}_magnetic_sensor_bracket_tcp_link" />
       <axis xyz="0 0 0" />
     </joint>
   </xacro:macro>
+  <!-- Macro for Full Tool (includes joint to parent) -->
+  <xacro:macro name="magnetic_sensor_bracket" params="prefix parent">
+    <joint name="${prefix}_tool_joint" type="fixed">
+      <parent link="${parent}"/>
+      <child link="${prefix}_magnetic_sensor_bracket_base_link"/>
+      <origin xyz="0 0 0" rpy="0 0 0"/>
+    </joint>
+    <xacro:magnetic_sensor_bracket_links prefix="${prefix}" />
+  </xacro:macro>
 </robot>

File: src/zlab_robots_descriptions/zlab_tools_description/tools/magnetic_sensor_bracket/urdf/magnetic_sensor_bracket.urdf.xacro (robot description, xacro)
@@ -1,46 +1,6 @@
 <?xml version="1.0" encoding="utf-8"?>
-<!-- This URDF was automatically created by SolidWorks to URDF Exporter! Originally created by Stephen Brawner (brawner@gmail.com)
-     Commit Version: 1.6.0-4-g7f85cfe  Build Version: 1.6.7995.38578
-     For more information, please see http://wiki.ros.org/sw_urdf_exporter -->
-<robot xmlns:xacro="http://www.ros.org/wiki/xacro"
-  name="bracket">
-  <!-- Arm ID: 从父xacro文件传递的全局变量tool_arm_id -->
-  <!-- 直接使用tool_arm_id作为前缀，避免循环定义 -->
-  <!-- Prefix for link names to avoid conflicts in dual arm setup -->
-  <xacro:property name="prefix" value="${tool_arm_id}_"/>
-  <link name="${prefix}bracket_base_link">
-    <inertial>
-      <origin xyz="6.56146448854258E-18 0.000826414697970227 0.0706784267775077" rpy="0 0 0" />
-      <mass value="0.0579905724459555" />
-      <inertia ixx="0.000211769100600281" ixy="-3.38369218983175E-21" ixz="-3.91554592312132E-21" iyy="0.00020950452248673" iyz="-3.65286260042818E-06" izz="2.30343305370622E-05" />
-    </inertial>
-    <visual>
-      <origin xyz="0 0 0" rpy="0 0 0" />
-      <geometry>
-        <mesh filename="package://zlab_tools_description/tools/magnetic_sensor_bracket/meshes/bracket_base_link.STL" />
-      </geometry>
-      <material name="">
-        <color rgba="0.792156862745098 0.819607843137255 0.933333333333333 1.0" />
-      </material>
-    </visual>
-    <collision>
-      <origin xyz="0 0 0" rpy="0 0 0" />
-      <geometry>
-        <mesh filename="package://zlab_tools_description/tools/magnetic_sensor_bracket/meshes/bracket_base_link.STL" />
-      </geometry>
-    </collision>
-  </link>
-  <link name="${prefix}bracket_tcp_link">
-    <inertial>
-      <origin xyz="0.036673 0.024999 -0.077722" rpy="0 0 0" />
-      <mass value="0.0001" />
-      <inertia ixx="1e-6" ixy="0" ixz="0" iyy="1e-6" iyz="0" izz="1e-6" />
-    </inertial>
-    <!-- TCP link intentionally has no geometry; visualization happens on bracket_base_link -->
-  </link>
-  <joint name="${prefix}bracket_tcp_joint" type="fixed">
-    <parent link="${prefix}bracket_base_link" />
-    <child link="${prefix}bracket_tcp_link" />
-    <origin xyz="-0.024999 0.037499 0.1484" rpy="0 0 -1.5708" />
-  </joint>
+<robot name="bracket" xmlns:xacro="http://www.ros.org/wiki/xacro">
+  <xacro:include filename="$(find zlab_tools_description)/tools/magnetic_sensor_bracket/urdf/bracket_macro.xacro"/>
+  <!-- Instantiate Links using tool_arm_id prefix -->
+  <xacro:magnetic_sensor_bracket_links prefix="${tool_arm_id}" />
 </robot>

File: src/zlab_robots_descriptions/zlab_tools_description/tools/magnetometer_array/urdf/magnetometer_array.urdf.xacro (robot description, xacro)
@@ -8,4 +8,4 @@
   <xacro:include filename="$(find zlab_tools_description)/tools/magnetometer_array/urdf/magnetometer_array_macro.xacro"/>
   <!-- 实例化 Links，使用机械臂前缀 -->
-  <xacro:magnetometer_array_links prefix="${tool_arm_id}_" />
+  <xacro:magnetometer_array_links prefix="${tool_arm_id}" />
 </robot>

File: src/zlab_robots_descriptions/zlab_tools_description/tools/magnetometer_array/urdf/magnetometer_array_macro.xacro (robot description, xacro)
@@ -3,5 +3,5 @@
   <!-- 仅定义 Links 的宏 -->
   <xacro:macro name="magnetometer_array_links" params="prefix">
-    <link name="${prefix}magnetometer_base_link">
+    <link name="${prefix}_magnetometer_array_base_link">
       <inertial>
         <origin xyz="-2.07166456525017E-07 0.0021604655211999 0.0362476651991424" rpy="0 0 0" />
@@ -24,13 +24,7 @@
         </geometry>
       </collision>
-    </link>
-    <link name="${prefix}magnetometer_tcp_link">
-      <inertial>
-        <origin xyz="-0.000190659438675016 0.00189080741259228 -0.0604428602463941" rpy="0 0 0" />
-        <mass value="0.00226226919267647" />
-        <inertia ixx="3.35022731202412E-07" ixy="6.2725681636899E-20" ixz="-6.82910069048886E-10" iyy="4.1094183087163E-07" iyz="1.82178739960353E-19" izz="8.71724385779425E-08" />
-      </inertial>
+      <!-- TCP Geometry moved to Base Link to avoid self-collision -->
       <visual>
-        <origin xyz="0 0 0" rpy="0 0 0" />
+        <origin xyz="0 0.00023753 0.19309" rpy="0 0 0" />
         <geometry>
           <mesh filename="package://zlab_tools_description/tools/magnetometer_array/meshes/magnetometer_tcp_link.STL" />
@@ -41,5 +35,5 @@
       </visual>
       <collision>
-        <origin xyz="0 0 0" rpy="0 0 0" />
+        <origin xyz="0 0.00023753 0.19309" rpy="0 0 0" />
         <geometry>
           <mesh filename="package://zlab_tools_description/tools/magnetometer_array/meshes/magnetometer_tcp_link.STL" />
@@ -47,8 +41,16 @@
       </collision>
     </link>
-    <joint name="${prefix}magnetometer_joint" type="fixed">
+    <link name="${prefix}_magnetometer_array_tcp_link">
+      <inertial>
+        <origin xyz="-0.000190659438675016 0.00189080741259228 -0.0604428602463941" rpy="0 0 0" />
+        <mass value="0.00226226919267647" />
+        <inertia ixx="3.35022731202412E-07" ixy="6.2725681636899E-20" ixz="-6.82910069048886E-10" iyy="4.1094183087163E-07" iyz="1.82178739960353E-19" izz="8.71724385779425E-08" />
+      </inertial>
+      <!-- Visual and Collision moved to base_link -->
+    </link>
+    <joint name="${prefix}_magnetometer_array_tcp_joint" type="fixed">
       <origin xyz="0 0.00023753 0.19309" rpy="0 0 0" />
-      <parent link="${prefix}magnetometer_base_link" />
-      <child link="${prefix}magnetometer_tcp_link" />
+      <parent link="${prefix}_magnetometer_array_base_link" />
+      <child link="${prefix}_magnetometer_array_tcp_link" />
       <axis xyz="0 0 0" />
     </joint>
@@ -56,7 +58,7 @@
   <!-- 完整定义的宏（包含与 parent 的连接） -->
   <xacro:macro name="magnetometer_array" params="prefix parent">
-    <joint name="${prefix}tool_joint" type="fixed">
+    <joint name="${prefix}_tool_joint" type="fixed">
       <parent link="${parent}"/>
-      <child link="${prefix}magnetometer_base_link"/>
+      <child link="${prefix}_magnetometer_array_base_link"/>
       <origin xyz="0 0 0" rpy="0 0 0"/>
     </joint>
