Commit message: 20251230所有关于工具部分全部更新

File: src/zlab_robots_descriptions/zlab_tools_description/tools/permanent_magnet/urdf/permanent_magnet.urdf.xacro (robot description, xacro)
@@ -1,53 +1,10 @@
 <?xml version="1.0" encoding="utf-8"?>
 <robot xmlns:xacro="http://www.ros.org/wiki/xacro" name="permanent_magnet">
-  <link name="${tool_arm_id}_pm_base_link">
-    <inertial>
-      <origin xyz="-1.4589E-05 0.00097471 0.054744" rpy="0 0 0" />
-      <mass value="0.136" />
-      <inertia ixx="0.00022399" ixy="1.6941E-08" ixz="-9.6464E-09" iyy="0.00018815" iyz="1.4376E-05" izz="0.00010598" />
-    </inertial>
-    <visual>
-      <origin xyz="0 0 0" rpy="0 0 0" />
-      <geometry>
-        <mesh filename="package://zlab_tools_description/tools/permanent_magnet/meshes/visual/pm_base_link.STL" />
-      </geometry>
-      <material name="">
-        <color rgba="1 1 1 1" />
-      </material>
-    </visual>
-    <collision>
-      <origin xyz="0 0 0" rpy="0 0 0" />
-      <geometry>
-        <mesh filename="package://zlab_tools_description/tools/permanent_magnet/meshes/collision/pm_base_link.STL" />
-      </geometry>
-    </collision>
-  </link>
-  <link name="${tool_arm_id}_pm_tcp_link">
-    <inertial>
-      <origin xyz="-1.4589E-05 0.00097471 -0.026256" rpy="0 0 0" />
-      <mass value="0.136" />
-      <inertia ixx="0.00022399" ixy="1.6941E-08" ixz="-9.6464E-09" iyy="0.00018815" iyz="1.4376E-05" izz="0.00010598" />
-    </inertial>
-    <visual>
-      <origin xyz="0 0 0" rpy="0 0 0" />
-      <geometry>
-        <mesh filename="package://zlab_tools_description/tools/permanent_magnet/meshes/visual/pm_tcp_link.STL" />
-      </geometry>
-      <material name="">
-        <color rgba="1 1 1 1" />
-      </material>
-    </visual>
-    <collision>
-      <origin xyz="0 0 0" rpy="0 0 0" />
-      <geometry>
-        <mesh filename="package://zlab_tools_description/tools/permanent_magnet/meshes/collision/pm_tcp_link.STL" />
-      </geometry>
-    </collision>
-  </link>
-  <joint name="${tool_arm_id}_permanent_magnet" type="fixed">
-    <origin xyz="0 0 0.081" rpy="0 0 0" />
-    <parent link="${tool_arm_id}_pm_base_link" />
-    <child link="${tool_arm_id}_pm_tcp_link" />
-    <axis xyz="0 0 0" />
-  </joint>
+  <xacro:arg name="prefix" default=""/>
+  <xacro:arg name="parent" default="tool0"/>
+  <xacro:include filename="$(find zlab_tools_description)/tools/permanent_magnet/urdf/permanent_magnet_macro.xacro"/>
+  <link name="$(arg parent)"/>
+  <xacro:permanent_magnet prefix="$(arg prefix)" parent="$(arg parent)">
+    <origin xyz="0 0 0" rpy="0 0 0"/>
+  </xacro:permanent_magnet>
 </robot>

File: src/zlab_robots_descriptions/zlab_tools_description/tools/permanent_magnet/urdf/permanent_magnet_macro.xacro (robot description, xacro)
@@ -1,16 +1,7 @@
 <?xml version="1.0" encoding="utf-8"?>
 <robot xmlns:xacro="http://www.ros.org/wiki/xacro">
-  <xacro:macro name="permanent_magnet" params="prefix parent">
-    <joint name="${prefix}tool_joint" type="fixed">
-      <parent link="${parent}"/>
-      <child link="${prefix}pm_base_link"/>
-      <origin xyz="0 0 0" rpy="0 0 0"/>
-    </joint>
-    <link name="${prefix}pm_base_link">
-      <inertial>
-        <origin xyz="-1.4589E-05 0.00097471 0.054744" rpy="0 0 0" />
-        <mass value="0.136" />
-        <inertia ixx="0.00022399" ixy="1.6941E-08" ixz="-9.6464E-09" iyy="0.00018815" iyz="1.4376E-05" izz="0.00010598" />
-      </inertial>
+  <!-- Macro for Links and Internal Joints -->
+  <xacro:macro name="permanent_magnet_links" params="prefix">
+    <link name="${prefix}_permanent_magnet_base_link">
       <visual>
         <origin xyz="0 0 0" rpy="0 0 0" />
@@ -22,4 +13,14 @@
         </material>
       </visual>
+      <!-- Moved TCP visual to base link to avoid self-collision issues -->
+      <visual>
+        <origin xyz="0 0 0.12" rpy="0 0 0" /> <!-- TODO: Verify this offset -->
+        <geometry>
+          <mesh filename="package://zlab_tools_description/tools/permanent_magnet/meshes/visual/pm_tcp_link.STL" />
+        </geometry>
+        <material name="">
+          <color rgba="0.8 0.8 0.8 1" />
+        </material>
+      </visual>
       <collision>
         <origin xyz="0 0 0" rpy="0 0 0" />
@@ -29,31 +30,18 @@
       </collision>
     </link>
-    <link name="${prefix}pm_tcp_link">
-      <inertial>
-        <origin xyz="-1.4589E-05 0.00097471 -0.026256" rpy="0 0 0" />
-        <mass value="0.136" />
-        <inertia ixx="0.00022399" ixy="1.6941E-08" ixz="-9.6464E-09" iyy="0.00018815" iyz="1.4376E-05" izz="0.00010598" />
-      </inertial>
-      <visual>
-        <origin xyz="0 0 0" rpy="0 0 0" />
-        <geometry>
-          <mesh filename="package://zlab_tools_description/tools/permanent_magnet/meshes/visual/pm_tcp_link.STL" />
-        </geometry>
-        <material name="">
-          <color rgba="1 1 1 1" />
-        </material>
-      </visual>
-      <collision>
-        <origin xyz="0 0 0" rpy="0 0 0" />
-        <geometry>
-          <mesh filename="package://zlab_tools_description/tools/permanent_magnet/meshes/collision/pm_tcp_link.STL" />
-        </geometry>
-      </collision>
-    </link>
-    <joint name="${prefix}pm_tcp_joint" type="fixed">
-      <origin xyz="0 0 0.081" rpy="0 0 0" />
-      <parent link="${prefix}pm_base_link" />
-      <child link="${prefix}pm_tcp_link" />
-      <axis xyz="0 0 0" />
+    <link name="${prefix}_permanent_magnet_tcp"/>
+    <joint name="${prefix}_permanent_magnet_tcp_joint" type="fixed">
+      <origin xyz="0 0 0.12" rpy="0 0 0" /> <!-- TODO: Verify this offset -->
+      <parent link="${prefix}_permanent_magnet_base_link" />
+      <child link="${prefix}_permanent_magnet_tcp" />
+    </joint>
+  </xacro:macro>
+  <!-- Macro for Tool Instantiation -->
+  <xacro:macro name="permanent_magnet" params="prefix parent *origin">
+    <xacro:permanent_magnet_links prefix="${prefix}"/>
+    <joint name="${prefix}_permanent_magnet_joint" type="fixed">
+      <xacro:insert_block name="origin"/>
+      <parent link="${parent}"/>
+      <child link="${prefix}_permanent_magnet_base_link"/>
     </joint>
   </xacro:macro>

File: src/zlab_robots_moveit_config/fr5_dual_moveit_config/config/zlab_dual_arms.srdf.xacro (robot description, xacro)
@@ -179,3 +179,11 @@
     <disable_collisions link1="arm2_link_4" link2="arm2_link_6" reason="Never"/>
     <disable_collisions link1="arm2_link_5" link2="arm2_link_6" reason="Adjacent"/>
+    <xacro:macro name="disable_tool_collisions" params="prefix tool_name last_link ee_link">
+        <xacro:unless value="${tool_name == 'none'}">
+            <disable_collisions link1="${ee_link}" link2="${prefix}_${tool_name}_base_link" reason="Adjacent"/>
+            <disable_collisions link1="${last_link}" link2="${prefix}_${tool_name}_base_link" reason="Adjacent"/>
+        </xacro:unless>
+    </xacro:macro>
+    <xacro:disable_tool_collisions prefix="arm1" tool_name="$(arg arm1_tool)" last_link="arm1_link_6" ee_link="arm1_ee_link"/>
+    <xacro:disable_tool_collisions prefix="arm2" tool_name="$(arg arm2_tool)" last_link="arm2_link_6" ee_link="arm2_ee_link"/>
 </robot>

File: src/zlab_robots_moveit_config/triple_arm_moveit_config/config/zlab_triple_arms.srdf.xacro (robot description, xacro)
@@ -1,4 +1,8 @@
 <?xml version="1.0" encoding="UTF-8"?>
 <robot name="zlab_triple_arms" xmlns:xacro="http://www.ros.org/wiki/xacro">
+    <xacro:arg name="arm1_tool" default="none"/>
+    <xacro:arg name="arm2_tool" default="none"/>
+    <xacro:arg name="diana7_tool" default="none"/>
+    <xacro:property name="diana7_tool" value="$(arg diana7_tool)"/>
     <!-- GROUPS -->
     <group name="arm1">
@@ -115,4 +119,6 @@
     <!-- Diana7 Internal -->
     <disable_collisions link1="diana7_pedestal_link" link2="diana7_base_link" reason="Adjacent" />
+    <disable_collisions link1="diana7_pedestal_link" link2="diana7_pedestal_flange_link" reason="Adjacent" />
+    <disable_collisions link1="diana7_pedestal_flange_link" link2="diana7_base_link" reason="Adjacent" />
     <disable_collisions link1="diana7_base_link" link2="diana7_link_1" reason="Adjacent" />
     <disable_collisions link1="diana7_link_1" link2="diana7_link_2" reason="Adjacent" />
@@ -125,3 +131,13 @@
     <!-- We leave cross-collisions enabled for safety, except maybe bases if they overlap in model but not reality -->
     <!-- Assuming bases are far enough apart (0.8m) -->
+    <!-- Tool Collisions -->
+    <xacro:macro name="disable_tool_collisions" params="prefix tool_name last_link ee_link">
+        <xacro:unless value="${tool_name == 'none'}">
+            <disable_collisions link1="${ee_link}" link2="${prefix}_${tool_name}_base_link" reason="Adjacent"/>
+            <disable_collisions link1="${last_link}" link2="${prefix}_${tool_name}_base_link" reason="Adjacent"/>
+        </xacro:unless>
+    </xacro:macro>
+    <xacro:disable_tool_collisions prefix="arm1" tool_name="$(arg arm1_tool)" last_link="arm1_link_6" ee_link="arm1_ee_link"/>
+    <xacro:disable_tool_collisions prefix="arm2" tool_name="$(arg arm2_tool)" last_link="arm2_link_6" ee_link="arm2_ee_link"/>
+    <xacro:disable_tool_collisions prefix="diana7" tool_name="$(arg diana7_tool)" last_link="diana7_link_7" ee_link="diana7_ee_link"/>
 </robot>
