Commit message: 20260126 添加新的工具

File: src/zlab_robots_moveit_config/fr5_dual_moveit_config/config/zlab_dual_arms.srdf.xacro (robot description, xacro)
@@ -182,11 +182,25 @@
     <disable_collisions link1="arm2_link_4" link2="arm2_link_6" reason="Never"/>
     <disable_collisions link1="arm2_link_5" link2="arm2_link_6" reason="Adjacent"/>
-    <xacro:macro name="disable_tool_collisions" params="prefix tool_name last_link ee_link">
+    <xacro:macro name="disable_tool_collisions" params="prefix tool_name last_link ee_link prev_link">
         <xacro:unless value="${tool_name == 'none'}">
+            <!-- 禁用工具基座与机械臂末端链接的碰撞 -->
             <disable_collisions link1="${ee_link}" link2="${prefix}_${tool_name}_base_link" reason="Adjacent"/>
             <disable_collisions link1="${last_link}" link2="${prefix}_${tool_name}_base_link" reason="Adjacent"/>
+            <disable_collisions link1="${prev_link}" link2="${prefix}_${tool_name}_base_link" reason="Never"/>
+            <!-- 加载工具配置以获取更多链接信息 -->
+            <xacro:property name="tool_config_file" value="$(find tools_description)/tools/${tool_name}/config/tool.yaml"/>
+            <xacro:property name="tool_config" value="${xacro.load_yaml(tool_config_file)}"/>
+            <!-- 如果存在TCP链接，也禁用其与机械臂末端的碰撞（某些工具TCP链接较大） -->
+            <xacro:if value="${'urdf_package' in tool_config}">
+                <xacro:property name="tcp_link_name" value="${tool_config['urdf_package']['tcp_link_name']}"/>
+                <disable_collisions link1="${ee_link}" link2="${prefix}_${tcp_link_name}" reason="Never"/>
+                <disable_collisions link1="${last_link}" link2="${prefix}_${tcp_link_name}" reason="Never"/>
+                <disable_collisions link1="${prev_link}" link2="${prefix}_${tcp_link_name}" reason="Never"/>
+                <!-- 禁用工具内部链接之间的碰撞 -->
+                <disable_collisions link1="${prefix}_${tool_name}_base_link" link2="${prefix}_${tcp_link_name}" reason="Adjacent"/>
+            </xacro:if>
         </xacro:unless>
     </xacro:macro>
-    <xacro:disable_tool_collisions prefix="arm1" tool_name="$(arg arm1_tool)" last_link="arm1_link_6" ee_link="arm1_ee_link"/>
-    <xacro:disable_tool_collisions prefix="arm2" tool_name="$(arg arm2_tool)" last_link="arm2_link_6" ee_link="arm2_ee_link"/>
+    <xacro:disable_tool_collisions prefix="arm1" tool_name="$(arg arm1_tool)" last_link="arm1_link_6" ee_link="arm1_ee_link" prev_link="arm1_link_5"/>
+    <xacro:disable_tool_collisions prefix="arm2" tool_name="$(arg arm2_tool)" last_link="arm2_link_6" ee_link="arm2_ee_link" prev_link="arm2_link_5"/>
 </robot>

File: src/zlab_robots_moveit_config/fr5_single_moveit_config/config/fr5.srdf.xacro (robot description, xacro)
@@ -7,4 +7,5 @@
     <!-- Arm ID parameter -->
     <xacro:arg name="arm_id" default="arm1" />
+    <xacro:arg name="tool_name" default="none" />
     <!--GROUPS: Representation of a set of joints and links. This can be useful for specifying DOF to plan for, defining arms, end effectors, etc-->
     <!--LINKS: When a link is specified, the parent joint of that link (if it exists) is automatically included-->
@@ -82,3 +83,24 @@
     <disable_collisions link1="$(arg arm_id)_link_4" link2="$(arg arm_id)_link_6" reason="Never"/>
     <disable_collisions link1="$(arg arm_id)_link_5" link2="$(arg arm_id)_link_6" reason="Adjacent"/>
+    <xacro:macro name="disable_tool_collisions" params="prefix tool_name last_link ee_link prev_link">
+        <xacro:unless value="${tool_name == 'none'}">
+            <!-- 禁用工具基座与机械臂末端链接的碰撞 -->
+            <disable_collisions link1="${ee_link}" link2="${prefix}_${tool_name}_base_link" reason="Adjacent"/>
+            <disable_collisions link1="${last_link}" link2="${prefix}_${tool_name}_base_link" reason="Adjacent"/>
+            <disable_collisions link1="${prev_link}" link2="${prefix}_${tool_name}_base_link" reason="Never"/>
+            <!-- 加载工具配置以获取更多链接信息 -->
+            <xacro:property name="tool_config_file" value="$(find tools_description)/tools/${tool_name}/config/tool.yaml"/>
+            <xacro:property name="tool_config" value="${xacro.load_yaml(tool_config_file)}"/>
+            <!-- 如果存在TCP链接，也禁用其与机械臂末端的碰撞（某些工具TCP链接较大） -->
+            <xacro:if value="${'urdf_package' in tool_config}">
+                <xacro:property name="tcp_link_name" value="${tool_config['urdf_package']['tcp_link_name']}"/>
+                <disable_collisions link1="${ee_link}" link2="${prefix}_${tcp_link_name}" reason="Never"/>
+                <disable_collisions link1="${last_link}" link2="${prefix}_${tcp_link_name}" reason="Never"/>
+                <disable_collisions link1="${prev_link}" link2="${prefix}_${tcp_link_name}" reason="Never"/>
+                <!-- 禁用工具内部链接之间的碰撞 -->
+                <disable_collisions link1="${prefix}_${tool_name}_base_link" link2="${prefix}_${tcp_link_name}" reason="Adjacent"/>
+            </xacro:if>
+        </xacro:unless>
+    </xacro:macro>
+    <xacro:disable_tool_collisions prefix="$(arg arm_id)" tool_name="$(arg tool_name)" last_link="$(arg arm_id)_link_6" ee_link="$(arg arm_id)_ee_link" prev_link="$(arg arm_id)_link_5"/>
 </robot>

File: src/zlab_robots_moveit_config/triple_arm_moveit_config/config/zlab_triple_arms.srdf.xacro (robot description, xacro)
@@ -132,12 +132,26 @@
     <!-- Assuming bases are far enough apart (0.8m) -->
     <!-- Tool Collisions -->
-    <xacro:macro name="disable_tool_collisions" params="prefix tool_name last_link ee_link">
+    <xacro:macro name="disable_tool_collisions" params="prefix tool_name last_link ee_link prev_link">
         <xacro:unless value="${tool_name == 'none'}">
+            <!-- 禁用工具基座与机械臂末端链接的碰撞 -->
             <disable_collisions link1="${ee_link}" link2="${prefix}_${tool_name}_base_link" reason="Adjacent"/>
             <disable_collisions link1="${last_link}" link2="${prefix}_${tool_name}_base_link" reason="Adjacent"/>
+            <disable_collisions link1="${prev_link}" link2="${prefix}_${tool_name}_base_link" reason="Never"/>
+            <!-- 加载工具配置以获取更多链接信息 -->
+            <xacro:property name="tool_config_file" value="$(find tools_description)/tools/${tool_name}/config/tool.yaml"/>
+            <xacro:property name="tool_config" value="${xacro.load_yaml(tool_config_file)}"/>
+            <!-- 如果存在TCP链接，也禁用其与机械臂末端的碰撞（某些工具TCP链接较大） -->
+            <xacro:if value="${'urdf_package' in tool_config}">
+                <xacro:property name="tcp_link_name" value="${tool_config['urdf_package']['tcp_link_name']}"/>
+                <disable_collisions link1="${ee_link}" link2="${prefix}_${tcp_link_name}" reason="Never"/>
+                <disable_collisions link1="${last_link}" link2="${prefix}_${tcp_link_name}" reason="Never"/>
+                <disable_collisions link1="${prev_link}" link2="${prefix}_${tcp_link_name}" reason="Never"/>
+                <!-- 禁用工具内部链接之间的碰撞 -->
+                <disable_collisions link1="${prefix}_${tool_name}_base_link" link2="${prefix}_${tcp_link_name}" reason="Adjacent"/>
+            </xacro:if>
         </xacro:unless>
     </xacro:macro>
-    <xacro:disable_tool_collisions prefix="arm1" tool_name="$(arg arm1_tool)" last_link="arm1_link_6" ee_link="arm1_ee_link"/>
-    <xacro:disable_tool_collisions prefix="arm2" tool_name="$(arg arm2_tool)" last_link="arm2_link_6" ee_link="arm2_ee_link"/>
-    <xacro:disable_tool_collisions prefix="diana7" tool_name="$(arg diana7_tool)" last_link="diana7_link_7" ee_link="diana7_ee_link"/>
+    <xacro:disable_tool_collisions prefix="arm1" tool_name="$(arg arm1_tool)" last_link="arm1_link_6" ee_link="arm1_ee_link" prev_link="arm1_link_5"/>
+    <xacro:disable_tool_collisions prefix="arm2" tool_name="$(arg arm2_tool)" last_link="arm2_link_6" ee_link="arm2_ee_link" prev_link="arm2_link_5"/>
+    <xacro:disable_tool_collisions prefix="diana7" tool_name="$(arg diana7_tool)" last_link="diana7_link_7" ee_link="diana7_ee_link" prev_link="diana7_link_6"/>
 </robot>
