Commit message: 20260126 修改工具坐标bug

File: src/zlab_robots_descriptions/tools_description/tools/bracket/urdf/bracket_macro.xacro (robot description, xacro)
@@ -25,5 +25,5 @@
       </collision>
     </link>
-    <link name="${prefix}_bracket_ee_Link">
+    <link name="${prefix}_bracket_tcp_link">
       <inertial>
         <origin xyz="0.0057496 -2.6647E-05 -0.036233" rpy="0 0 0" />
@@ -50,5 +50,5 @@
       <origin xyz="0 0 0.1616" rpy="0 0 0" />
       <parent link="${prefix}_bracket_base_link" />
-      <child link="${prefix}_bracket_ee_Link" />
+      <child link="${prefix}_bracket_tcp_link" />
       <axis xyz="0 0 0" />
     </joint>

File: src/zlab_robots_descriptions/tools_description/tools/permanent_magnet/urdf/permanent_magnet_macro.xacro (robot description, xacro)
@@ -30,9 +30,9 @@
       </collision>
     </link>
-    <link name="${prefix}_permanent_magnet_tcp"/>
+    <link name="${prefix}_permanent_magnet_tcp_link"/>
     <joint name="${prefix}_permanent_magnet_tcp_joint" type="fixed">
       <origin xyz="0 0 0.12" rpy="0 0 0" /> <!-- TODO: Verify this offset -->
       <parent link="${prefix}_permanent_magnet_base_link" />
-      <child link="${prefix}_permanent_magnet_tcp" />
+      <child link="${prefix}_permanent_magnet_tcp_link" />
     </joint>
   </xacro:macro>
